File: chorus/chorus/chorus.sch (KiCad schematic (older format))
At the start: 19 parts, among them J1 IN, J3 Jack-DC, J4 OUT, SW1 SW_3PDT_x3, U2 TL074, U5 LM7805, U6 TL072, U8 TLE2426xLP

Commit message: assembled psu and clock
Other:
- note added: "TODO: do we need to scale up and back down the signal\nto increase the dynamic range?\nTypical guitar signal is +/- 0.5V. Line level can be +/- 2V.\nOpamps should be able to handle +/- 3V without clipping.\nIf the delay is more efficient with higher signals, can scale up\nand back down on the summing stages"
- note added: "TODO: use other LM13700 buffer on output?"
- note removed: "TODO: do we need to scale up and back down the signal\nto increase the dynamic range?"
- note removed: "todo: tone filter has a smaller filter\nwhich with the aggressive filters\ncreates a notch at ~2-3KHz (depending on tone pos)\nis this a problem? Making a 8th order filter to fix it doesn’t\nseem worthwhile…"
Changed lines of the file:
@@
 	1    0    0    -1
 $EndComp
-Text Notes 1950 7350 0    50   ~ 0
-TODO: do we need to scale up and back down the signal\nto increase the dynamic range?
+Text Notes 1900 7700 0    50   ~ 0
+TODO: do we need to scale up and back down the signal\nto increase the dynamic range?\nTypical guitar signal is +/- 0.5V. Line level can be +/- 2V.\nOpamps should be able to handle +/- 3V without clipping.\nIf the delay is more efficient with higher signals, can scale up\nand back down on the summing stages
 Text Notes 1950 7050 0    50   ~ 0
 TODO: pots oriented correctly?
@@
 Wire Wire Line
 	8050 5400 2100 5400
-Text Notes 4400 6900 0    50   ~ 0
-todo: tone filter has a smaller filter\nwhich with the aggressive filters\ncreates a notch at ~2-3KHz (depending on tone pos)\nis this a problem? Making a 8th order filter to fix it doesn’t\nseem worthwhile…
 Text Notes 7700 5700 0    50   ~ 0
 sum half dry signal plus half wet signal
+Text Notes 9600 4750 0    50   ~ 0
+TODO: use other LM13700 buffer on output?
 $EndSCHEMATC
