File: chorus/chorus/chorus.kicad_pcb (KiCad board)
At the start: 2 copper layers, 54.6 x 95.2 mm, 46 parts, among them J1 IN, J2 ISP, J3 Jack-DC, J4 OUT, Q1 2N3904, SW1 SW_3PDT_x3, U1 ATTINY85, U2 TL074, U3 MN3102, U4 MN3207, U5 LM7805, U6 TL072

Commit message: redesign
Parts:
- removed Q1: 2N3904, Package_TO_SOT_THT:TO-92_Inline
- added C10: 3.3u, Capacitor_THT:C_Disc_D6.0mm_W2.5mm_P5.00mm, F.Cu at (201.3, 118.7)
- added C11: 33n, Capacitor_THT:C_Disc_D6.0mm_W2.5mm_P5.00mm, F.Cu at (207.7, 135.5)
- added C12: 33n, Capacitor_THT:C_Disc_D6.0mm_W2.5mm_P5.00mm, F.Cu at (207.7, 139.6)
- added R20: 100K, Resistor_THT:R_Axial_DIN0204_L3.6mm_D1.6mm_P2.54mm_Vertical, F.Cu at (232.4, 122.6)
- added R21: 100K, Resistor_THT:R_Axial_DIN0204_L3.6mm_D1.6mm_P2.54mm_Vertical, F.Cu at (234.3, 127.0)
- added R22: 5.6K, Resistor_THT:R_Axial_DIN0204_L3.6mm_D1.6mm_P2.54mm_Vertical, F.Cu at (226.1, 127.0)
- added R23: 5.6K, Resistor_THT:R_Axial_DIN0204_L3.6mm_D1.6mm_P2.54mm_Vertical, F.Cu at (225.4, 121.9)
- added R24: 1K, Resistor_THT:R_Axial_DIN0204_L3.6mm_D1.6mm_P2.54mm_Vertical, F.Cu at (207.7, 143.2)
- added R25: 1K, Resistor_THT:R_Axial_DIN0204_L3.6mm_D1.6mm_P2.54mm_Vertical, F.Cu at (207.7, 146.3)
- added RV_AGND_TRIMMER1: 5K, Potentiometer_THT:Potentiometer_Bourns_3296W_Vertical, F.Cu at (193.7, 108.0)
- added U7: MN3207, Package_DIP:DIP-8_W7.62mm, F.Cu at (161.3, 110.5)
- C1: value 33n -> 100n
- C2: value 33n -> 220n
- C3: value 3.3u -> 470p
- R10: value 5.6K -> 5.1k
- R11: value 5.6K -> 2.2k
- R12: value 240 -> 10k
- R13: value 240 -> 220
- R3: value 1K -> 100K
- R4: value 1K -> 1M
- R5: value 10K -> 10k
- R8: value 100K -> 240
- R9: value 100K -> 2.5k
- U1: value ATTINY85 -> LM13700; footprint Package_DIP:DIP-8_W7.62mm -> Package_DIP:DIP-16_W7.62mm
- U3: value MN3102 -> ATTINY85
- U4: value MN3207 -> MN3102
- moved R15 162.1 mm to (176.3, 64.5), turned to 180 degrees
- moved R14 160.0 mm to (177.8, 59.4)
- moved R16 155.1 mm to (173.7, 70.1)
- moved R4 147.1 mm to (163.6, 49.3), turned to 180 degrees
- moved R1 146.0 mm to (155.4, 54.4), turned to 90 degrees
- moved R6 129.6 mm to (191.8, 114.9), turned to 270 degrees
- moved R12 121.8 mm to (206.2, 116.3), turned to 270 degrees
- moved R3 120.2 mm to (151.9, 85.3)
- moved R2 117.4 mm to (154.9, 67.1), turned to 270 degrees
- moved R19 114.1 mm to (228.6, 104.8), turned to 180 degrees
- moved R18 111.4 mm to (226.1, 110.5)
- moved R7 109.2 mm to (195.6, 117.5), turned to 90 degrees
- moved R17 108.1 mm to (228.6, 116.8), turned to 180 degrees
- moved R8 93.2 mm to (66.0, 48.8), turned to 270 degrees
- moved R10 90.8 mm to (140.2, 59.9), turned to 270 degrees
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Connections:
- C2 pad 1: Net-(C2-Pad1) -> GND
- C2 pad 2: Net-(C1-Pad1) -> LFO_OUT
- C3 pad 1: GND -> Net-(C3-Pad1)
- C3 pad 2: Net-(C3-Pad2) -> GNDA
- C6 pad 1: /Anti-Aliasing Filter/OUT -> /delay/IN
- C9 pad 1: /sheet629A6A5C/OUT -> /Anti-Aliasing Filter 2/OUT
- D1 pad 2: +5V -> LFO_OUT
- J2 pad 1: LFO_CLOCK -> MISO
- R10 pad 1: /sheet629A6A5C/IN -> +9V
- R11 pad 1: /sheet629A6A5C/IN -> Net-(R11-Pad1)
- R11 pad 2: Net-(R11-Pad2) -> GNDA
- R12 pad 1: Net-(D1-Pad1) -> /Clock Generator/CLOCK
- R12 pad 2: LFO_CLOCK -> GND
- R17 pad 2: /sheet629A6A5C/IN -> /Anti-Aliasing Filter 2/IN
- R2 pad 1: Net-(C1-Pad2) -> /Tone Filter/IN
- R3 pad 1: Net-(R3-Pad1) -> Net-(C1-Pad2)
- R3 pad 2: Net-(C2-Pad1) -> GND
- R4 pad 1: Net-(R4-Pad1) -> Net-(C1-Pad1)
- R4 pad 2: Net-(C1-Pad1) -> GNDA
- R5 pad 1: BBD_CLOCK -> LFO_OUT
- R5 pad 2: +9V -> MOSI
- R7 pad 2: Net-(R6-Pad1) -> Net-(R7-Pad2)
- R8 pad 1: GNDA -> Net-(D1-Pad1)
- R8 pad 2: Net-(R11-Pad2) -> GND
- R9 pad 1: GNDA -> LFO_OUT
- R9 pad 2: Net-(R10-Pad2) -> Net-(R9-Pad2)
- R_CUTOFF_1 pad 2: Net-(R3-Pad1) -> Net-(R24-Pad1)
- R_CUTOFF_1 pad 3: Net-(R3-Pad1) -> Net-(R24-Pad1)
- R_CUTOFF_1 pad 5: Net-(R4-Pad1) -> Net-(R25-Pad1)
- R_CUTOFF_1 pad 6: Net-(R4-Pad1) -> Net-(R25-Pad1)
- R_FLANGE1 pad 1: Net-(R_FLANGE1-Pad1) -> /Anti-Aliasing Filter 2/OUT
- R_FLANGE1 pad 2: Net-(R_FLANGE1-Pad1) -> /Anti-Aliasing Filter 2/OUT
- SW1 pad 7: /sheet629A6A5C/OUT -> Net-(C1-Pad1)
- U1 pad 1: ~RST -> Net-(R10-Pad2)
- U1 pad 2: Net-(R_RATE1-Pad2) -> Net-(U1-Pad2)
- U1 pad 3: Net-(R_DEPTH1-Pad2) -> Net-(R11-Pad1)
- U1 pad 4: GND -> Net-(C3-Pad1)
- U1 pad 5: MOSI -> Net-(R11-Pad1)
- U1 pad 6: LFO_CLOCK -> (no net)
- U1 pad 7: SCK -> Net-(R11-Pad1)
- U1 pad 8: +5V -> /Clock Generator/CLOCK
- U2 pad 1: Net-(C1-Pad2) -> /Tone Filter/IN
- U2 pad 10: /sheet629A6A5C/OUT -> (no net)
- U2 pad 12: Net-(R6-Pad1) -> Net-(RV_AGND_TRIMMER1-Pad2)
- U2 pad 5: Net-(C2-Pad1) -> Net-(C12-Pad1)
- U2 pad 8: Net-(R_FLANGE1-Pad1) -> (no net)
- U2 pad 9: Net-(R_FLANGE1-Pad1) -> (no net)
- U3 pad 1: +9V -> ~RST
- U3 pad 2: Net-(U3-Pad2) -> Net-(R_RATE1-Pad2)
- U3 pad 3: GND -> Net-(R_DEPTH1-Pad2)
- U3 pad 4: Net-(U3-Pad4) -> GND
- U3 pad 5: Net-(U3-Pad5) -> MOSI
- U3 pad 6: Net-(U3-Pad6) -> MISO
- U3 pad 7: BBD_CLOCK -> SCK
- U3 pad 8: Net-(C3-Pad2) -> +5V
- U4 pad 1: GND -> +9V
- U4 pad 2: Net-(U3-Pad2) -> Net-(U4-Pad2)
- U4 pad 3: /Anti-Aliasing Filter/OUT -> GND
- U4 pad 4: Net-(C3-Pad2) -> Net-(U4-Pad4)
- U4 pad 5: +9V -> Net-(U4-Pad5)
- U4 pad 6: Net-(U3-Pad4) -> Net-(U4-Pad6)
- U4 pad 7: Net-(R10-Pad2) -> /Clock Generator/CLOCK
- U4 pad 8: Net-(R11-Pad2) -> Net-(C10-Pad2)
- U6 pad 1: /Anti-Aliasing Filter/OUT -> /delay/IN
- U6 pad 2: /Anti-Aliasing Filter/OUT -> /delay/IN
- U6 pad 6: /sheet629A6A5C/OUT -> /Anti-Aliasing Filter 2/OUT
- U6 pad 7: /sheet629A6A5C/OUT -> /Anti-Aliasing Filter 2/OUT
Routing:
- net Net-(J3-Pad1): track 0.00 -> 111.6 mm, vias 0 -> 1
- net GND: track 0.00 -> 68.1 mm
- net +9V: track 0.00 -> 65.5 mm
- net Net-(J4-PadT): track 0.00 -> 49.5 mm
- net +5V: track 0.00 -> 39.7 mm
- net Net-(J1-PadR): track 0.00 -> 32.5 mm
- net Net-(D2-Pad1): track 0.00 -> 14.2 mm
- net Net-(SW1-Pad3): track 0.00 -> 10.1 mm
- added copper zone on F.Cu, net GNDA
Other:
- board size 54.6 x 95.2 mm -> 143.5 x 95.2 mm
- board text added: "TODO: height?"

Commit message: update to kicad 6
Parts:
- removed RV_AGND_TRIMMER1: 5K, Potentiometer_THT:Potentiometer_Bourns_3296W_Vertical
- added R26: 500K, kicad-legacy/kicad-footprints/Resistor_THT.pretty:R_Axial_DIN0204_L3.6mm_D1.6mm_P2.54mm_Vertical, F.Cu at (256.2, 62.8)
- added R27: 1K, kicad-legacy/kicad-footprints/Resistor_THT.pretty:R_Axial_DIN0204_L3.6mm_D1.6mm_P2.54mm_Vertical, F.Cu at (212.6, 65.9)
- added R28: 5.6k, kicad-legacy/kicad-footprints/Resistor_THT.pretty:R_Axial_DIN0204_L3.6mm_D1.6mm_P2.54mm_Vertical, F.Cu at (207.0, 72.3)
- added R29: 100K, kicad-legacy/kicad-footprints/Resistor_THT.pretty:R_Axial_DIN0204_L3.6mm_D1.6mm_P2.54mm_Vertical, F.Cu at (212.6, 62.8)
- added R30: 100K, kicad-legacy/kicad-footprints/Resistor_THT.pretty:R_Axial_DIN0204_L3.6mm_D1.6mm_P2.54mm_Vertical, F.Cu at (201.4, 69.2)
- added R31: 100K, kicad-legacy/kicad-footprints/Resistor_THT.pretty:R_Axial_DIN0204_L3.6mm_D1.6mm_P2.54mm_Vertical, F.Cu at (207.0, 69.2)
- added R32: 100K, kicad-legacy/kicad-footprints/Resistor_THT.pretty:R_Axial_DIN0204_L3.6mm_D1.6mm_P2.54mm_Vertical, F.Cu at (201.4, 72.3)
- added R33: 330, kicad-legacy/kicad-footprints/Resistor_THT.pretty:R_Axial_DIN0204_L3.6mm_D1.6mm_P2.54mm_Vertical, F.Cu at (236.6, 62.8)
- added R34: 91K, kicad-legacy/kicad-footprints/Resistor_THT.pretty:R_Axial_DIN0204_L3.6mm_D1.6mm_P2.54mm_Vertical, F.Cu at (212.3, 81.8)
- added R35: 30K, kicad-legacy/kicad-footprints/Resistor_THT.pretty:R_Axial_DIN0204_L3.6mm_D1.6mm_P2.54mm_Vertical, F.Cu at (212.3, 78.7)
- added RV1: R_TRIM_10K, kicad-legacy/Potentiometers.pretty:Potentiometer_Trimmer_Bourns_3296W, F.Cu at (208.0, 64.4)
- added U10: MN3102, kicad-legacy/Housings_DIP.pretty:DIP-8_W7.62mm, F.Cu at (224.9, 79.2)
- added U11: TL072, kicad-legacy/Housings_DIP.pretty:DIP-8_W7.62mm, F.Cu at (201.5, 79.2)
- added U8: TLE2426xLP, kicad-legacy/TO_SOT_Packages_THT.pretty:TO-92_Inline_Wide, F.Cu at (248.0, 64.4)
- added U9: ATTINY85-20PU, kicad-legacy/Housings_DIP.pretty:DIP-8_W7.62mm, F.Cu at (225.8, 63.2)
- D1, D2: footprint LED_THT:LED_D3.0mm -> kicad-official/LED_THT.pretty:LED_D3.0mm
- J1, J4: footprint Connector_Audio:Jack_6.35mm_Neutrik_NMJ6HCD2_Horizontal -> kicad-legacy/kicad-footprints/Connector_Audio.pretty:Jack_6.35mm_Neutrik_NMJ6HCD2_Horizontal
- J2: footprint Connector_PinSocket_2.54mm:PinSocket_2x03_P2.54mm_Vertical -> kicad-official/Connector_PinSocket_2.54mm.pretty:PinSocket_2x03_P2.54mm_Vertical
- J3: footprint Connector_PinSocket_2.54mm:PinSocket_2x01_P2.54mm_Vertical -> kicad-official/Connector_PinSocket_2.54mm.pretty:PinSocket_2x01_P2.54mm_Vertical
- R1, R11, R13, R2, R20, R21, R22, R23, R24, R25, R4, R8: footprint Resistor_THT:R_Axial_DIN0204_L3.6mm_D1.6mm_P2.54mm_Vertical -> kicad-legacy/kicad-footprints/Resistor_THT.pretty:R_Axial_DIN0204_L3.6mm_D1.6mm_P2.54mm_Vertical
- R10: value 5.1k -> 2.7k; footprint Resistor_THT:R_Axial_DIN0204_L3.6mm_D1.6mm_P2.54mm_Vertical -> kicad-legacy/kicad-footprints/Resistor_THT.pretty:R_Axial_DIN0204_L3.6mm_D1.6mm_P2.54mm_Vertical
- R12: value 10k -> 1K; footprint Resistor_THT:R_Axial_DIN0204_L3.6mm_D1.6mm_P2.54mm_Vertical -> kicad-legacy/kicad-footprints/Resistor_THT.pretty:R_Axial_DIN0204_L3.6mm_D1.6mm_P2.54mm_Vertical
- R14, R17: value 8.2K -> 11k; footprint Resistor_THT:R_Axial_DIN0204_L3.6mm_D1.6mm_P2.54mm_Vertical -> kicad-legacy/kicad-footprints/Resistor_THT.pretty:R_Axial_DIN0204_L3.6mm_D1.6mm_P2.54mm_Vertical
- R15: value 120k -> 150k; footprint Resistor_THT:R_Axial_DIN0204_L3.6mm_D1.6mm_P2.54mm_Vertical -> kicad-legacy/kicad-footprints/Resistor_THT.pretty:R_Axial_DIN0204_L3.6mm_D1.6mm_P2.54mm_Vertical
- R16: value 39K -> 47k; footprint Resistor_THT:R_Axial_DIN0204_L3.6mm_D1.6mm_P2.54mm_Vertical -> kicad-legacy/kicad-footprints/Resistor_THT.pretty:R_Axial_DIN0204_L3.6mm_D1.6mm_P2.54mm_Vertical
- R18: value 120k -> 75K; footprint Resistor_THT:R_Axial_DIN0204_L3.6mm_D1.6mm_P2.54mm_Vertical -> kicad-legacy/kicad-footprints/Resistor_THT.pretty:R_Axial_DIN0204_L3.6mm_D1.6mm_P2.54mm_Vertical
- R19: value 39K -> 51K; footprint Resistor_THT:R_Axial_DIN0204_L3.6mm_D1.6mm_P2.54mm_Vertical -> kicad-legacy/kicad-footprints/Resistor_THT.pretty:R_Axial_DIN0204_L3.6mm_D1.6mm_P2.54mm_Vertical
- R3, R6, R7: value 100K -> 1M; footprint Resistor_THT:R_Axial_DIN0204_L3.6mm_D1.6mm_P2.54mm_Vertical -> kicad-legacy/kicad-footprints/Resistor_THT.pretty:R_Axial_DIN0204_L3.6mm_D1.6mm_P2.54mm_Vertical
- R5: value 10k -> 100; footprint Resistor_THT:R_Axial_DIN0204_L3.6mm_D1.6mm_P2.54mm_Vertical -> kicad-legacy/kicad-footprints/Resistor_THT.pretty:R_Axial_DIN0204_L3.6mm_D1.6mm_P2.54mm_Vertical
- R9: value 2.5k -> 4.8k; footprint Resistor_THT:R_Axial_DIN0204_L3.6mm_D1.6mm_P2.54mm_Vertical -> kicad-legacy/kicad-footprints/Resistor_THT.pretty:R_Axial_DIN0204_L3.6mm_D1.6mm_P2.54mm_Vertical
- R_CUTOFF_1: footprint Potentiometer_THT:Potentiometer_Alps_RK09L_Double_Vertical -> kicad-legacy/kicad-footprints/Potentiometer_THT.pretty:Potentiometer_Alps_RK09L_Double_Vertical
- R_DEPTH1, R_FLANGE1, R_RATE1: footprint Potentiometer_THT:Potentiometer_Alps_RK09K_Single_Vertical -> kicad-legacy/kicad-footprints/Potentiometer_THT.pretty:Potentiometer_Alps_RK09K_Single_Vertical
- U1: footprint Package_DIP:DIP-16_W7.62mm -> kicad-legacy/kicad-footprints/Package_DIP.pretty:DIP-16_W7.62mm
- U2: footprint Package_DIP:DIP-14_W7.62mm -> kicad-legacy/kicad-footprints/Package_DIP.pretty:DIP-14_W7.62mm
- U3: value ATTINY85 -> TL074; footprint Package_DIP:DIP-8_W7.62mm -> kicad-legacy/kicad-footprints/Package_DIP.pretty:DIP-14_W7.62mm
- U4: value MN3102 -> TL074; footprint Package_DIP:DIP-8_W7.62mm -> kicad-legacy/kicad-footprints/Package_DIP.pretty:DIP-14_W7.62mm
- U5: footprint Package_TO_SOT_THT:TO-220-3_Vertical -> kicad-official/Package_TO_SOT_THT.pretty:TO-220F-3_Vertical
- U6, U7: footprint Package_DIP:DIP-8_W7.62mm -> kicad-legacy/Housings_DIP.pretty:DIP-8_W7.62mm
- moved J1 21.7 mm to (29.2, 95.3), turned to 180 degrees
Connections:
- D1 pad 2: LFO_OUT -> MOSI
- J2 pad 5: ~RST -> ~{RST}
- R10 pad 1: +9V -> +5V
- R17 pad 2: /Anti-Aliasing Filter 2/IN -> Net-(C15-Pad1)
- R22 pad 1: /Anti-Aliasing Filter 2/IN -> /Reconstruction Filter/IN
- R23 pad 1: /Anti-Aliasing Filter 2/IN -> /Reconstruction Filter/IN
- R3 pad 1: Net-(C1-Pad2) -> Net-(R3-Pad1)
- R3 pad 2: GND -> Net-(R26-Pad1)
- R4 pad 1: Net-(C1-Pad1) -> Net-(R26-Pad2)
- R4 pad 2: GNDA -> /Reconstruction Filter/OUT
- R5 pad 1: LFO_OUT -> Net-(C2-Pad2)
- R6 pad 1: Net-(R6-Pad1) -> Net-(R26-Pad2)
- R6 pad 2: +9V -> /Tone Filter/DRY_OUT
- R7 pad 1: GND -> Net-(R26-Pad2)
- R7 pad 2: Net-(R7-Pad2) -> Net-(R1-Pad2)
- R9 pad 1: LFO_OUT -> Net-(C2-Pad2)
- R_CUTOFF_1 pad 4: /Anti-Aliasing Filter/IN -> Net-(R27-Pad2)
- R_FLANGE1 pad 1: /Anti-Aliasing Filter 2/OUT -> Net-(R3-Pad1)
- R_FLANGE1 pad 2: /Anti-Aliasing Filter 2/OUT -> Net-(R3-Pad1)
- U1 pad 1: Net-(R10-Pad2) -> Net-(R9-Pad2)
- U1 pad 10: /Anti-Aliasing Filter 2/OUT -> (no net)
- U1 pad 12: Net-(C3-Pad1) -> Net-(R11-Pad1)
- U1 pad 13: GNDA -> Net-(C3-Pad1)
- U1 pad 15: Net-(U1-Pad15) -> unconnected-(U1-Pad15)
- U1 pad 16: Net-(R9-Pad2) -> Net-(R10-Pad2)
- U1 pad 2: Net-(U1-Pad2) -> unconnected-(U1-Pad2)
- U1 pad 4: Net-(C3-Pad1) -> GNDA
- U1 pad 5: Net-(R11-Pad1) -> Net-(C3-Pad1)
- U1 pad 8: /Clock Generator/CLOCK -> Net-(R33-Pad1)
- U1 pad 9: Net-(C1-Pad2) -> (no net)
- U2 pad 12: Net-(RV_AGND_TRIMMER1-Pad2) -> (no net)
- U2 pad 13: GNDA -> (no net)
- U2 pad 14: GNDA -> (no net)
- U2 pad 6: /Anti-Aliasing Filter/IN -> Net-(R27-Pad2)
- U2 pad 7: /Anti-Aliasing Filter/IN -> Net-(R27-Pad2)
- U3 pad 1: ~RST -> Net-(R26-Pad1)
- U3 pad 2: Net-(R_RATE1-Pad2) -> Net-(R26-Pad2)
- U3 pad 3: Net-(R_DEPTH1-Pad2) -> GNDA
- U3 pad 4: GND -> (no net)
- U3 pad 5: MOSI -> Net-(C13-Pad2)
- U3 pad 6: MISO -> /Anti-Aliasing Filter/IN
- U3 pad 7: SCK -> /Anti-Aliasing Filter/IN
- U3 pad 8: +5V -> (no net)
- U4 pad 1: +9V -> (no net)
- U4 pad 2: Net-(U4-Pad2) -> (no net)
- U4 pad 3: GND -> (no net)
- U4 pad 4: Net-(U4-Pad4) -> (no net)
- U4 pad 7: /Clock Generator/CLOCK -> /Tone Filter/DRY_OUT
- U4 pad 8: Net-(C10-Pad2) -> (no net)
- U6 pad 1: /delay/IN -> /Anti-Aliasing Filter/OUT
- U6 pad 2: /delay/IN -> /Anti-Aliasing Filter/OUT
- U6 pad 6: /Anti-Aliasing Filter 2/OUT -> /Reconstruction Filter/OUT
- U6 pad 7: /Anti-Aliasing Filter 2/OUT -> /Reconstruction Filter/OUT
- U7 pad 2: Net-(U4-Pad2) -> Net-(U10-Pad2)
- U7 pad 3: /delay/IN -> /Anti-Aliasing Filter/OUT
- U7 pad 5: +9V -> +5V
- U7 pad 6: Net-(U4-Pad4) -> Net-(U10-Pad4)
Other:
- net class Default removed
