File: chorus/chorus/file62F7B2B3.kicad_sch (KiCad schematic)
At the start: 17 parts, among them U9 ATTINY85-20PU

Commit message: add output buffer
Parts:
- C2: renamed from C?; value (none) -> 220u
- C3: renamed from C?; value (none) -> 220p
- D1: renamed from D?; value (none) -> LED
- J2: renamed from J?; value (none) -> ISP
- R10: renamed from R?; value (none) -> 2.7k
- R11, R8: renamed from R?; value (none) -> 2.2k
- R12: renamed from R?; value (none) -> 1K
- R33: renamed from R?; value (none) -> 330
- R5: renamed from R?; value (none) -> 100
- R9: renamed from R?; value (none) -> 4.8k
- R_RATE1: renamed from R_RATE?; value (none) -> 100K
- U1: renamed from U?; value (none) -> LM13700
- gave numbers to parts that had none: 1
Other:
- company: (none) -> rabidaudio
