File: splitter/splitter/splitter.sch (KiCad schematic (older format))
At the start: 33 parts, among them J1 JACKIN, J2 JACKSEND, J3 JACKRECV, J4 JACKOUT, J5 Jack-DC, J6 CONN_SEND_DRY, J7 RING_SEND, J8 CONN_RECV_DRY, J9 RING_RECV, SW1 SW_MODE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

Commit message: bug fixes
Parts:
- removed RV2: A1M_DUAL_MIX, Potentiometer_THT:Potentiometer_Alpha_RD902F-40-00D_Dual_Vertical, symbol Device:R_POT_Dual_Separate
- added RV2: B1M_MIX, Potentiometer_THT:Potentiometer_Alpha_RD901F-40-00D_Single_Vertical, symbol Device:R_POT
- R7, R8: value 1M -> 470K
- renumbered R9 to R10, R10 to R9
Connections:
- net GND: now also RV1.2
- net HIGH: now also RV1.5
- net RECV_DRY: now also R8.2
- net RECV_WET: now also R7.1
- net at R2.1, RV1.1: no longer RV1.2
- net at R1.1, RV1.4: no longer RV1.5
- net at R9.1, U1.9 (-): now also RV2.2; no longer R7.2, R8.2
- net at R8.1: now also RV2.1
- new net: R7.2, RV2.3
Other:
- note added: "TODO: check switch orientation + pins"
- note added: "input impedance: 470K to 1.4M\nop-amp output impedance (20mA @ 0.5V?)"
- note removed: "TODO: check pot orientation\nTODO: check switch orientation + pins\nTODO: verify mixer on bb\nTODO: verify switching on bb"
- note removed: "input impedance: 500K to 1M\nop-amp output impedance (20mA @ 0.5V?)"
- moved on the sheet: R7, R8
Changed lines of the file:
@@
 U 1 1 62D478AE
 P 4150 3700
-F 0 "U1" H 4150 3333 50  0000 C CNN
-F 1 "TL074" H 4150 3424 50  0000 C CNN
+F 0 "U1" H 4250 3550 50  0000 C CNN
+F 1 "TL074" H 4100 3700 50  0000 C CNN
 F 2 "Package_DIP:DIP-14_W7.62mm" H 4100 3800 50  0001 C CNN
 F 3 "http://www.ti.com/lit/ds/symlink/tl071.pdf" H 4200 3900 50  0001 C CNN
@@
 U 2 1 62D4D1DF
 P 2050 3600
-F 0 "U1" H 2050 3967 50  0000 C CNN
-F 1 "TL074" H 2050 3876 50  0000 C CNN
+F 0 "U1" H 2100 3800 50  0000 C CNN
+F 1 "TL074" H 2000 3600 50  0000 C CNN
 F 2 "Package_DIP:DIP-14_W7.62mm" H 2000 3700 50  0001 C CNN
 F 3 "http://www.ti.com/lit/ds/symlink/tl071.pdf" H 2100 3800 50  0001 C CNN
@@
 $EndComp
 Text Notes 7400 5700 0    50   ~ 0
-TODO: check pot orientation\nTODO: check switch orientation + pins\nTODO: verify mixer on bb\nTODO: verify switching on bb
+TODO: check switch orientation + pins
 $Comp
 L power:GND #PWR02
@@
 Connection ~ 4500 3700
 Wire Wire Line
-	3450 3000 3350 3000
-Wire Wire Line
 	3600 2850 3600 2750
-Wire Wire Line
-	3600 2750 3350 2750
-Wire Wire Line
-	3350 2750 3350 3000
-Connection ~ 3350 3000
-Wire Wire Line
-	3350 3000 3300 3000
 Wire Wire Line
 	2850 3600 2950 3600
@@
 	3550 3600 3850 3600
 Wire Wire Line
-	3550 4150 3550 4200
-Wire Wire Line
-	3550 4200 3350 4200
-Wire Wire Line
-	3350 4200 3350 4400
-Wire Wire Line
-	3350 4400 3400 4400
-Connection ~ 3550 4200
-Wire Wire Line
-	3550 4200 3550 4250
-Wire Wire Line
-	3550 4550 3550 4700
-Wire Wire Line
-	3750 3000 4500 3000
+	3550 4550 3550 4600
+Wire Wire Line
+	3750 3000 3850 3000
 Wire Wire Line
 	3000 3000 2950 3000
@@
 U 3 1 62D6659B
 P 10300 3850
-F 0 "U1" H 10300 3483 50  0000 C CNN
-F 1 "TL074" H 10300 3574 50  0000 C CNN
+F 0 "U1" H 10400 4050 50  0000 C CNN
+F 1 "TL074" H 10250 3850 50  0000 C CNN
 F 2 "Package_DIP:DIP-14_W7.62mm" H 10250 3950 50  0001 C CNN
 F 3 "http://www.ti.com/lit/ds/symlink/tl071.pdf" H 10350 4050 50  0001 C CNN
@@
 U 4 1 62D7837B
 P 5600 3800
-F 0 "U1" H 5700 4050 50  0000 C CNN
-F 1 "TL074" H 5700 3950 50  0000 C CNN
+F 0 "U1" H 5750 3950 50  0000 C CNN
+F 1 "TL074" H 5550 3800 50  0000 C CNN
 F 2 "Package_DIP:DIP-14_W7.62mm" H 5550 3900 50  0001 C CNN
 F 3 "http://www.ti.com/lit/ds/symlink/tl071.pdf" H 5650 4000 50  0001 C CNN
@@
 L Device:R R8
 U 1 1 62D7B481
-P 9600 3750
-F 0 "R8" V 9807 3750 50  0000 C CNN
-F 1 "1M" V 9716 3750 50  0000 C CNN
-F 2 "Resistor_THT:R_Axial_DIN0207_L6.3mm_D2.5mm_P7.62mm_Horizontal" V 9530 3750 50  0001 C CNN
-F 3 "~" H 9600 3750 50  0001 C CNN
-	1    9600 3750
-	0    -1   -1   0
+P 9350 4150
+F 0 "R8" V 9557 4150 50  0000 C CNN
+F 1 "470K" V 9466 4150 50  0000 C CNN
+F 2 "Resistor_THT:R_Axial_DIN0207_L6.3mm_D2.5mm_P7.62mm_Horizontal" V 9280 4150 50  0001 C CNN
+F 3 "~" H 9350 4150 50  0001 C CNN
+	1    9350 4150
+	1    0    0    -1
 $EndComp
 $Comp
 L Device:R R7
 U 1 1 62D7C138
-P 9600 3300
-F 0 "R7" V 9807 3300 50  0000 C CNN
-F 1 "1M" V 9716 3300 50  0000 C CNN
-F 2 "Resistor_THT:R_Axial_DIN0207_L6.3mm_D2.5mm_P7.62mm_Horizontal" V 9530 3300 50  0001 C CNN
-F 3 "~" H 9600 3300 50  0001 C CNN
-	1    9600 3300
-	0    -1   -1   0
-$EndComp
-Wire Wire Line
-	9750 3750 9900 3750
-Connection ~ 9900 3750
-Wire Wire Line
-	9900 3750 9950 3750
-$Comp
-L Device:R_POT_Dual_Separate RV2
-U 2 1 62D7EC04
-P 9200 3300
-F 0 "RV2" H 9130 3254 50  0000 R CNN
-F 1 "A1M_DUAL_MIX" H 9130 3345 50  0000 R CNN
-F 2 "Potentiometer_THT:Potentiometer_Alpha_RD902F-40-00D_Dual_Vertical" H 9200 3300 50  0001 C CNN
-F 3 "~" H 9200 3300 50  0001 C CNN
-	2    9200 3300
-	1    0    0    -1
-$EndComp
-$Comp
-L Device:R_POT_Dual_Separate RV2
-U 1 1 62D7FACD
-P 9200 3750
-F 0 "RV2" H 9050 3700 50  0000 C CNN
-F 1 "A1M_DUAL_MIX" H 8950 3800 50  0000 C CNN
-F 2 "Potentiometer_THT:Potentiometer_Alpha_RD902F-40-00D_Dual_Vertical" H 9200 3750 50  0001 C CNN
-F 3 "~" H 9200 3750 50  0001 C CNN
-	1    9200 3750
-	1    0    0    -1
-$EndComp
-Wire Wire Line
-	9750 3300 9900 3300
-Wire Wire Line
-	9450 3750 9350 3750
-Wire Wire Line
-	9450 3300 9350 3300
-$Comp
-L power:GND #PWR07
-U 1 1 62D865EB
-P 8750 3550
-F 0 "#PWR07" H 8750 3300 50  0001 C CNN
-F 1 "GND" H 8755 3377 50  0000 C CNN
-F 2 "" H 8750 3550 50  0001 C CNN
-F 3 "" H 8750 3550 50  0001 C CNN
-	1    8750 3550
-	1    0    0    -1
-$EndComp
-Wire Wire Line
-	9200 3600 9200 3500
-Wire Wire Line
-	8750 3550 8750 3500
-Wire Wire Line
-	8750 3500 9200 3500
-Connection ~ 9200 3500
-Wire Wire Line
-	9200 3500 9200 3450
+P 9350 3350
+F 0 "R7" V 9557 3350 50  0000 C CNN
+F 1 "470K" V 9466 3350 50  0000 C CNN
+F 2 "Resistor_THT:R_Axial_DIN0207_L6.3mm_D2.5mm_P7.62mm_Horizontal" V 9280 3350 50  0001 C CNN
+F 3 "~" H 9350 3350 50  0001 C CNN
+	1    9350 3350
+	1    0    0    -1
+$EndComp
 $Comp
 L power:GND #PWR010
@@
 Wire Wire Line
 	7750 1250 7600 1250
-Text Label 9000 4100 2    50   ~ 0
+Text Label 9150 4300 2    50   ~ 0
 RECV_DRY
-Text Label 9000 3000 2    50   ~ 0
+Text Label 9150 3200 2    50   ~ 0
 RECV_WET
 Wire Wire Line
-	9000 3000 9200 3000
-Wire Wire Line
-	9200 3000 9200 3150
-Wire Wire Line
-	9000 4100 9200 4100
-Wire Wire Line
-	9200 4100 9200 3900
+	9150 3200 9350 3200
+Wire Wire Line
+	9150 4300 9350 4300
 Text Label 10750 3850 0    50   ~ 0
 OUT
@@
 Wire Wire Line
 	10900 1200 10900 1300
-Text Notes 8700 4550 0    50   ~ 0
-input impedance: 500K to 1M\nop-amp output impedance (20mA @ 0.5V?)
+Text Notes 9350 4650 0    50   ~ 0
+input impedance: 470K to 1.4M\nop-amp output impedance (20mA @ 0.5V?)
 $Comp
 L Device:LED D1
@@
 $EndComp
 $Comp
-L Device:R R9
+L Device:R R10
 U 1 1 630C9EA9
 P 8550 1600
-F 0 "R9" H 8620 1646 50  0000 L CNN
+F 0 "R10" H 8620 1646 50  0000 L CNN
 F 1 "220" H 8620 1555 50  0000 L CNN
 F 2 "Resistor_THT:R_Axial_DIN0207_L6.3mm_D2.5mm_P7.62mm_Horizontal" V 8480 1600 50  0001 C CNN
@@
 	2700 6300 2700 6650
 Wire Wire Line
-	9900 3300 9900 3750
-$Comp
-L Device:R R10
+	10550 3550 10650 3550
+Wire Wire Line
+	10250 3550 9950 3550
+Wire Wire Line
+	9950 3550 9950 3750
+Wire Wire Line
+	9950 3750 10000 3750
+Wire Wire Line
+	3550 4150 3550 4250
+Wire Wire Line
+	3550 4600 3350 4600
+Wire Wire Line
+	3350 4600 3350 4400
+Wire Wire Line
+	3350 4400 3400 4400
+Connection ~ 3550 4600
+Wire Wire Line
+	3550 4600 3550 4700
+Wire Wire Line
+	3300 3000 3450 3000
+Wire Wire Line
+	3600 2750 3850 2750
+Wire Wire Line
+	3850 2750 3850 3000
+Connection ~ 3850 3000
+Wire Wire Line
+	3850 3000 4500 3000
+$Comp
+L Device:R_POT RV2
+U 1 1 62F12114
+P 9350 3750
+F 0 "RV2" H 9281 3704 50  0000 R CNN
+F 1 "B1M_MIX" H 9281 3795 50  0000 R CNN
+F 2 "Potentiometer_THT:Potentiometer_Alpha_RD901F-40-00D_Single_Vertical" H 9350 3750 50  0001 C CNN
+F 3 "~" H 9350 3750 50  0001 C CNN
+	1    9350 3750
+	1    0    0    1
+$EndComp
+Wire Wire Line
+	9350 4000 9350 3900
+Wire Wire Line
+	9350 3500 9350 3600
+Wire Wire Line
+	9500 3750 9950 3750
+Connection ~ 9950 3750
+$Comp
+L Device:R R9
 U 1 1 640FC6F5
 P 10400 3550
-F 0 "R10" V 10607 3550 50  0000 C CNN
+F 0 "R9" V 10607 3550 50  0000 C CNN
 F 1 "1M" V 10516 3550 50  0000 C CNN
 F 2 "Resistor_THT:R_Axial_DIN0207_L6.3mm_D2.5mm_P7.62mm_Horizontal" V 10330 3550 50  0001 C CNN
@@
 	0    -1   -1   0
 $EndComp
-Wire Wire Line
-	10550 3550 10650 3550
-Wire Wire Line
-	10250 3550 9950 3550
-Wire Wire Line
-	9950 3550 9950 3750
-Connection ~ 9950 3750
-Wire Wire Line
-	9950 3750 10000 3750
 $EndSCHEMATC

Commit message: cleanup
Parts:
- C3, C4: value 10u -> .1u
Other:
- note removed: "TODO: check switch orientation + pins"
Changed lines of the file:
@@
 	-1   0    0    -1
 $EndComp
-Text Notes 7400 5700 0    50   ~ 0
-TODO: check switch orientation + pins
 $Comp
 L power:GND #PWR02
@@
 P 10900 1000
 F 0 "C3" H 11015 1046 50  0000 L CNN
-F 1 "10u" H 11015 955 50  0000 L CNN
+F 1 ".1u" H 11015 955 50  0000 L CNN
 F 2 "Capacitor_THT:CP_Radial_D6.3mm_P2.50mm" H 10938 850 50  0001 C CNN
 F 3 "~" H 10900 1000 50  0001 C CNN
@@
 P 10900 1450
 F 0 "C4" H 11015 1496 50  0000 L CNN
-F 1 "10u" H 11015 1405 50  0000 L CNN
+F 1 ".1u" H 11015 1405 50  0000 L CNN
 F 2 "Capacitor_THT:CP_Radial_D6.3mm_P2.50mm" H 10938 1300 50  0001 C CNN
 F 3 "~" H 10900 1450 50  0001 C CNN

Commit message: rev b based on learnings from assembly
Parts:
- C3, C4: footprint Capacitor_THT:CP_Radial_D6.3mm_P2.50mm -> Capacitor_THT:C_Rect_L7.0mm_W2.0mm_P5.00mm
- U2: footprint Package_TO_SOT_THT:TO-92_Inline -> Package_TO_SOT_THT:TO-92_Inline_Wide
Changed lines of the file:
@@
 F 0 "U2" H 9400 1317 50  0000 C CNN
 F 1 "TLE2426xLP" H 9400 1226 50  0000 C CNN
-F 2 "Package_TO_SOT_THT:TO-92_Inline" H 9400 550 50  0001 C CIN
+F 2 "Package_TO_SOT_THT:TO-92_Inline_Wide" H 9400 550 50  0001 C CIN
 F 3 "http://www.ti.com/lit/ds/symlink/tle2426.pdf" H 8000 1800 50  0001 C CIN
 	1    9400 950
@@
 F 0 "C3" H 11015 1046 50  0000 L CNN
 F 1 ".1u" H 11015 955 50  0000 L CNN
-F 2 "Capacitor_THT:CP_Radial_D6.3mm_P2.50mm" H 10938 850 50  0001 C CNN
+F 2 "Capacitor_THT:C_Rect_L7.0mm_W2.0mm_P5.00mm" H 10938 850 50  0001 C CNN
 F 3 "~" H 10900 1000 50  0001 C CNN
 	1    10900 1000
@@
 F 0 "C4" H 11015 1496 50  0000 L CNN
 F 1 ".1u" H 11015 1405 50  0000 L CNN
-F 2 "Capacitor_THT:CP_Radial_D6.3mm_P2.50mm" H 10938 1300 50  0001 C CNN
+F 2 "Capacitor_THT:C_Rect_L7.0mm_W2.0mm_P5.00mm" H 10938 1300 50  0001 C CNN
 F 3 "~" H 10900 1450 50  0001 C CNN
 	1    10900 1450

Commit message: rev B
Parts:
- R10: value 220 -> 1k
Connections:
- net GND: no longer J4.RN, J4.TN
- no-connect marks 3 -> 11
Changed lines of the file:
@@
 $EndComp
-Wire Wire Line
-	5550 7450 5550 7350
-Wire Wire Line
-	5550 7350 5650 7350
-Wire Wire Line
-	5650 7150 5550 7150
-Wire Wire Line
-	5550 7150 5550 7350
-Connection ~ 5550 7350
-Connection ~ 5550 7150
 Wire Wire Line
 	5650 6950 5550 6950
-Wire Wire Line
-	5550 6950 5550 7150
 $Comp
 L Connector:AudioJack3_Switch J3
@@
 P 8550 1600
 F 0 "R10" H 8620 1646 50  0000 L CNN
-F 1 "220" H 8620 1555 50  0000 L CNN
+F 1 "1k" H 8620 1555 50  0000 L CNN
 F 2 "Resistor_THT:R_Axial_DIN0207_L6.3mm_D2.5mm_P7.62mm_Horizontal" V 8480 1600 50  0001 C CNN
 F 3 "~" H 8550 1600 50  0001 C CNN
@@
 	0    -1   -1   0
 $EndComp
+NoConn ~ 5650 7350
+Wire Wire Line
+	5550 6950 5550 7450
+NoConn ~ 5650 7150
+NoConn ~ 5050 6300
+NoConn ~ 6550 6600
+NoConn ~ 7800 8400
+NoConn ~ 5300 4700
+NoConn ~ 4250 4350
+NoConn ~ 6900 6600
 $EndSCHEMATC

Commit message: cleanup
Connections:
- no-connect marks 11 -> 5
Other:
- note added: "power led\nmay need to adjust resistor for brightness"
- note removed: "power led"
Changed lines of the file:
@@
 power filter caps, close to IC
 Text Notes 8450 2150 0    50   ~ 0
-power led
+power led\nmay need to adjust resistor for brightness
 Text Notes 6950 1700 0    50   ~ 0
 9V ac/dc center negative\ncould also be 9V battery
@@
 U 1 1 63360589
 P 3950 5600
-F 0 "J8" H 3978 5576 50  0000 L CNN
-F 1 "CONN_RECV_DRY" H 3978 5485 50  0000 L CNN
+F 0 "J8" H 4000 5550 50  0000 L CNN
+F 1 "CONN_RECV_DRY" H 3850 5700 50  0000 L CNN
 F 2 "Connector_PinSocket_2.54mm:PinSocket_1x02_P2.54mm_Vertical" H 3950 5600 50  0001 C CNN
 F 3 "~" H 3950 5600 50  0001 C CNN
@@
 P 2950 6100
 F 0 "J7" H 2978 6076 50  0000 L CNN
-F 1 "RING_SEND" H 2900 6150 50  0000 L CNN
+F 1 "RING_SEND" H 2800 6200 50  0000 L CNN
 F 2 "Connector_PinSocket_2.54mm:PinSocket_1x02_P2.54mm_Vertical" H 2950 6100 50  0001 C CNN
 F 3 "~" H 2950 6100 50  0001 C CNN
@@
 U 1 1 63576DE8
 P 4000 6100
-F 0 "J9" H 3892 5775 50  0000 C CNN
-F 1 "RING_RECV" H 4100 5950 50  0000 C CNN
+F 0 "J9" H 4050 6050 50  0000 C CNN
+F 1 "RING_RECV" H 4050 6200 50  0000 C CNN
 F 2 "Connector_PinSocket_2.54mm:PinSocket_1x02_P2.54mm_Vertical" H 4000 6100 50  0001 C CNN
 F 3 "~" H 4000 6100 50  0001 C CNN
@@
 U 1 1 6335F761
 P 2950 5600
-F 0 "J6" H 2842 5275 50  0000 C CNN
-F 1 "CONN_SEND_DRY" H 3050 5650 50  0000 C CNN
+F 0 "J6" H 3050 5550 50  0000 C CNN
+F 1 "CONN_SEND_DRY" H 3050 5700 50  0000 C CNN
 F 2 "Connector_PinSocket_2.54mm:PinSocket_1x02_P2.54mm_Vertical" H 2950 5600 50  0001 C CNN
 F 3 "~" H 2950 5600 50  0001 C CNN
@@
 	5550 6950 5550 7450
 NoConn ~ 5650 7150
-NoConn ~ 5050 6300
-NoConn ~ 6550 6600
-NoConn ~ 7800 8400
-NoConn ~ 5300 4700
-NoConn ~ 4250 4350
-NoConn ~ 6900 6600
 $EndSCHEMATC
