File: splitter/splitter/splitter.kicad_pcb (KiCad board)
At the start: 2 copper layers, 50.8 x 63 mm, 33 parts, among them J1 JACKIN, J2 JACKSEND, J3 JACKRECV, J4 JACKOUT, J5 Jack-DC, J6 CONN_SEND_DRY, J7 RING_SEND, J8 CONN_RECV_DRY, J9 RING_RECV, SW1 SW_MODE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

Commit message: refactor
Parts:
- J1: value JACKIN -> IN; footprint Connector_Audio:Jack_6.35mm_Neutrik_NMJ6HCD2_Horizontal -> kicad-legacy/kicad-footprints/Connector_Audio.pretty:Jack_6.35mm_Neutrik_NMJ6HFD2_Horizontal
- J2: value JACKSEND -> SEND; footprint Connector_Audio:Jack_6.35mm_Neutrik_NMJ6HCD2_Horizontal -> kicad-legacy/kicad-footprints/Connector_Audio.pretty:Jack_6.35mm_Neutrik_NMJ6HFD2_Horizontal
- J3: value JACKRECV -> RECV; footprint Connector_Audio:Jack_6.35mm_Neutrik_NMJ6HCD2_Horizontal -> kicad-legacy/kicad-footprints/Connector_Audio.pretty:Jack_6.35mm_Neutrik_NMJ6HFD2_Horizontal
- J4: value JACKOUT -> OUT; footprint Connector_Audio:Jack_6.35mm_Neutrik_NMJ6HCD2_Horizontal -> kicad-legacy/kicad-footprints/Connector_Audio.pretty:Jack_6.35mm_Neutrik_NMJ6HFD2_Horizontal
- J6: value CONN_SEND_DRY -> SEND2; footprint Connector_PinSocket_2.54mm:PinSocket_1x02_P2.54mm_Vertical -> kicad-legacy/kicad-footprints/Connector_Audio.pretty:Jack_6.35mm_Neutrik_NMJ6HFD2_Horizontal; moved to B.Cu
- J8: value CONN_RECV_DRY -> RECV2; footprint Connector_PinSocket_2.54mm:PinSocket_1x02_P2.54mm_Vertical -> kicad-legacy/kicad-footprints/Connector_Audio.pretty:Jack_6.35mm_Neutrik_NMJ6HFD2_Horizontal; moved to B.Cu
- R10: value 1k -> 10K
- moved J8 19.1 mm to (20.0, 10.9)
- moved R3 15.7 mm to (36.3, 19.6)
- moved J5 14.8 mm to (23.9, 13.5), turned to 180 degrees
- moved J6 12.6 mm to (40.0, 27.2), turned to 0 degrees
- moved U2 7.28 mm to (22.0, 16.8), turned to -90 degrees
- moved R7 3.38 mm to (42.7, 25.1)
- moved RV1 3.38 mm to (10.0, 21.9)
- moved RV2 3.38 mm to (45.0, 21.9)
- moved JP2 2.95 mm to (38.1, 22.4)
Connections:
- J2 pad RN: Net-(J2-PadRN) -> unconnected-(J2-PadRN)
- J2 pad TN: Net-(J2-PadTN) -> unconnected-(J2-PadTN)
- J4 pad RN: Net-(J4-PadRN) -> unconnected-(J4-PadRN)
- J4 pad TN: Net-(J4-PadTN) -> unconnected-(J4-PadTN)
- SW2 pad 3: Net-(SW2-Pad3) -> unconnected-(SW2-Pad3)
Routing:
- net /RECV_DRY: track 32.0 -> 55.0 mm
- net Net-(J5-Pad1): track 74.2 -> 97.2 mm
- net +9V: track 128.6 -> 109.2 mm
- net /SEND_DRY: track 19.2 -> 36.7 mm
- net /SEND_WET: track 57.2 -> 71.6 mm, vias 0 -> 1
- net GND: track 12.6 -> 0.40 mm, vias 3 -> 1
- net GNDD: track 60.8 -> 49.1 mm, vias 1 -> 0
- net /RECV_WET: track 35.2 -> 27.9 mm, vias 1 -> 0
- net /IN: track 73.2 -> 80.2 mm
- net Net-(R3-Pad1): track 35.3 -> 41.3 mm, vias 1 -> 0
- net Net-(R2-Pad1): track 13.3 -> 17.8 mm
- net Net-(R8-Pad1): track 11.9 -> 15.3 mm
- net Net-(R9-Pad1): track 37.5 -> 40.7 mm
- net Net-(R1-Pad1): track 8.88 -> 11.8 mm
- net /HIGH: track 57.3 -> 58.9 mm, vias 0 -> 1
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Other:
- net class Default removed
- board text added: "REV.C TONE SPLITTER 2023-08-31"
- board text removed: "REV.B CROSSOVER 2022-07-17"
- board text removed: "rabid.audio"
