File: splitter/splitter/splitter.kicad_sch (KiCad schematic)
At the start: 39 parts, among them J1 JACKIN, J2 JACKSEND, J3 JACKSEND2, J4 JACKRECV, J5 JACKRECV2, J6 JACKOUT, J7 Jack-DC, J8 Conn_01x08, J9 Conn_01x08, SW1 SW_BYPASS, SW2 SW_MODE, U1 TL074, U2 TLE2426xLP

Commit message: uncommited changes
Connections:
- net at R6.1, R9.1: now also RV2.3; no longer RV2.1
- net at R5.2, R8.1: now also RV2.1; no longer RV2.3
Changed lines of the file:
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@@
     (pin "TN")
   )
-  (symbol (lib_id "Device:R_Potentiometer") (at 223.52 99.06 0) (mirror x) (unit 1)
+  (symbol (lib_id "Device:R_Potentiometer") (at 223.52 99.06 0) (unit 1)
     (in_bom yes) (on_board yes)
-    (property "Reference" "RV2" (id 0) (at 221.7674 97.8916 0)
+    (property "Reference" "RV2" (id 0) (at 221.7674 100.2284 0)
       (effects (font (size 1.27 1.27)) (justify right))
     )
-    (property "Value" "B10K_MIX" (id 1) (at 221.7674 100.203 0)
+    (property "Value" "B10K_MIX" (id 1) (at 221.7674 97.917 0)
       (effects (font (size 1.27 1.27)) (justify right))
     )

Commit message: redesign using VCF
Parts:
- removed RV1: A1M_DUAL_CUTOFF, kicad-official/Potentiometer_THT.pretty:Potentiometer_Alpha_RD902F-40-00D_Dual_Vertical, symbol Device:R_Potentiometer_Dual_Separate
- added R10, R11: 10k, kicad-official/Resistor_SMD.pretty:R_0805_2012Metric, symbol Device:R
- added R5, R6: 220, kicad-official/Resistor_SMD.pretty:R_0805_2012Metric, symbol Device:R
- added R7, R8: 100k, kicad-official/Resistor_SMD.pretty:R_0805_2012Metric, symbol Device:R
- added R9: 2.2k, kicad-official/Resistor_SMD.pretty:R_0805_2012Metric, symbol Device:R
- added RV1: R_Potentiometer_Trim_100K, kicad-official/Potentiometer_THT.pretty:Potentiometer_Bourns_3296W_Vertical, symbol Device:R_Potentiometer_Trim
- added RV3: A100K_DUAL_MIX, kicad-official/Potentiometer_THT.pretty:Potentiometer_Alpha_RD902F-40-00D_Dual_Vertical, symbol Device:R_Potentiometer_Dual_Separate
- added U2: LM13700, kicad-official/Package_SO.pretty:SOIC-16_3.9x9.9mm_P1.27mm, symbol Amplifier_Operational:LM13700
- C1, C4, C5, C6, C7: footprint kicad-official/Capacitor_THT.pretty:C_Rect_L7.0mm_W2.5mm_P5.00mm -> kicad-official/Capacitor_SMD.pretty:C_0805_2012Metric
- C10: renamed from C8; footprint kicad-official/Capacitor_THT.pretty:C_Rect_L7.0mm_W2.5mm_P5.00mm -> kicad-official/Capacitor_SMD.pretty:C_0805_2012Metric
- C2, C3: value 6.8n -> 1.5n; footprint kicad-official/Capacitor_THT.pretty:C_Rect_L7.0mm_W2.5mm_P5.00mm -> kicad-official/Capacitor_SMD.pretty:C_0805_2012Metric
- C8: renamed from C9; footprint kicad-official/Capacitor_THT.pretty:CP_Radial_D4.0mm_P1.50mm -> kicad-official/Capacitor_SMD.pretty:C_0805_2012Metric
- C9: renamed from C10; footprint kicad-official/Capacitor_THT.pretty:CP_Radial_D4.0mm_P1.50mm -> kicad-official/Capacitor_SMD.pretty:C_0805_2012Metric
- J8: footprint kicad-official/Connector_IDC.pretty:IDC-Header_2x04_P2.54mm_Horizontal -> kicad-official/Connector_PinHeader_2.54mm.pretty:PinHeader_1x08_P2.54mm_Vertical
- J9: footprint kicad-official/Connector_IDC.pretty:IDC-Header_2x04_P2.54mm_Vertical -> kicad-official/Connector_PinHeader_2.54mm.pretty:PinHeader_1x08_P2.54mm_Vertical
- R1, R2: value 1K -> 22k; footprint kicad-official/Resistor_THT.pretty:R_Axial_DIN0207_L6.3mm_D2.5mm_P7.62mm_Horizontal -> kicad-official/Resistor_SMD.pretty:R_0805_2012Metric
- R12: renamed from R5; footprint kicad-official/Resistor_THT.pretty:R_Axial_DIN0207_L6.3mm_D2.5mm_P7.62mm_Horizontal -> kicad-official/Resistor_SMD.pretty:R_0805_2012Metric
- R13: renamed from R6; footprint kicad-official/Resistor_THT.pretty:R_Axial_DIN0207_L6.3mm_D2.5mm_P7.62mm_Horizontal -> kicad-official/Resistor_SMD.pretty:R_0805_2012Metric
- R14: renamed from R7; footprint kicad-official/Resistor_THT.pretty:R_Axial_DIN0207_L6.3mm_D2.5mm_P7.62mm_Horizontal -> kicad-official/Resistor_SMD.pretty:R_0805_2012Metric
- R15: renamed from R8; footprint kicad-official/Resistor_THT.pretty:R_Axial_DIN0207_L6.3mm_D2.5mm_P7.62mm_Horizontal -> kicad-official/Resistor_SMD.pretty:R_0805_2012Metric
- R16: renamed from R9; footprint kicad-official/Resistor_THT.pretty:R_Axial_DIN0207_L6.3mm_D2.5mm_P7.62mm_Horizontal -> kicad-official/Resistor_SMD.pretty:R_0805_2012Metric
- R17: renamed from R10; value 1.2M -> 100K; footprint kicad-official/Resistor_THT.pretty:R_Axial_DIN0207_L6.3mm_D2.5mm_P7.62mm_Horizontal -> kicad-official/Resistor_SMD.pretty:R_0805_2012Metric
- R3, R4: value 1M -> 220; footprint kicad-official/Resistor_THT.pretty:R_Axial_DIN0207_L6.3mm_D2.5mm_P7.62mm_Horizontal -> kicad-official/Resistor_SMD.pretty:R_0805_2012Metric
- RV2: value B10K_MIX -> A2.2M_RPOT_CUTOFF
- U1: footprint kicad-official/Package_DIP.pretty:DIP-14_W7.62mm_Socket -> kicad-official/Package_SO.pretty:SOIC-16_3.9x9.9mm_P1.27mm
- renumbered J4 to J3, J7 to J4, J6 to J5, J3 to J6, J5 to J7, JP3 to JP2, JP2 to JP3, U2 to U3
Connections:
- net +9V: now also R9.1, RV1.1, U2.11 (V+)
- net GND: now also C2.1, R3.2, R4.2, U1.12 (+), U1.5 (+), R5.2, R6.2; no longer RV2.2
- net GNDD: now also R10.2, R11.2, RV1.3, U2.6 (V-)
- net HIGH: now also C5.2; no longer C4.2
- net LOW: now also C4.2; no longer C5.2
- net at U1.1, U1.2 (-): now also C3.1, R2.2; no longer C4.1, R3.2
- net at R2.1: now also R4.1, U2.14 (+)
- net at R1.1: now also R3.1, U2.3 (+)
- net at C10.1, R17.2: now also U1.14; no longer U1.8
- net at R15.2, R16.2, R17.1: now also U1.13 (-); no longer U1.9 (-)
- new net: R13.1, RV3.1, U1.9 (-)
- new net: R12.2, RV3.4, RV3.5, U1.6 (-)
- new net: R15.1, RV3.6, U1.7
- new net: C2.2, U2.10, U2.12
- new net: C4.1, R10.1, R7.1, U2.9
- new net: C3.2, U2.5, U2.7
- new net: C5.1, R11.1, R8.1, U2.8
- new net: R6.1, R8.2, U2.4 (-)
- new net: R1.2, RV1.2
- new net: R5.1, R7.2, U2.13 (-)
- new net: RV2.3, U2.1, U2.16
- new net: R16.1, RV3.2, RV3.3, U1.8
- new net: R9.2, RV2.1, RV2.2
- new net: C1.1, U1.3 (+)
- no-connect marks 10 -> 12
Other:
- note added: "$ 1 0.0000015625 10.20027730826997 50 5 50 5e-11 402 96 336 224 336 1 0\s0\s40\s-9\s0\s0\s0.5 0\s0\s40\s9\s0\s0\s0.5 0\s1\s-7.493679334946873\s0.5079767893706686\s100\sdefault 0\s1\s-0.5079767893706686\s0.5077219659282157\s100\sdefault 0\s1\s0\s0.5077219659282157\s100\sdefault 0\s1\s-8.021397243928236\s0.48982985547616675\s100\sdefault 0\s1\s-8.02162952553591\s0.48975243284041936\s100\sdefault 0\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"
- note added: "1% or 5% caps"
- note added: "HP VCA"
- note added: "LP VCA"
- note added: "Parallel 1st order HP and LP VCF with adjustable cutoff. f0 = (Ra*gm)/((R+Ra)*2*pi*C) where gm ~= 19.2*Iabc R,RA chosen so ~= 1. with 1.5nF: 2mA Iabc => f0 ~= 9KHz 2uA Iabc => f0 ~= 9Hz DC blocking caps on analog boundaries because of difference in ground reference."
- note added: "TODO LIST 1. check Vpp of raw bass active, passive, and pedal output. adjust input divider as necessary 2. confirm VCFs on breadboard, with and without offset null, down to 9V supply 3. confirm mix amp on breadboard 3. compute pot orientations"
- note added: "TODO: confirm orientation"
- note added: "TODO: will this work grounded?"
- note added: "falstad sim:"
- note added: "op-amp input impedance (>1Mohm) transistor buffer output impedance (20mA @ 0.5V?)"
- note added: "power filter caps, close to ICs"
- note added: "todo can we connect these?"
- note added: "todo confirm orientation"
- note added: "voltage divider from ~2.6Vpp to 26mVpp (TODO confirm ranges)"
- note added: "wet/dry mix summing amp"
- note removed: "6.8n, 1K -> 23.4Hz, Q=0.5 6.8n, 1001K -> 23.4KHz, Q=0.5 Note: subtracting instead of creating separate LP and HP filters creates an uneven split as opposed to summing LR filters. Creating a true crossover would require VCFs, which would be more complicated. DC blocking caps on analog boundaries because of difference in ground reference."
- note removed: "op-amp input impedance (>1Mohm) op-amp output impedance (20mA @ 0.5V?)"
- note removed: "power filter caps, close to IC"
- moved on the sheet: C10, C6, C7, C8, C9, D1, J1, J2, J3, J4, J5, J6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

Commit message: do layout
Parts:
- removed R1: 22k, kicad-official/Resistor_SMD.pretty:R_0805_2012Metric, symbol Device:R
- removed RV1: R_Potentiometer_Trim_100K, kicad-official/Potentiometer_THT.pretty:Potentiometer_Bourns_3296W_Vertical, symbol Device:R_Potentiometer_Trim
- added C11, C12: 1u, kicad-official/Capacitor_SMD.pretty:C_0805_2012Metric, symbol Device:C
- U1: footprint kicad-official/Package_SO.pretty:SOIC-16_3.9x9.9mm_P1.27mm -> kicad-official/Package_SO.pretty:SOIC-14_3.9x8.7mm_P1.27mm
Connections:
- net +9V: now also J8.4 (Pin_4), C11.1; no longer J8.1 (Pin_1)
- net 9V_B: now also J9.4 (Pin_4); no longer J9.1 (Pin_1)
- net GND: now also C11.2, C12.1
- net GNDD: now also C12.2
- net IN: now also J8.3 (Pin_3); no longer J8.5 (Pin_5)
- net INR: now also J8.2 (Pin_2); no longer J8.7 (Pin_7)
- net INR_B: now also J9.2 (Pin_2); no longer J9.7 (Pin_7)
- net IN_B: now also J9.3 (Pin_3); no longer J9.5 (Pin_5)
- net LED: now also J8.1 (Pin_1); no longer J8.2 (Pin_2)
- net LED_B: now also J9.1 (Pin_1); no longer J9.2 (Pin_2)
- net OUT: now also J8.6 (Pin_6); no longer J8.3 (Pin_3)
- net OUTR: now also J8.7 (Pin_7); no longer J8.6 (Pin_6)
- net OUTR_B: now also J9.7 (Pin_7); no longer J9.6 (Pin_6)
- net OUTT: now also J8.5 (Pin_5); no longer J8.8 (Pin_8)
- net OUTT_B: now also J9.5 (Pin_5); no longer J9.8 (Pin_8)
- net OUT_B: now also J9.6 (Pin_6); no longer J9.3 (Pin_3)
- net RECVR: now also J8.8 (Pin_8); no longer J8.4 (Pin_4)
- net RECVR_B: now also J9.8 (Pin_8); no longer J9.4 (Pin_4)
Other:
- note removed: "TODO: will this work grounded?"
- moved on the sheet: C8, C9, J8, J9, R3, U1E, U2E

Commit message: fix pot orientation
Connections:
- net at R13.1, RV3.1, U1.9 (-): now also RV3.2
- net at R12.2, RV3.4, U1.6 (-): no longer RV3.5
- net at R15.1, RV3.6, U1.7: now also RV3.5
- net at RV2.3, U2.1, U2.16: now also RV2.2
- net at R16.1, RV3.3, U1.8: no longer RV3.2
- net at R9.2, RV2.1: no longer RV2.2
- net 9V_B renamed +9V_B
Other:
- note added: "pot: full clockwise -> short 1-2"
- note removed: "TODO LIST 1. check Vpp of raw bass active, passive, and pedal output. adjust input divider as necessary 2. confirm VCFs on breadboard, with and without offset null, down to 9V supply 3. confirm mix amp on breadboard 3. compute pot orientations"
- note removed: "TODO: confirm orientation"
- note removed: "todo can we connect these?"
- note removed: "todo confirm orientation"

Commit message: re-design mixer
Parts:
- removed R12, R13, R15, R16, R17: 100K, kicad-official/Resistor_SMD.pretty:R_0805_2012Metric, symbol Device:R
- removed RV3: A100K_DUAL_MIX, kicad-official/Potentiometer_THT.pretty:Potentiometer_Alpha_RD902F-40-00D_Dual_Vertical, symbol Device:R_Potentiometer_Dual_Separate
- added RV1: B100K_RPOT_MIX, kicad-official/Potentiometer_THT.pretty:Potentiometer_Alpha_RD901F-40-00D_Single_Vertical, symbol Device:R_Potentiometer
- C2, C3: value 1.5n -> 680p
- RV2: value A2.2M_RPOT_CUTOFF -> A1M_RPOT_CUTOFF
Connections:
- net GND: no longer U1.12 (+)
- net at U1.9 (-): now also C7.1, U1.8, RV1.1
- net at C6.2: now also U1.6 (-), U1.7, RV1.3
- net at U1.13 (-): now also C10.1, U1.14
- new net: RV1.2, U1.12 (+)
Other:
- note added: "Parallel 1st order HP and LP VCF with adjustable cutoff. f0 = (Ra*gm)/((R+Ra)*2*pi*C) where gm ~= 19.2*Iabc R,RA chosen so ~= 1 2mA Iabc => f0 ~= 20KHz 4.5uA Iabc => f0 ~= 45Hz DC blocking caps on analog boundaries because of difference in ground reference."
- note added: "op-amp input impedance op-amp output impedance (20mA @ 0.5V?)"
- note removed: "Parallel 1st order HP and LP VCF with adjustable cutoff. f0 = (Ra*gm)/((R+Ra)*2*pi*C) where gm ~= 19.2*Iabc R,RA chosen so ~= 1. with 1.5nF: 2mA Iabc => f0 ~= 9KHz 2uA Iabc => f0 ~= 9Hz DC blocking caps on analog boundaries because of difference in ground reference."
- note removed: "input impedance: >=100K op-amp output impedance (20mA @ 0.5V?)"
- moved on the sheet: C10, C6, C7, U1D

Commit message: new ribbon cable
Parts:
- J8, J9: footprint kicad-official/Connector_PinHeader_2.54mm.pretty:PinHeader_1x08_P2.54mm_Vertical -> kicad-official/Connector_PinHeader_1.00mm.pretty:PinHeader_1x08_P1.00mm_Vertical
Connections:
- net INR: now also J8.1 (Pin_1); no longer J8.2 (Pin_2)
- net INR_B: now also J9.1 (Pin_1); no longer J9.2 (Pin_2)
- net LED: now also J8.2 (Pin_2); no longer J8.1 (Pin_1)
- net LED_B: now also J9.2 (Pin_2); no longer J9.1 (Pin_1)
Other:
- note added: "$ 1 0.000005 4.43302224444953 45 5 43 5e-11 a 128 144 240 144 8 15 -15 1000000 -0.25121916034945285 -0.2512216725410563 100000 a 128 256 240 256 8 15 -15 1000000 -4.632465387707845 -4.6325117123617225 100000 a 400 176 496 176 8 15 -15 1000000 -0.8369834111131588 -0.8369917809472699 100000 174 320 160 352 224 1 10000 0.1337 Resistance w 320 224 320 256 0 w 320 256 240 256 0 w 240 144 320 144 0 w 3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"
- note removed: "pot: full clockwise -> short 1-2"
Changed lines of the file:
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@@
+    (effects (font (size 1.27 1.27)) (justify left bottom))
+  )
+  (text "$ 1 0.000005 4.43302224444953 45 5 43 5e-11\na 128 144 240 144 8 15 -15 1000000 -0.25121916034945285 -0.2512216725410563 100000\na 128 256 240 256 8 15 -15 1000000 -4.632465387707845 -4.6325117123617225 100000\na 400 176 496 176 8 15 -15 1000000 -0.8369834111131588 -0.8369917809472699 100000\n174 320 160 352 224 1 10000 0.1337 Resistance\nw 320 224 320 256 0\nw 320 256 240 256 0\nw 240 144 320 144 0\nw 320 144 320 160 0\nw 128 128 128 96 0\nw 128 96 240 96 0\nw 240 96 240 144 0\nw 128 240 128 208 0\nw 128 208 240 208 0\nw 240 208 240 256 0\nw 400 192 352 192 0\nw 400 160 400 128 0\nw 400 128 496 128 0\nw 496 128 496 176 0\n207 496 176 528 176 4 out\nR 128 160 64 160 0 1 440 5 0 0 0.5\nR 128 272 64 272 0 1 1500 5 0 0 0.5\no 18 16 0 5122 5 0.1 0 2 18 3\n"
+    (at 302.26 241.3 0)
     (effects (font (size 1.27 1.27)) (justify left bottom))
   )
@@
     (effects (font (size 1.27 1.27)) (justify left bottom))
   )
-  (text "pot: full clockwise -> short 1-2" (at 154.94 -5.08 0)
-    (effects (font (size 1.27 1.27)) (justify left bottom))
-  )
   (text "op-amp input impedance\nop-amp output impedance (20mA @ 0.5V?)"
     (at 240.03 105.41 0)
@@
     (effects (font (size 1.27 1.27)) (justify left bottom))
   )
-  (label "LED_B" (at 270.51 139.7 0)
+  (label "LED_B" (at 270.51 142.24 0)
     (effects (font (size 1.27 1.27)) (justify left bottom))
   )
@@
     (effects (font (size 1.27 1.27)) (justify left bottom))
   )
-  (label "INR" (at 251.46 142.24 180)
+  (label "INR" (at 251.46 139.7 180)
     (effects (font (size 1.27 1.27)) (justify right bottom))
   )
@@
     (effects (font (size 1.27 1.27)) (justify left bottom))
   )
-  (label "LED" (at 251.46 139.7 180)
+  (label "LED" (at 251.46 142.24 180)
     (effects (font (size 1.27 1.27)) (justify right bottom))
   )
@@
     (effects (font (size 1.27 1.27)) (justify right bottom))
   )
-  (label "INR_B" (at 270.51 142.24 0)
+  (label "INR_B" (at 270.51 139.7 0)
     (effects (font (size 1.27 1.27)) (justify left bottom))
   )
@@
       (effects (font (size 1.27 1.27)) (justify left))
     )
-    (property "Footprint" "kicad-official/Connector_PinHeader_2.54mm.pretty:PinHeader_1x08_P2.54mm_Vertical" (id 2) (at 259.08 147.32 0)
+    (property "Footprint" "kicad-official/Connector_PinHeader_1.00mm.pretty:PinHeader_1x08_P1.00mm_Vertical" (id 2) (at 259.08 147.32 0)
       (effects (font (size 1.27 1.27)) hide)
     )
@@
       (effects (font (size 1.27 1.27)) (justify left))
     )
-    (property "Footprint" "kicad-official/Connector_PinHeader_2.54mm.pretty:PinHeader_1x08_P2.54mm_Vertical" (id 2) (at 262.89 147.32 0)
+    (property "Footprint" "kicad-official/Connector_PinHeader_1.00mm.pretty:PinHeader_1x08_P1.00mm_Vertical" (id 2) (at 262.89 147.32 0)
       (effects (font (size 1.27 1.27)) hide)
     )
@@
     )
     (path "/79db6451-6a70-445a-acbf-38bc9701ab57"
-      (reference "J8") (unit 1) (value "Conn_01x08") (footprint "kicad-official/Connector_PinHeader_2.54mm.pretty:PinHeader_1x08_P2.54mm_Vertical")
+      (reference "J8") (unit 1) (value "Conn_01x08") (footprint "kicad-official/Connector_PinHeader_1.00mm.pretty:PinHeader_1x08_P1.00mm_Vertical")
     )
     (path "/c79d681c-f44c-4d1b-9ea8-c239ce5ca323"
-      (reference "J9") (unit 1) (value "Conn_01x08") (footprint "kicad-official/Connector_PinHeader_2.54mm.pretty:PinHeader_1x08_P2.54mm_Vertical")
+      (reference "J9") (unit 1) (value "Conn_01x08") (footprint "kicad-official/Connector_PinHeader_1.00mm.pretty:PinHeader_1x08_P1.00mm_Vertical")
     )
     (path "/75f534ea-57ee-49ff-9960-6d48d840c311"

Commit message: cleanup
Other:
- note added: "voltage divider from ~2.6Vpp to 26mVpp"
- note removed: "voltage divider from ~2.6Vpp to 26mVpp (TODO confirm ranges)"
- company: (none) -> RabidAudio
- title: (none) -> Amoeba
Changed lines of the file:
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@@
 (kicad_sch (version 20211123) (generator eeschema)
   (paper "A4")
+  (title_block
+    (title "Amoeba")
+    (date "2024-09-16")
+    (rev "F")
+    (company "RabidAudio")
+    (comment 1 "Analog Tone Splitter")
+  )
   (junction (at 171.45 26.67) (diameter 0) (color 0 0 0 0)
   )
@@
     (effects (font (size 1.27 1.27)) (justify left bottom))
   )
-  (text "voltage divider from\n~2.6Vpp to 26mVpp\n(TODO confirm ranges)"
-    (at 83.82 41.91 180)
+  (text "voltage divider from\n~2.6Vpp to 26mVpp" (at 83.82 41.91 180)
     (effects (font (size 1.27 1.27)) (justify right bottom))
   )

Commit message: re-annotate
Parts:
- renumbered C2 to C1, C9 to C10, C3 to C2, C1 to C3, C10 to C8, C8 to C9, R2 to R1, R11 to R10, R14 to R11, R4 to R2, R5 to R4, R6 to R5, R7 to R6, R8 to R7, R9 to R8, R10 to R9, RV2 to RV1, RV1 to RV2
Other:
- note added: "Adjust R11 for brightness red, blue: 10K yellow: 1K white, green: 33K"
- note removed: "Adjust R7 for brightness red, blue: 10K yellow: 1K white, green: 33K"
- moved on the sheet: C10, C11, C12, C9, D1, J4, R11, SW1A, U1E, U2E, U3
