File: splitter/splitter/splitter.kicad_sch (KiCad schematic)
At the start: 39 parts, among them J1 JACKIN, J2 JACKSEND, J3 JACKSEND2, J4 JACKRECV, J5 JACKRECV2, J6 JACKOUT, J7 Jack-DC, J8 Conn_01x08, J9 Conn_01x08, SW1 SW_BYPASS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

Commit message: switch to IPC cables for switch
Parts:
- J8: footprint kicad-official/Connector_PinSocket_2.54mm.pretty:PinSocket_2x04_P2.54mm_Vertical -> kicad-official/Connector_IDC.pretty:IDC-Header_2x04_P2.54mm_Horizontal
- J9: footprint kicad-official/Connector_PinHeader_2.54mm.pretty:PinHeader_2x04_P2.54mm_Vertical -> kicad-official/Connector_IDC.pretty:IDC-Header_2x04_P2.54mm_Vertical
Changed lines of the file:
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@@
       (effects (font (size 1.27 1.27)) (justify left))
     )
-    (property "Footprint" "kicad-official/Connector_PinSocket_2.54mm.pretty:PinSocket_2x04_P2.54mm_Vertical" (id 2) (at 241.3 143.51 0)
+    (property "Footprint" "kicad-official/Connector_IDC.pretty:IDC-Header_2x04_P2.54mm_Horizontal" (id 2) (at 241.3 143.51 0)
       (effects (font (size 1.27 1.27)) hide)
     )
@@
       (effects (font (size 1.27 1.27)) (justify left))
     )
-    (property "Footprint" "kicad-official/Connector_PinHeader_2.54mm.pretty:PinHeader_2x04_P2.54mm_Vertical" (id 2) (at 246.38 143.51 0)
+    (property "Footprint" "kicad-official/Connector_IDC.pretty:IDC-Header_2x04_P2.54mm_Vertical" (id 2) (at 246.38 143.51 0)
       (effects (font (size 1.27 1.27)) hide)
     )
@@
     )
     (path "/79db6451-6a70-445a-acbf-38bc9701ab57"
-      (reference "J8") (unit 1) (value "Conn_01x08") (footprint "kicad-official/Connector_PinSocket_2.54mm.pretty:PinSocket_2x04_P2.54mm_Vertical")
+      (reference "J8") (unit 1) (value "Conn_01x08") (footprint "kicad-official/Connector_IDC.pretty:IDC-Header_2x04_P2.54mm_Horizontal")
     )
     (path "/c79d681c-f44c-4d1b-9ea8-c239ce5ca323"
-      (reference "J9") (unit 1) (value "Conn_01x08") (footprint "kicad-official/Connector_PinHeader_2.54mm.pretty:PinHeader_2x04_P2.54mm_Vertical")
+      (reference "J9") (unit 1) (value "Conn_01x08") (footprint "kicad-official/Connector_IDC.pretty:IDC-Header_2x04_P2.54mm_Vertical")
     )
     (path "/75f534ea-57ee-49ff-9960-6d48d840c311"

Commit message: update input buffer
Parts:
- added R11, R12: 1M, Resistor_THT:R_Axial_DIN0207_L6.3mm_D2.5mm_P7.62mm_Horizontal, symbol Device:R
- C1, C4, C5, C6, C7, C8: value 100n -> 10u; footprint kicad-official/Capacitor_THT.pretty:C_Rect_L7.0mm_W2.5mm_P5.00mm -> Capacitor_SMD:C_0805_2012Metric
- C10, C9: footprint kicad-official/Capacitor_THT.pretty:CP_Radial_D4.0mm_P1.50mm -> Capacitor_SMD:C_0805_2012Metric
- C2, C3: footprint kicad-official/Capacitor_THT.pretty:C_Rect_L7.0mm_W2.5mm_P5.00mm -> Capacitor_THT:C_Rect_L7.0mm_W2.5mm_P5.00mm
- D1: footprint kicad-official/LED_THT.pretty:LED_D3.0mm -> LED_THT:LED_D3.0mm
- J1, J2, J3, J4, J5, J6: footprint kicad-legacy/kicad-footprints/Connector_Audio.pretty:Jack_6.35mm_Neutrik_NMJ6HFD2_Horizontal -> Connector_Audio:Jack_6.35mm_Neutrik_NMJ6HFD2_Horizontal; symbol Connector:AudioJack3_Switch -> Connector_Audio:AudioJack3_Switch
- R1, R10, R2, R3, R4, R5, R6, R7, R8, R9: footprint kicad-official/Resistor_THT.pretty:R_Axial_DIN0207_L6.3mm_D2.5mm_P7.62mm_Horizontal -> Resistor_THT:R_Axial_DIN0207_L6.3mm_D2.5mm_P7.62mm_Horizontal
- RV1: footprint kicad-official/Potentiometer_THT.pretty:Potentiometer_Alpha_RD902F-40-00D_Dual_Vertical -> Potentiometer_THT:Potentiometer_Alpha_RD902F-40-00D_Dual_Vertical
- RV2: footprint kicad-official/Potentiometer_THT.pretty:Potentiometer_Alpha_RD901F-40-00D_Single_Vertical -> Potentiometer_THT:Potentiometer_Alpha_RD901F-40-00D_Single_Vertical
Connections:
- net GND: now also U1.5 (+)
- net at C2.2, U1.7: now also U1.12 (+), R12.1; no longer U1.6 (-)
- new net: R11.1, R12.2, U1.6 (-)
- new net: C1.1, R11.2
Other:
- note added: "1M input impedance op-amp output impedance (20mA @ 0.5V?)"
- note removed: "op-amp input impedance (>1Mohm) op-amp output impedance (20mA @ 0.5V?)"
- moved on the sheet: C1, J2, J3, J4, J5, JP1, JP2, SW1B

Commit message: redesign board: rev F
Parts:
- C2, C3: footprint Capacitor_THT:C_Rect_L7.0mm_W2.5mm_P5.00mm -> Capacitor_SMD:C_0805_2012Metric
- J7: footprint kicad-official/Connector_PinSocket_2.54mm.pretty:PinSocket_1x02_P2.54mm_Vertical -> Connector_PinSocket_2.54mm:PinSocket_1x02_P2.54mm_Vertical
- J8: footprint kicad-official/Connector_IDC.pretty:IDC-Header_2x04_P2.54mm_Horizontal -> Connector_IDC:IDC-Header_2x04_P2.54mm_Vertical
- J9: footprint kicad-official/Connector_IDC.pretty:IDC-Header_2x04_P2.54mm_Vertical -> Connector_IDC:IDC-Header_2x04_P2.54mm_Vertical
- JP1, JP3: footprint kicad-official/Jumper.pretty:SolderJumper-3_P1.3mm_Open_RoundedPad1.0x1.5mm -> Jumper:SolderJumper-3_P1.3mm_Open_RoundedPad1.0x1.5mm
- JP2: footprint kicad-official/Jumper.pretty:SolderJumper-2_P1.3mm_Open_RoundedPad1.0x1.5mm -> Jumper:SolderJumper-2_P1.3mm_Open_RoundedPad1.0x1.5mm
- R1, R10, R11, R12, R2, R3, R4, R5, R6, R8, R9: footprint Resistor_THT:R_Axial_DIN0207_L6.3mm_D2.5mm_P7.62mm_Horizontal -> Resistor_SMD:R_0805_2012Metric
- R7: value 10K -> 100K; footprint Resistor_THT:R_Axial_DIN0207_L6.3mm_D2.5mm_P7.62mm_Horizontal -> Resistor_SMD:R_0805_2012Metric
- U1: footprint kicad-official/Package_DIP.pretty:DIP-14_W7.62mm_Socket -> Package_DIP:DIP-14_W7.62mm_Socket
- U2: footprint kicad-official/Package_TO_SOT_THT.pretty:TO-92_Inline_Wide -> Package_TO_SOT_THT:TO-92_Inline_Wide
Changed lines of the file:
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@@
 			)
 		)
-		(property "Footprint" "kicad-official/Package_DIP.pretty:DIP-14_W7.62mm_Socket"
+		(property "Footprint" "Package_DIP:DIP-14_W7.62mm_Socket"
 			(at 102.87 48.26 0)
 			(effects
@@
 			)
 		)
-		(property "Footprint" "Capacitor_THT:C_Rect_L7.0mm_W2.5mm_P5.00mm"
+		(property "Footprint" "Capacitor_SMD:C_0805_2012Metric"
 			(at 64.77 49.2252 0)
 			(effects
@@
 			)
 		)
-		(property "Footprint" "Capacitor_THT:C_Rect_L7.0mm_W2.5mm_P5.00mm"
+		(property "Footprint" "Capacitor_SMD:C_0805_2012Metric"
 			(at 77.47 49.2252 0)
 			(effects
@@
 			)
 		)
-		(property "Footprint" "kicad-official/Package_DIP.pretty:DIP-14_W7.62mm_Socket"
+		(property "Footprint" "Package_DIP:DIP-14_W7.62mm_Socket"
 			(at 50.8 50.8 0)
 			(effects
@@
 			)
 		)
-		(property "Footprint" "Resistor_THT:R_Axial_DIN0207_L6.3mm_D2.5mm_P7.62mm_Horizontal"
+		(property "Footprint" "Resistor_SMD:R_0805_2012Metric"
 			(at 90.678 58.42 90)
 			(effects
@@
 			)
 		)
-		(property "Footprint" "Resistor_THT:R_Axial_DIN0207_L6.3mm_D2.5mm_P7.62mm_Horizontal"
+		(property "Footprint" "Resistor_SMD:R_0805_2012Metric"
 			(at 80.01 31.242 90)
 			(effects
@@
 			)
 		)
-		(property "Footprint" "kicad-official/Package_DIP.pretty:DIP-14_W7.62mm_Socket"
+		(property "Footprint" "Package_DIP:DIP-14_W7.62mm_Socket"
 			(at 251.46 102.87 0)
 			(effects
@@
 			)
 		)
-		(property "Footprint" "Resistor_THT:R_Axial_DIN0207_L6.3mm_D2.5mm_P7.62mm_Horizontal"
+		(property "Footprint" "Resistor_SMD:R_0805_2012Metric"
 			(at 124.46 65.532 90)
 			(effects
@@
 			)
 		)
-		(property "Footprint" "Resistor_THT:R_Axial_DIN0207_L6.3mm_D2.5mm_P7.62mm_Horizontal"
+		(property "Footprint" "Resistor_SMD:R_0805_2012Metric"
 			(at 140.97 55.372 90)
 			(effects
@@
 			)
 		)
-		(property "Footprint" "kicad-official/Package_DIP.pretty:DIP-14_W7.62mm_Socket"
+		(property "Footprint" "Package_DIP:DIP-14_W7.62mm_Socket"
 			(at 264.16 27.94 0)
 			(effects
@@
 			)
 		)
-		(property "Footprint" "kicad-official/Package_DIP.pretty:DIP-14_W7.62mm_Socket"
+		(property "Footprint" "Package_DIP:DIP-14_W7.62mm_Socket"
 			(at 139.7 72.39 0)
 			(effects
@@
 			)
 		)
-		(property "Footprint" "Resistor_THT:R_Axial_DIN0207_L6.3mm_D2.5mm_P7.62mm_Horizontal"
+		(property "Footprint" "Resistor_SMD:R_0805_2012Metric"
 			(at 215.9 102.362 90)
 			(effects
@@
 			)
 		)
-		(property "Footprint" "Resistor_THT:R_Axial_DIN0207_L6.3mm_D2.5mm_P7.62mm_Horizontal"
+		(property "Footprint" "Resistor_SMD:R_0805_2012Metric"
 			(at 215.9 94.488 90)
 			(effects
@@
 			)
 		)
-		(property "Footprint" "kicad-official/Package_TO_SOT_THT.pretty:TO-92_Inline_Wide"
+		(property "Footprint" "Package_TO_SOT_THT:TO-92_Inline_Wide"
 			(at 238.76 34.29 0)
 			(effects
@@
 			)
 		)
-		(property "Value" "10K"
+		(property "Value" "100K"
 			(at 218.948 41.783 0)
 			(effects
@@
 			)
 		)
-		(property "Footprint" "Resistor_THT:R_Axial_DIN0207_L6.3mm_D2.5mm_P7.62mm_Horizontal"
+		(property "Footprint" "Resistor_SMD:R_0805_2012Metric"
 			(at 215.392 40.64 90)
 			(effects
@@
 			)
 		)
-		(property "Footprint" "kicad-official/Connector_PinSocket_2.54mm.pretty:PinSocket_1x02_P2.54mm_Vertical"
+		(property "Footprint" "Connector_PinSocket_2.54mm:PinSocket_1x02_P2.54mm_Vertical"
 			(at 177.8 30.226 0)
 			(effects
@@
 			)
 		)
-		(property "Footprint" "kicad-official/Jumper.pretty:SolderJumper-2_P1.3mm_Open_RoundedPad1.0x1.5mm"
+		(property "Footprint" "Jumper:SolderJumper-2_P1.3mm_Open_RoundedPad1.0x1.5mm"
 			(at 78.74 187.96 0)
 			(effects
@@
 			)
 		)
-		(property "Footprint" "Resistor_THT:R_Axial_DIN0207_L6.3mm_D2.5mm_P7.62mm_Horizontal"
+		(property "Footprint" "Resistor_SMD:R_0805_2012Metric"
 			(at 255.27 94.488 90)
 			(effects
@@
 			)
 		)
-		(property "Footprint" "Resistor_THT:R_Axial_DIN0207_L6.3mm_D2.5mm_P7.62mm_Horizontal"
+		(property "Footprint" "Resistor_SMD:R_0805_2012Metric"
 			(at 34.29 43.942 90)
 			(effects
@@
 			)
 		)
-		(property "Footprint" "kicad-official/Jumper.pretty:SolderJumper-3_P1.3mm_Open_RoundedPad1.0x1.5mm"
+		(property "Footprint" "Jumper:SolderJumper-3_P1.3mm_Open_RoundedPad1.0x1.5mm"
 			(at 46.99 116.84 0)
 			(effects
@@
 			)
 		)
-		(property "Footprint" "kicad-official/Connector_IDC.pretty:IDC-Header_2x04_P2.54mm_Horizontal"
+		(property "Footprint" "Connector_IDC:IDC-Header_2x04_P2.54mm_Vertical"
 			(at 241.3 143.51 0)
 			(effects
@@
 			)
 		)
-		(property "Footprint" "Resistor_THT:R_Axial_DIN0207_L6.3mm_D2.5mm_P7.62mm_Horizontal"
+		(property "Footprint" "Resistor_SMD:R_0805_2012Metric"
 			(at 232.41 94.488 90)
 			(effects
@@
 			)
 		)
-		(property "Footprint" "Resistor_THT:R_Axial_DIN0207_L6.3mm_D2.5mm_P7.62mm_Horizontal"
+		(property "Footprint" "Resistor_SMD:R_0805_2012Metric"
 			(at 50.8 38.862 90)
 			(effects
@@
 			)
 		)
-		(property "Footprint" "kicad-official/Jumper.pretty:SolderJumper-3_P1.3mm_Open_RoundedPad1.0x1.5mm"
+		(property "Footprint" "Jumper:SolderJumper-3_P1.3mm_Open_RoundedPad1.0x1.5mm"
 			(at 113.03 116.84 0)
 			(effects
@@
 			)
 		)
-		(property "Footprint" "kicad-official/Connector_IDC.pretty:IDC-Header_2x04_P2.54mm_Vertical"
+		(property "Footprint" "Connector_IDC:IDC-Header_2x04_P2.54mm_Vertical"
 			(at 246.38 143.51 0)
 			(effects
@@
 			)
 		)
-		(property "Footprint" "Resistor_THT:R_Axial_DIN0207_L6.3mm_D2.5mm_P7.62mm_Horizontal"
+		(property "Footprint" "Resistor_SMD:R_0805_2012Metric"
 			(at 232.41 105.918 90)
 			(effects
