File: splitter/splitter/splitter.kicad_sch (KiCad schematic)
At the start: 41 parts, among them J1 JACKIN, J2 JACKSEND, J3 JACKSEND2, J4 JACKRECV, J5 JACKRECV2, J6 JACKOUT, J7 Jack-DC, J8 Conn_01x08, J9 Conn_01x08, SW1 SW_BYPASS, SW2 SW_MODE, U1 TL074, U2 TLE2426xLP

Commit message: unsaved changes
Changed lines of the file:
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@@
 (kicad_sch
-	(version 20231120)
+	(version 20250114)
 	(generator "eeschema")
-	(generator_version "8.0")
+	(generator_version "9.0")
 	(paper "A4")
+	(text "Modes:\nMono in/out/send/recv: all jumpers open\nStereo in/send/recv/out, right channel switched but not filtered:\n  JP1=closed, JP2+JP3=1:2\nStereo in/out (right pass through), mono send/recv1 (\"wet\") and separate send/recv2 (\"dry\"):\n  JP1=open, JP2+JP3=1:2, send2+recv2 jacks populated\nMono in/out, stereo send/recv (right channel \"dry\"):\n  JP1=closed, JP2+JP3=2:3"
+		(exclude_from_sim no)
+		(at 119.38 171.45 0)
+		(effects
+			(font
+				(size 1.27 1.27)
+			)
+			(justify left bottom)
+		)
+	)
+	(text "Optional, if you want two send-receive channels.\nIf not, tie the jumper closed and leave the jacks unpopulated"
+		(exclude_from_sim no)
+		(at 55.245 193.675 0)
+		(effects
+			(font
+				(size 1.27 1.27)
+			)
+			(justify left bottom)
+		)
+	)
+	(text "Adjust R7 for brightness\nred, blue: 10K\nyellow: 1K\nwhite, green: 33K"
+		(exclude_from_sim no)
+		(at 222.25 52.705 0)
+		(effects
+			(font
+				(size 1.27 1.27)
+			)
+			(justify left bottom)
+		)
+	)
+	(text "power led"
+		(exclude_from_sim no)
+		(at 212.725 57.785 0)
+		(effects
+			(font
+				(size 1.27 1.27)
+			)
+			(justify left bottom)
+		)
+	)
+	(text "power filter caps, close to IC"
+		(exclude_from_sim no)
+		(at 255.27 52.07 0)
+		(effects
+			(font
+				(size 1.27 1.27)
+			)
+			(justify left bottom)
+		)
+	)
+	(text "input impedance: >=100K\nop-amp output impedance (20mA @ 0.5V?)"
+		(exclude_from_sim no)
+		(at 221.615 118.745 0)
+		(effects
+			(font
+				(size 1.27 1.27)
+			)
+			(justify left bottom)
+		)
+	)
+	(text "1M input impedance\nop-amp output impedance (20mA @ 0.5V?)"
+		(exclude_from_sim no)
+		(at 40.005 88.9 0)
+		(effects
+			(font
+				(size 1.27 1.27)
+			)
+			(justify left bottom)
+		)
+	)
+	(text "6.8n, 1K -> 23.4Hz, Q=0.5\n6.8n, 1001K -> 23.4KHz, Q=0.5\nNote: subtracting instead of creating separate LP and HP\nfilters creates an uneven split as opposed to summing LR\nfilters. Creating a true crossover would require VCFs,\nwhich would be more complicated.\n\nDC blocking caps on analog boundaries because of difference\nin ground reference."
+		(exclude_from_sim no)
+		(at 15.24 34.29 0)
+		(effects
+			(font
+				(size 1.27 1.27)
+			)
+			(justify left bottom)
+		)
+	)
+	(text "Stereo jumpers control the behavior of the ring\nchannel (if stereo cables are used).\n1::2 - true bypass of signal on or off, no effect\n2::3 - dry signal on send/receive ring channel"
+		(exclude_from_sim no)
+		(at 54.61 111.125 0)
+		(effects
+			(font
+				(size 1.27 1.27)
+			)
+			(justify left bottom)
+		)
+	)
+	(text "9V ac/dc center negative\ncould also be 9V battery"
+		(exclude_from_sim no)
+		(at 167.64 43.18 0)
+		(effects
+			(font
+				(size 1.27 1.27)
+			)
+			(justify left bottom)
+		)
+	)
+	(text "Bypass switch board interconnect"
+		(exclude_from_sim no)
+		(at 229.87 157.48 0)
+		(effects
+			(font
+				(size 1.27 1.27)
+			)
+			(justify left bottom)
+		)
+	)
+	(text "Even though our analog reference is 4.5V,\nother pedals will use the power supply ground (0V)\nas their ground. So we need to use GNDD for the\njack grounds"
+		(exclude_from_sim no)
+		(at 14.605 160.655 0)
+		(effects
+			(font
+				(size 1.27 1.27)
+			)
+			(justify left bottom)
+		)
+	)
 	(junction
 		(at 130.81 67.31)
@@
 		)
 	)
-	(text "Modes:\nMono in/out/send/recv: all jumpers open\nStereo in/send/recv/out, right channel switched but not filtered:\n  JP1=closed, JP2+JP3=1:2\nStereo in/out (right pass through), mono send/recv1 (\"wet\") and separate send/recv2 (\"dry\"):\n  JP1=open, JP2+JP3=1:2, send2+recv2 jacks populated\nMono in/out, stereo send/recv (right channel \"dry\"):\n  JP1=closed, JP2+JP3=2:3"
-		(exclude_from_sim no)
-		(at 119.38 171.45 0)
-		(effects
-			(font
-				(size 1.27 1.27)
-			)
-			(justify left bottom)
-		)
-	)
-	(text "Optional, if you want two send-receive channels.\nIf not, tie the jumper closed and leave the jacks unpopulated"
-		(exclude_from_sim no)
-		(at 55.245 193.675 0)
-		(effects
-			(font
-				(size 1.27 1.27)
-			)
-			(justify left bottom)
-		)
-	)
-	(text "Adjust R7 for brightness\nred, blue: 10K\nyellow: 1K\nwhite, green: 33K"
-		(exclude_from_sim no)
-		(at 222.25 52.705 0)
-		(effects
-			(font
-				(size 1.27 1.27)
-			)
-			(justify left bottom)
-		)
-	)
-	(text "power led"
-		(exclude_from_sim no)
-		(at 212.725 57.785 0)
-		(effects
-			(font
-				(size 1.27 1.27)
-			)
-			(justify left bottom)
-		)
-	)
-	(text "power filter caps, close to IC"
-		(exclude_from_sim no)
-		(at 255.27 52.07 0)
-		(effects
-			(font
-				(size 1.27 1.27)
-			)
-			(justify left bottom)
-		)
-	)
-	(text "input impedance: >=100K\nop-amp output impedance (20mA @ 0.5V?)"
-		(exclude_from_sim no)
-		(at 221.615 118.745 0)
-		(effects
-			(font
-				(size 1.27 1.27)
-			)
-			(justify left bottom)
-		)
-	)
-	(text "1M input impedance\nop-amp output impedance (20mA @ 0.5V?)"
-		(exclude_from_sim no)
-		(at 40.005 88.9 0)
-		(effects
-			(font
-				(size 1.27 1.27)
-			)
-			(justify left bottom)
-		)
-	)
-	(text "6.8n, 1K -> 23.4Hz, Q=0.5\n6.8n, 1001K -> 23.4KHz, Q=0.5\nNote: subtracting instead of creating separate LP and HP\nfilters creates an uneven split as opposed to summing LR\nfilters. Creating a true crossover would require VCFs,\nwhich would be more complicated.\n\nDC blocking caps on analog boundaries because of difference\nin ground reference."
-		(exclude_from_sim no)
-		(at 15.24 34.29 0)
-		(effects
-			(font
-				(size 1.27 1.27)
-			)
-			(justify left bottom)
-		)
-	)
-	(text "Stereo jumpers control the behavior of the ring\nchannel (if stereo cables are used).\n1::2 - true bypass of signal on or off, no effect\n2::3 - dry signal on send/receive ring channel"
-		(exclude_from_sim no)
-		(at 54.61 111.125 0)
-		(effects
-			(font
-				(size 1.27 1.27)
-			)
-			(justify left bottom)
-		)
-	)
-	(text "9V ac/dc center negative\ncould also be 9V battery"
-		(exclude_from_sim no)
-		(at 167.64 43.18 0)
-		(effects
-			(font
-				(size 1.27 1.27)
-			)
-			(justify left bottom)
-		)
-	)
-	(text "Bypass switch board interconnect"
-		(exclude_from_sim no)
-		(at 229.87 157.48 0)
-		(effects
-			(font
-				(size 1.27 1.27)
-			)
-			(justify left bottom)
-		)
-	)
-	(text "Even though our analog reference is 4.5V,\nother pedals will use the power supply ground (0V)\nas their ground. So we need to use GNDD for the\njack grounds"
-		(exclude_from_sim no)
-		(at 14.605 160.655 0)
-		(effects
-			(font
-				(size 1.27 1.27)
-			)
-			(justify left bottom)
-		)
-	)
 	(label "9V_B"
 		(at 254 135.89 0)
@@
 		)
 	)
+	(embedded_fonts no)
 )
