File: dist/dynafuzz/dynafuzz.kicad_pcb (KiCad board)
At the start: 2 copper layers, 54 parts, among them J1 AudioJack3_Switch, J2 AudioJack3_Switch, J3 Jack-DC, Q1 Q_NPN, Q2 Q_NPN, Q3 Q_NPN, Q4 Q_NPN, SW1 SW_3PDT_x3

Commit message: update silkscreen
Parts:
- C1, C10, C11, C12, C13, C2, C3, C4, C5, C6, C7, C8, C9: footprint Capacitor_THT:C_Rect_L7.0mm_W2.5mm_P5.00mm -> _project:C
- R1, R10, R11, R12, R13, R14, R15, R16, R17, R18, R19, R2, R20, R21, R22, R23, R3, R4, R5, R6, R7, R8, R9: footprint Resistor_THT:R_Axial_DIN0207_L6.3mm_D2.5mm_P2.54mm_Vertical -> _project:R

Commit message: layout stage 2 and 3
Parts:
- J1: value AudioJack3_Switch -> AudioJack_IN
- J2: value AudioJack3_Switch -> AudioJack_OUT
- J3: moved to B.Cu
- moved Q4 165.4 mm to (115.1, 86.0)
- moved R23 158.4 mm to (112.3, 81.5), turned to 90 degrees
- moved C10 155.1 mm to (109.7, 60.0)
- moved C11 155.1 mm to (109.7, 64.0)
- moved C12 155.1 mm to (109.7, 68.1)
- moved R21 154.6 mm to (111.5, 87.1), turned to 90 degrees
- moved R20 150.5 mm to (116.3, 81.5), turned to 90 degrees
- moved R19 150.1 mm to (121.6, 64.3), turned to 180 degrees
- moved R22 149.8 mm to (120.7, 79.5), turned to -90 degrees
- moved R17 148.7 mm to (121.6, 59.9), turned to 180 degrees
- moved C13 139.0 mm to (124.5, 86.8), turned to 90 degrees
- moved Q3 129.8 mm to (157.5, 69.3), turned to 90 degrees
- moved Q2 122.3 mm to (163.1, 69.3), turned to 90 degrees
- moved R15 117.1 mm to (157.5, 63.0), turned to 90 degrees
- moved R16 115.6 mm to (151.9, 76.7), turned to 180 degrees
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Connections:
- J1 pad T: Net-(SW1A-B) -> Net-(SW1C-B)
- J2 pad T: Net-(SW1B-B) -> Net-(SW1A-B)
- R1 pad 1: IN -> Net-(C1-Pad1)
- R1 pad 2: Net-(C1-Pad1) -> IN
- R10 pad 1: +9V -> Net-(D1-A)
- R10 pad 2: Net-(D1-A) -> +9V
- R15 pad 1: +9V -> Net-(D3-A)
- R15 pad 2: Net-(D3-A) -> +9V
- SW1 pad 1: IN -> OUT
- SW1 pad 4: OUT -> +9V
- SW1 pad 5: Net-(SW1B-B) -> Net-(D5-A)
- SW1 pad 6: Net-(SW1A-C) -> unconnected-(SW1B-C-Pad6)
- SW1 pad 7: +9V -> IN
- SW1 pad 8: Net-(D5-A) -> Net-(SW1C-B)
- SW1 pad 9: unconnected-(SW1C-C-Pad9) -> Net-(SW1A-C)
Routing:
- net +9V: track 0.00 -> 19.0 mm
- net OUT: track 0.00 -> 9.22 mm
- added copper zone on B.Cu, net GND
- added copper zone on F.Cu, net GND
Other:
- board text added: "+"

Commit message: placed components
Parts:
- moved R19 53.3 mm to (170.7, 85.1)
- moved R2 52.0 mm to (158.5, 95.5), turned to 90 degrees
- moved R17 48.5 mm to (163.1, 85.1)
- moved C3 47.2 mm to (179.5, 83.3), turned to 180 degrees
- moved C11 44.6 mm to (146.5, 89.2), turned to 180 degrees
- moved R5 42.3 mm to (177.8, 89.2), turned to 90 degrees
- moved C13 41.0 mm to (148.1, 53.3), turned to 0 degrees
- moved C10 41.0 mm to (141.5, 85.9)
- moved R4 40.5 mm to (174.0, 89.2), turned to 90 degrees
- moved Q1 37.5 mm to (181.1, 88.4), turned to 0 degrees
- moved C12 34.9 mm to (141.5, 82.5)
- moved R3 33.6 mm to (187.5, 89.2)
- moved C2 26.6 mm to (182.9, 83.3)
- moved R21 23.7 mm to (134.9, 83.1), turned to 180 degrees
- moved R23 21.5 mm to (132.3, 89.2)
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Routing:
- net Net-(SW1C-B): track 0.00 -> 23.4 mm
- net Net-(D5-A): track 0.00 -> 20.2 mm
- net Net-(C3-Pad2): track 0.00 -> 18.8 mm
- net Net-(SW1A-C): track 0.00 -> 16.9 mm
- net Net-(R6-Pad1): track 0.00 -> 13.8 mm
- net +9V: track 19.0 -> 5.59 mm
- net Net-(D1-A): track 0.00 -> 13.3 mm
- net Net-(C4-Pad1): track 0.00 -> 9.82 mm
- net Net-(SW1A-B): track 0.00 -> 8.20 mm
- net Net-(D5-K): track 0.00 -> 4.68 mm

Commit message: routed up to tone stack
Parts:
- moved R11 7.11 mm to (168.1, 67.3)
- moved R16 7.11 mm to (151.9, 67.3)
- moved C7 4.06 mm to (148.3, 58.2)
- moved C8 4.06 mm to (152.4, 63.2)
- moved D1 3.56 mm to (170.7, 70.9)
- moved D2 3.56 mm to (168.1, 74.4)
- moved D3 3.56 mm to (149.4, 70.9)
- moved D4 3.56 mm to (151.9, 74.4)
Routing:
- net +9V: track 5.59 -> 67.0 mm
- net Net-(Q1-B): track 0.00 -> 52.5 mm
- net Net-(C10-Pad1): track 0.00 -> 50.3 mm
- net Net-(Q3-B): track 0.00 -> 32.9 mm
- net Net-(Q2-B): track 0.00 -> 32.1 mm
- net Net-(D1-A): track 13.3 -> 44.2 mm
- net Net-(D3-A): track 0.00 -> 25.0 mm
- net Net-(Q1-C): track 0.00 -> 24.4 mm
- net Net-(D3-K): track 0.00 -> 17.4 mm
- net Net-(D1-K): track 0.00 -> 17.4 mm
- net Net-(C7-Pad2): track 0.00 -> 15.8 mm
- net Net-(C4-Pad2): track 0.00 -> 15.8 mm
- net Net-(R19-Pad1): track 0.00 -> 11.0 mm
- net Net-(Q3-E): track 0.00 -> 5.69 mm
- net Net-(Q2-E): track 0.00 -> 5.19 mm
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
Commit message: first pass route
Parts:
- moved R20 27.8 mm to (149.8, 85.1), turned to 0 degrees
- moved R23 23.9 mm to (155.9, 85.1), turned to 0 degrees
- moved R22 18.9 mm to (141.7, 89.7)
- moved R21 11.2 mm to (145.3, 87.1), turned to -90 degrees
- moved Q4 10.2 mm to (144.5, 82.8), turned to 180 degrees
- moved C10 8.92 mm to (133.1, 82.8)
- moved C11 8.92 mm to (138.1, 86.1)
- moved C12 7.65 mm to (138.1, 89.4), turned to 180 degrees
- moved R17 1.50 mm to (164.6, 85.1)
Routing:
- net Net-(Q4-C): track 0.00 -> 36.4 mm
- net Net-(C11-Pad1): track 0.00 -> 31.5 mm
- net OUT: track 9.70 -> 39.8 mm, vias 0 -> 1
- net Net-(D3-A): track 25.0 -> 54.5 mm
- net Net-(C13-Pad2): track 0.00 -> 24.0 mm
- net +9V: track 67.0 -> 86.2 mm
- net Net-(Q4-B): track 0.00 -> 18.6 mm
- net Net-(C12-Pad2): track 0.00 -> 12.8 mm
- net Net-(Q4-E): track 0.00 -> 12.3 mm
- net Net-(C10-Pad1): track 50.3 -> 56.0 mm

Commit message: update positions
Parts:
- RV1, RV2, RV3, RV4: footprint Potentiometer_THT:Potentiometer_Alpha_RD901F-40-00D_Single_Vertical -> _effects_shared_footprints:Potentiometer_Alpha_RD901F-40-00D_Single_Vertical
- moved D1 3.56 mm to (170.7, 74.4)
- moved D2 3.56 mm to (168.1, 70.9)
- moved D3 3.56 mm to (149.4, 74.4)
- moved D4 3.56 mm to (151.9, 70.9)
- moved R1 2.09 mm to (162.6, 93.4), turned to -90 degrees
- moved R10 2.09 mm to (163.1, 58.6), turned to -90 degrees
- moved R15 2.09 mm to (157.5, 58.6), turned to -90 degrees
- moved R18 2.09 mm to (158.5, 102.0), turned to -90 degrees
- moved R2 2.09 mm to (158.5, 93.4), turned to -90 degrees
Connections:
- R1 pad 1: Net-(C1-Pad1) -> IN
- R1 pad 2: IN -> Net-(C1-Pad1)
- R10 pad 1: Net-(D1-A) -> +9V
- R10 pad 2: +9V -> Net-(D1-A)
- R15 pad 1: Net-(D3-A) -> +9V
- R15 pad 2: +9V -> Net-(D3-A)
- R18 pad 1: Net-(D5-K) -> GND
- R18 pad 2: GND -> Net-(D5-K)
- R2 pad 1: Net-(Q1-B) -> GND
- R2 pad 2: GND -> Net-(Q1-B)
Routing:
- net Net-(D3-A): track 54.5 -> 58.5 mm
- net Net-(C10-Pad1): track 56.0 -> 52.9 mm
Other:
- board outline added: 58.4 x 60.2 mm

Commit message: finish layout
Connections:
- RV1 pad 1: Net-(C3-Pad2) -> Net-(R6-Pad1)
- RV1 pad 3: Net-(R6-Pad1) -> Net-(C3-Pad2)
- RV2 pad 1: Net-(R19-Pad1) -> Net-(C10-Pad1)
- RV2 pad 3: Net-(C10-Pad1) -> Net-(R19-Pad1)
- RV3 pad 1: Net-(C10-Pad1) -> Net-(C11-Pad1)
- RV3 pad 3: Net-(C11-Pad1) -> Net-(C10-Pad1)
- RV4 pad 1: Net-(C13-Pad2) -> GND
- RV4 pad 3: GND -> Net-(C13-Pad2)
Routing:
- net Net-(R19-Pad1): track 11.0 -> 14.3 mm
- net Net-(C11-Pad1): track 31.5 -> 34.6 mm
- net OUT: track 39.8 -> 37.4 mm
- net Net-(D1-A): track 44.2 -> 41.9 mm
- net Net-(R6-Pad1): track 18.4 -> 16.1 mm
- net Net-(C12-Pad2): track 12.8 -> 15.1 mm
- net Net-(C13-Pad2): track 24.0 -> 21.9 mm
- net Net-(Q4-C): track 36.4 -> 35.3 mm
- net Net-(C3-Pad2): track 21.7 -> 22.6 mm
- net Net-(D3-A): track 58.5 -> 57.5 mm
- net Net-(Q1-C): track 24.4 -> 23.8 mm
- net Net-(Q3-B): track 32.9 -> 32.3 mm
- net Net-(Q2-B): track 32.1 -> 31.5 mm
Other:
- board size 58.4 x 60.2 mm -> 58.4 x 60.7 mm

Commit message: board interconnect
Parts:
- added J4: MAIN_BIC, Connector_PinSocket_2.54mm:PinSocket_1x06_P2.54mm_Vertical, B.Cu at (166.6, 88.9)
- added J5: SWITCH_BIC, Connector_PinSocket_2.54mm:PinSocket_1x06_P2.54mm_Vertical, B.Cu at (166.4, 115.8)
- SW1: footprint Connector_PinSocket_2.54mm:PinSocket_1x09_P2.54mm_Vertical -> _effects_shared_footprints:Stompbox Switch
- moved SW1 39.7 mm to (160.0, 127.3)
Connections:
- D5 pad 2: Net-(D5-A) -> LED
- J1 pad T: Net-(SW1C-B) -> Net-(J4-Pin_1)
- J2 pad T: Net-(SW1A-B) -> Net-(J4-Pin_5)
- SW1 pad 1: OUT -> Net-(J5-Pin_6)
- SW1 pad 2: Net-(SW1A-B) -> Net-(J5-Pin_5)
- SW1 pad 4: +9V -> Net-(J5-Pin_3)
- SW1 pad 5: Net-(D5-A) -> Net-(J5-Pin_4)
- SW1 pad 7: IN -> Net-(J5-Pin_2)
- SW1 pad 8: Net-(SW1C-B) -> Net-(J5-Pin_1)
Routing:
- net Net-(J4-Pin_1): track 0.00 -> 23.9 mm
- net Net-(SW1C-B): track 23.4 -> 0.00 mm
- net LED: track 0.00 -> 20.5 mm
- net Net-(D5-A): track 20.2 -> 0.00 mm
- net Net-(J5-Pin_1): track 0.00 -> 13.0 mm
- net Net-(J5-Pin_4): track 0.00 -> 12.9 mm
- net Net-(J5-Pin_5): track 0.00 -> 12.8 mm
- net Net-(J4-Pin_5): track 0.00 -> 12.3 mm
- net Net-(SW1A-B): track 8.20 -> 0.00 mm
- net OUT: track 37.4 -> 45.3 mm
- net Net-(J5-Pin_3): track 0.00 -> 7.28 mm
- net Net-(J5-Pin_2): track 0.00 -> 7.24 mm
- net Net-(J5-Pin_6): track 0.00 -> 7.22 mm
- net Net-(SW1A-C): track 16.9 -> 11.7 mm
- net +9V: track 86.0 -> 83.0 mm
Other:
- board size 58.4 x 60.7 mm -> 58.4 x 85.1 mm
