File: dist/dynafuzz/dynafuzz.kicad_pcb (KiCad board)
At the start: 2 copper layers, 58.4 x 85.1 mm, 56 parts, among them J1 AudioJack_IN, J2 AudioJack_OUT, J3 Jack-DC, J4 MAIN_BIC, J5 SWITCH_BIC, Q1 Q_NPN, Q2 Q_NPN, Q3 Q_NPN, Q4 Q_NPN, SW1 SW_3PDT_x3

Commit message: rev A
Parts:
- SW1: moved to F.Cu
- moved C10 5.00 mm to (138.1, 82.8), turned to 180 degrees
- turned SW1 to 90 degrees
Connections:
- SW1 pad 1: Net-(J5-Pin_6) -> Net-(SW1A-A)
- SW1 pad 3: Net-(SW1A-C) -> Net-(J5-Pin_6)
- SW1 pad 4: Net-(J5-Pin_3) -> unconnected-(SW1B-A-Pad4)
- SW1 pad 6: unconnected-(SW1B-C-Pad6) -> Net-(J5-Pin_3)
- SW1 pad 7: Net-(J5-Pin_2) -> Net-(SW1A-A)
- SW1 pad 9: Net-(SW1A-C) -> Net-(J5-Pin_2)
Routing:
- net Net-(SW1A-C): track 11.7 -> 0.00 mm
- net Net-(SW1A-A): track 0.00 -> 11.5 mm
- net Net-(J5-Pin_2): track 7.24 -> 8.98 mm
- net Net-(Q4-C): track 35.3 -> 36.7 mm
- net Net-(C10-Pad1): track 53.3 -> 52.3 mm
- net +9V: track 83.0 -> 83.7 mm
- net Net-(D3-A): track 57.5 -> 58.0 mm
- net Net-(C11-Pad1): track 34.6 -> 35.1 mm
Other:
- board text added: "FUZZ Rev A 2026-08-06"

Commit message: rev B - dynafuzz
Parts:
- added TP1: ~, TestPoint:TestPoint_Pad_D1.5mm, F.Cu at (188.0, 79.8)
- added TP2: ~, TestPoint:TestPoint_Pad_D1.5mm, F.Cu at (168.7, 55.6)
- added TP3: ~, TestPoint:TestPoint_Pad_D1.5mm, F.Cu at (155.2, 56.1)
- added TP4: ~, TestPoint:TestPoint_Pad_D1.5mm, F.Cu at (132.1, 79.0)
- added TP5: ~, TestPoint:TestPoint_Pad_D1.5mm, F.Cu at (132.3, 94.5)
- R18: value 1K -> 3.3k
- R23: value 100 -> 3.3k
- moved J1 3.25 mm to (170.7, 109.7)
- moved J2 3.00 mm to (149.1, 93.5)
Routing:
- net Net-(Q4-C): track 36.7 -> 49.3 mm
- net Net-(C12-Pad2): track 15.1 -> 25.9 mm
- net Net-(D1-A): track 41.9 -> 49.8 mm
- net Net-(D3-A): track 58.0 -> 64.0 mm
- net Net-(Q1-C): track 23.8 -> 27.3 mm
- net Net-(Q1-B): track 52.3 -> 49.2 mm
- net Net-(J4-Pin_5): track 12.3 -> 9.25 mm
- net Net-(J4-Pin_1): track 23.9 -> 22.5 mm
Other:
- board text added: "FUZZ Rev B 2026-08-25"
- board text removed: "FUZZ Rev A 2026-08-06"

Commit message: start layout
Parts:
- added C15: 100n, Capacitor_SMD:C_0805_2012Metric, F.Cu at (160.0, 83.8)
- added C16: 100n, Capacitor_SMD:C_0805_2012Metric, F.Cu at (-101.4, 75.2)
- added C17: 100n, Capacitor_SMD:C_0805_2012Metric, F.Cu at (-101.4, 78.2)
- added C18: 100n, Capacitor_SMD:C_0805_2012Metric, F.Cu at (-87.5, 156.2)
- added C19: 100n, Capacitor_SMD:C_0805_2012Metric, F.Cu at (167.6, 79.2)
- added C20: 100n, Capacitor_SMD:C_0805_2012Metric, F.Cu at (60.4, 33.2)
- added C21: 100n, Capacitor_SMD:C_0805_2012Metric, F.Cu at (60.4, 36.2)
- added C22: 470p, Capacitor_SMD:C_0805_2012Metric, F.Cu at (60.4, 39.3)
- added C23: 100n, Capacitor_SMD:C_0805_2012Metric, F.Cu at (60.4, 42.3)
- added C24: 100n, Capacitor_SMD:C_0805_2012Metric, F.Cu at (43.5, 144.1)
- added C25: 470p, Capacitor_SMD:C_0805_2012Metric, F.Cu at (43.5, 147.1)
- added C26: 100n, Capacitor_SMD:C_0805_2012Metric, F.Cu at (43.5, 150.1)
- added D6: D, Diode_SMD:D_0805_2012Metric, F.Cu at (66.8, 145.9)
- added Q5: MPS2907A, Package_TO_SOT_THT:TO-92_Inline, F.Cu at (-83.3, 152.0)
- added Q6: DMMT5401, Package_TO_SOT_SMD:SOT-23-6, F.Cu at (167.0, 85.1)
- added Q7: DMMT5401, Package_TO_SOT_SMD:SOT-23-6, F.Cu at (152.9, 85.4)
- added Q8: Q_NPN, Package_TO_SOT_THT:TO-92_Inline, F.Cu at (73.4, 48.9)
- added Q9: Q_NPN, Package_TO_SOT_THT:TO-92_Inline, F.Cu at (56.5, 153.4)
- added R24: 100k, Resistor_SMD:R_0805_2012Metric, F.Cu at (152.4, 79.2)
- added R25: 100k, Resistor_SMD:R_0805_2012Metric, F.Cu at (152.4, 76.7)
- added R26: 220k, Resistor_SMD:R_0805_2012Metric, F.Cu at (167.0, 92.1)
- added R27: 220k, Resistor_SMD:R_0805_2012Metric, F.Cu at (153.0, 94.6)
- added R28: 1k, Resistor_SMD:R_0805_2012Metric, F.Cu at (167.0, 94.6)
- added R29: 1k, Resistor_SMD:R_0805_2012Metric, F.Cu at (153.0, 92.1)
- added R30: 10k, Resistor_SMD:R_0805_2012Metric, F.Cu at (167.0, 89.5)
- added R31: 10k, Resistor_SMD:R_0805_2012Metric, F.Cu at (153.0, 89.5)
- added R32: 10k, Resistor_SMD:R_0805_2012Metric, F.Cu at (167.0, 97.2)
- added R33: 10k, Resistor_SMD:R_0805_2012Metric, F.Cu at (153.0, 97.2)
- added R34: R, Resistor_SMD:R_0805_2012Metric, F.Cu at (152.4, 81.8)
- added R35: 1K, Resistor_SMD:R_0805_2012Metric, F.Cu at (64.8, 33.2)
- added R36: 8.2k, Resistor_SMD:R_0805_2012Metric, F.Cu at (64.8, 36.2)
- added R37: 100k, Resistor_SMD:R_0805_2012Metric, F.Cu at (64.8, 39.1)
- added R38: 470k, Resistor_SMD:R_0805_2012Metric, F.Cu at (64.8, 42.1)
- added R39: 18k, Resistor_SMD:R_0805_2012Metric, F.Cu at (64.8, 45.0)
- added R40: 100, Resistor_SMD:R_0805_2012Metric, F.Cu at (64.8, 48.0)
- added R41: 8.2k, Resistor_SMD:R_0805_2012Metric, F.Cu at (52.3, 132.0)
- added R42: 100k, Resistor_SMD:R_0805_2012Metric, F.Cu at (52.3, 134.9)
- added R43: 470k, Resistor_SMD:R_0805_2012Metric, F.Cu at (52.3, 137.9)
- added R44: 18k, Resistor_SMD:R_0805_2012Metric, F.Cu at (52.3, 140.8)
- added R45: 100, Resistor_SMD:R_0805_2012Metric, F.Cu at (52.3, 143.8)
- added RV5: R_THRESHOLD_B1M, _effects_shared_footprints:Potentiometer_Alpha_RD901F-40-00D_Single_Vertical, F.Cu at (179.1, 68.7)
- added RV6: R_SUSTAIN-A100K, _effects_shared_footprints:Potentiometer_Alpha_RD901F-40-00D_Single_Vertical, F.Cu at (136.2, 68.7)
- added TP10: ~, TestPoint:TestPoint_Pad_D1.5mm, F.Cu at (208.5, 103.5)
- added TP11: ~, TestPoint:TestPoint_Pad_D1.5mm, F.Cu at (79.7, 47.4)
- added TP12: ~, TestPoint:TestPoint_Pad_D1.5mm, F.Cu at (62.8, 149.7)
- added TP6: ~, TestPoint:TestPoint_Pad_D1.5mm, F.Cu at (-92.3, 147.5)
- added TP7: ~, TestPoint:TestPoint_Pad_D1.5mm, F.Cu at (209.6, 69.2)
- added TP8: ~, TestPoint:TestPoint_Pad_D1.5mm, F.Cu at (200.7, 69.2)
- added TP9: ~, TestPoint:TestPoint_Pad_D1.5mm, F.Cu at (217.8, 103.5)
- added U1: TL074, Package_SO:SOIC-14_3.9x8.7mm_P1.27mm, F.Cu at (160.0, 77.5)
- added U2: MAX1044, Package_SO:SOIC-8_3.9x4.9mm_P1.27mm, F.Cu at (143.5, 98.4)
- added U3: LM317_TO-220, Package_TO_SOT_THT:TO-220-3_Vertical, F.Cu at (156.2, 109.2)
- added U4: LM337_TO220, Package_TO_SOT_THT:TO-220-3_Vertical, F.Cu at (144.8, 109.2)
- added U5: LM13700, Package_SO:SOIC-16_3.9x9.9mm_P1.27mm, F.Cu at (160.0, 91.4)
- C1, C10, C11, C12, C13, C4, C5, C8: footprint _project:C -> Capacitor_SMD:C_0805_2012Metric
- C14: value 10u -> 100n; footprint Capacitor_THT:CP_Radial_D6.3mm_P2.50mm -> Capacitor_SMD:C_0805_2012Metric
- C2, C6: value 470p -> 10u; footprint _project:C -> Capacitor_SMD:CP_Elec_5x3
- C3: value 100n -> 470p; footprint _project:C -> Capacitor_SMD:C_0805_2012Metric
- C7: value 100n -> 10u; footprint _project:C -> Capacitor_SMD:CP_Elec_5x3
- C9: value 470p -> 100n; footprint _project:C -> Capacitor_SMD:C_0805_2012Metric
- D1: value D -> LED; footprint Diode_THT:D_A-405_P2.54mm_Vertical_KathodeUp -> LED_THT:LED_D3.0mm
- D2, D3, D4: footprint Diode_THT:D_A-405_P2.54mm_Vertical_KathodeUp -> Diode_SMD:D_0805_2012Metric
- D5: value LED -> D; footprint LED_THT:LED_D3.0mm -> Diode_SMD:D_0805_2012Metric
- Q3, Q4: value Q_NPN -> 2N5088
- R1: value 33k -> 3.3k; footprint _project:R -> Resistor_SMD:R_0805_2012Metric
- R10: value 18k -> 220; footprint _project:R -> Resistor_SMD:R_0805_2012Metric
- R11: value 100 -> 220; footprint _project:R -> Resistor_SMD:R_0805_2012Metric
- R12: value 8.2k -> 3.3k; footprint _project:R -> Resistor_SMD:R_0805_2012Metric
- R13: value 100k -> 470k; footprint _project:R -> Resistor_SMD:R_0805_2012Metric
- R14, R3: value 470k -> 100k; footprint _project:R -> Resistor_SMD:R_0805_2012Metric
- R15: value 18k -> 10k; footprint _project:R -> Resistor_SMD:R_0805_2012Metric
- R16: value 100 -> 3.3k; footprint _project:R -> Resistor_SMD:R_0805_2012Metric
- R17: value 33k -> 1K; footprint _project:R -> Resistor_SMD:R_0805_2012Metric
- R18: value 3.3k -> 3.3M; footprint _project:R -> Resistor_SMD:R_0805_2012Metric
- R19: value 3.3k -> 10K; footprint _project:R -> Resistor_SMD:R_0805_2012Metric
- R2: value 100k -> 33k; footprint _project:R -> Resistor_SMD:R_0805_2012Metric
- R20: value 470k -> 10K; footprint _project:R -> Resistor_SMD:R_0805_2012Metric
- R21: value 100k -> 15k; footprint _project:R -> Resistor_SMD:R_0805_2012Metric
- R22: value 10k -> 100k; footprint _project:R -> Resistor_SMD:R_0805_2012Metric
- R23: value 3.3k -> 100k; footprint _project:R -> Resistor_SMD:R_0805_2012Metric
- R4: value 10k -> 470k; footprint _project:R -> Resistor_SMD:R_0805_2012Metric
- R5: value 100 -> 10k; footprint _project:R -> Resistor_SMD:R_0805_2012Metric
- R6: value 1K -> 100; footprint _project:R -> Resistor_SMD:R_0805_2012Metric
- R7: value 8.2k -> 1.2k; footprint _project:R -> Resistor_SMD:R_0805_2012Metric
- R8: value 100k -> 1.2k; footprint _project:R -> Resistor_SMD:R_0805_2012Metric
- R9: value 470k -> 33k; footprint _project:R -> Resistor_SMD:R_0805_2012Metric
- RV1: value R_SUSTAIN-A100K -> R_MID-B25K
- RV2: value R_MID-B25K -> R_TONE-B100K
- RV3: value R_TONE-B100K -> R_VOL-A100K
- RV4: value R_VOL-A100K -> R_INTENSITY_B100K
- moved Q4 259.3 mm to (-106.1, 149.3)
- moved R20 259.3 mm to (-100.9, 151.6)
- moved Q3 254.4 mm to (-96.9, 65.2)
- moved R17 252.3 mm to (-87.0, 66.5)
- moved R18 252.3 mm to (-93.1, 83.5)
- moved TP5 252.3 mm to (-119.3, 75.9)
- moved R19 252.3 mm to (-80.9, 66.5)
- moved Q2 237.1 mm to (79.4, 288.9)
- moved R13 237.1 mm to (68.2, 303.4)
- moved R14 237.1 mm to (73.3, 303.4)
- moved R15 237.1 mm to (73.8, 280.5)
- moved C14 237.1 mm to (80.0, 274.4)
- moved TP4 237.1 mm to (48.4, 300.9)
- moved R16 237.1 mm to (68.2, 289.2)
- moved C1 209.3 mm to (54.5, -79.7)
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Connections:
- C10 pad 2: Net-(D3-A) -> /vca/OUT
- C12 pad 1: Net-(Q4-B) -> Net-(Q2-B)
- C13 pad 1: Net-(Q4-C) -> +7.5V
- C13 pad 2: Net-(C13-Pad2) -> -7.5V
- C14 pad 1: +9V -> Net-(Q2-C)
- C14 pad 2: GND -> Net-(C14-Pad2)
- C2 pad 1: Net-(Q1-B) -> +9V
- C2 pad 2: Net-(Q1-C) -> GND
- C3 pad 1: Net-(Q1-C) -> Net-(Q1-B)
- C3 pad 2: Net-(C3-Pad2) -> Net-(Q1-C)
- C4 pad 1: Net-(C4-Pad1) -> +9V
- C4 pad 2: Net-(C4-Pad2) -> GND
- C5 pad 1: Net-(Q2-B) -> Net-(Q1-C)
- C5 pad 2: Net-(D1-K) -> /Devi Gain/DEVI_IN
- C6 pad 1: Net-(Q2-B) -> Net-(U2-CAP+)
- C6 pad 2: Net-(D1-A) -> Net-(U2-CAP-)
- C7 pad 1: Net-(D1-A) -> GND
- C7 pad 2: Net-(C7-Pad2) -> -9V
- C8 pad 1: Net-(Q3-B) -> +9V
- C8 pad 2: Net-(D3-K) -> GND
- C9 pad 1: Net-(Q3-B) -> GND
- C9 pad 2: Net-(D3-A) -> -9V
- D1 pad 2: Net-(D1-A) -> LED
- D2 pad 1: Net-(D1-A) -> /vca/IN
- D2 pad 2: Net-(D1-K) -> Net-(D2-A)
- D5 pad 2: LED -> Net-(D5-A)
- Q2 pad 3: Net-(D1-A) -> Net-(Q2-C)
- Q3 pad 1: Net-(Q3-E) -> (no net)
- Q3 pad 2: Net-(Q3-B) -> (no net)
- Q3 pad 3: Net-(D3-A) -> (no net)
- Q4 pad 1: Net-(Q4-E) -> (no net)
- Q4 pad 2: Net-(Q4-B) -> (no net)
- Q4 pad 3: Net-(Q4-C) -> (no net)
- R1 pad 1: IN -> GND
- R1 pad 2: Net-(C1-Pad1) -> Net-(D1-K)
- R10 pad 1: +9V -> +7.5V
- R10 pad 2: Net-(D1-A) -> Net-(U3-ADJ)
- R11 pad 1: Net-(Q2-E) -> Net-(U4-ADJ)
- R11 pad 2: GND -> -7.5V
- R12 pad 1: Net-(C7-Pad2) -> Net-(R12-Pad1)
- R12 pad 2: Net-(Q3-B) -> GND
- R13 pad 1: Net-(Q3-B) -> Net-(Q2-B)
- R13 pad 2: GND -> +9V
- R14 pad 1: Net-(Q3-B) -> Net-(Q2-B)
- R14 pad 2: Net-(D3-A) -> GND
- R15 pad 2: Net-(D3-A) -> Net-(Q2-C)
- R16 pad 1: Net-(Q3-E) -> Net-(Q2-E)
- R17 pad 1: Net-(D3-A) -> Net-(R17-Pad1)
- R17 pad 2: Net-(C11-Pad1) -> GND
- R18 pad 1: GND -> Net-(C16-Pad2)
- R18 pad 2: Net-(D5-K) -> Net-(C17-Pad1)
- R19 pad 1: Net-(R19-Pad1) -> +9V
- R19 pad 2: GND -> Net-(C17-Pad1)
- R2 pad 1: GND -> /vca/IN
- R2 pad 2: Net-(Q1-B) -> Net-(C1-Pad1)
- R20 pad 1: Net-(Q4-B) -> +9V
- R20 pad 2: +9V -> Net-(C18-Pad1)
- R21 pad 1: Net-(Q4-B) -> Net-(D2-A)
- R21 pad 2: GND -> Net-(U1B--)
- R22 pad 1: +9V -> Net-(U1B--)
- R22 pad 2: Net-(Q4-C) -> Net-(R22-Pad2)
- R23 pad 1: Net-(Q4-E) -> Net-(R23-Pad1)
- R23 pad 2: GND -> Net-(U1C--)
- R3 pad 1: Net-(Q1-B) -> GND
- R3 pad 2: Net-(Q1-C) -> Net-(Q1-B)
- R4 pad 1: +9V -> Net-(Q1-B)
- R5 pad 1: Net-(Q1-E) -> +9V
- R5 pad 2: GND -> Net-(Q1-C)
- R6 pad 1: Net-(R6-Pad1) -> Net-(Q1-E)
- R7 pad 1: Net-(C4-Pad2) -> Net-(U3-ADJ)
- R7 pad 2: Net-(Q2-B) -> GND
- R8 pad 1: Net-(Q2-B) -> GND
- R8 pad 2: GND -> Net-(U4-ADJ)
- R9 pad 1: Net-(Q2-B) -> /vca/OUT
- R9 pad 2: Net-(D1-A) -> Net-(C11-Pad1)
- RV1 pad 1: Net-(R6-Pad1) -> Net-(C10-Pad1)
- RV1 pad 2: Net-(C4-Pad1) -> Net-(C10-Pad1)
- RV1 pad 3: Net-(C3-Pad2) -> Net-(R12-Pad1)
- RV2 pad 1: Net-(C10-Pad1) -> Net-(C11-Pad1)
- RV2 pad 2: Net-(C10-Pad1) -> Net-(C12-Pad2)
- RV2 pad 3: Net-(R19-Pad1) -> Net-(C10-Pad1)
- RV3 pad 1: Net-(C11-Pad1) -> GND
- RV3 pad 2: Net-(C12-Pad2) -> OUT
- RV3 pad 3: Net-(C10-Pad1) -> Net-(C14-Pad2)
- RV4 pad 1: GND -> /Devi Gain/DEVI_IN
- RV4 pad 2: OUT -> Net-(C16-Pad1)
- RV4 pad 3: Net-(C13-Pad2) -> Net-(R17-Pad1)
- TP2 pad 1: Net-(D1-A) -> /vca/OUT
- TP3 pad 1: Net-(D3-A) -> Net-(C12-Pad2)
- TP4 pad 1: Net-(C12-Pad2) -> Net-(Q2-C)
- TP5 pad 1: Net-(Q4-C) -> Net-(C17-Pad1)
Routing:
- net +9V: track 83.7 -> 0.00 mm
- net Net-(D3-A): track 64.0 -> 0.00 mm
- net Net-(C10-Pad1): track 52.3 -> 0.00 mm
- net Net-(D1-A): track 49.8 -> 0.00 mm
- net Net-(Q4-C): track 49.3 -> 0.00 mm
- net Net-(Q1-B): track 49.2 -> 0.00 mm
- net OUT: track 45.3 -> 0.00 mm, vias 1 -> 0
- net Net-(C11-Pad1): track 35.1 -> 0.00 mm
- net Net-(Q3-B): track 32.3 -> 0.00 mm
- net Net-(Q2-B): track 31.5 -> 0.00 mm
- net Net-(Q1-C): track 27.3 -> 0.00 mm
- net Net-(C12-Pad2): track 25.9 -> 0.00 mm
- net Net-(C3-Pad2): track 22.6 -> 0.00 mm
- net Net-(J4-Pin_1): track 22.5 -> 0.00 mm
- net Net-(C13-Pad2): track 21.9 -> 0.00 mm
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Other:
- board size 58.4 x 85.1 mm -> 58.4 x 91.7 mm
