File: dist/dynafuzz/dynafuzz.kicad_sch (KiCad schematic)
At the start: 54 parts, among them J1 AudioJack_IN, J2 AudioJack_OUT, J3 Jack-DC, Q1 Q_NPN, Q2 Q_NPN, Q3 Q_NPN, Q4 Q_NPN, SW1 SW_3PDT_x3

Commit message: update positions
Parts:
- RV1, RV2, RV3, RV4: footprint Potentiometer_THT:Potentiometer_Alpha_RD901F-40-00D_Single_Vertical -> _effects_shared_footprints:Potentiometer_Alpha_RD901F-40-00D_Single_Vertical
Connections:
- net +9V: now also R10.1, R15.1; no longer R10.2, R15.2
- net GND: now also R18.1, R2.1; no longer R18.2, R2.2
- net IN: now also R1.1; no longer R1.2
- net at C10.2, C9.2, D3.2 (A)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: now also R15.2; no longer R15.1
- net at C1.2, C2.1, Q1.2 (B)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: now also R2.2; no longer R2.1
- net at C1.1: now also R1.2; no longer R1.1
- net at D5.1 (K): now also R18.2; no longer R18.1
- net at C6.2, C7.1, D1.2 (A)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: now also R10.2; no longer R10.1
Other:
- moved on the sheet: R1, R10, R15, R18, R2
Changed lines of the file:
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@@
 			)
 		)
-		(property "Footprint" "Potentiometer_THT:Potentiometer_Alpha_RD901F-40-00D_Single_Vertical"
+		(property "Footprint" "_effects_shared_footprints:Potentiometer_Alpha_RD901F-40-00D_Single_Vertical"
 			(at 88.9 109.22 0)
 			(effects
@@
 			)
 		)
-		(property "Footprint" "Potentiometer_THT:Potentiometer_Alpha_RD901F-40-00D_Single_Vertical"
+		(property "Footprint" "_effects_shared_footprints:Potentiometer_Alpha_RD901F-40-00D_Single_Vertical"
 			(at 256.54 114.3 0)
 			(effects
@@
 	(symbol
 		(lib_id "Device:R")
-		(at 55.88 111.76 0)
+		(at 55.88 111.76 180)
 		(unit 1)
 		(exclude_from_sim no)
@@
 					(size 1.27 1.27)
 				)
-				(justify left)
+				(justify right)
 			)
 		)
@@
 					(size 1.27 1.27)
 				)
-				(justify left)
+				(justify right)
 			)
 		)
 		(property "Footprint" "_project:R"
-			(at 54.102 111.76 90)
+			(at 57.658 111.76 90)
 			(effects
 				(font
@@
 			)
 		)
-		(property "Footprint" "Potentiometer_THT:Potentiometer_Alpha_RD901F-40-00D_Single_Vertical"
+		(property "Footprint" "_effects_shared_footprints:Potentiometer_Alpha_RD901F-40-00D_Single_Vertical"
 			(at 200.66 110.49 0)
 			(effects
@@
 	(symbol
 		(lib_id "Device:R")
-		(at 38.1 105.41 270)
+		(at 38.1 105.41 90)
 		(unit 1)
 		(exclude_from_sim no)
@@
 		)
 		(property "Footprint" "_project:R"
-			(at 38.1 103.632 90)
+			(at 38.1 107.188 90)
 			(effects
 				(font
@@
 			)
 		)
-		(property "Footprint" "Potentiometer_THT:Potentiometer_Alpha_RD901F-40-00D_Single_Vertical"
+		(property "Footprint" "_effects_shared_footprints:Potentiometer_Alpha_RD901F-40-00D_Single_Vertical"
 			(at 200.66 95.25 0)
 			(effects
@@
 	(symbol
 		(lib_id "Device:R")
-		(at 200.66 44.45 0)
+		(at 200.66 44.45 180)
 		(unit 1)
 		(exclude_from_sim no)
@@
 					(size 1.27 1.27)
 				)
-				(justify left)
+				(justify right)
 			)
 		)
@@
 					(size 1.27 1.27)
 				)
-				(justify left)
+				(justify right)
 			)
 		)
 		(property "Footprint" "_project:R"
-			(at 198.882 44.45 90)
+			(at 202.438 44.45 90)
 			(effects
 				(font
@@
 	(symbol
 		(lib_id "Device:R")
-		(at 129.54 78.74 180)
+		(at 129.54 78.74 0)
 		(unit 1)
 		(exclude_from_sim no)
@@
 					(size 1.27 1.27)
 				)
-				(justify right)
+				(justify left)
 			)
 		)
@@
 					(size 1.27 1.27)
 				)
-				(justify right)
+				(justify left)
 			)
 		)
 		(property "Footprint" "_project:R"
-			(at 131.318 78.74 90)
+			(at 127.762 78.74 90)
 			(effects
 				(font
@@
 	(symbol
 		(lib_id "Device:R")
-		(at 172.72 80.01 180)
+		(at 172.72 80.01 0)
 		(unit 1)
 		(exclude_from_sim no)
@@
 					(size 1.27 1.27)
 				)
-				(justify right)
+				(justify left)
 			)
 		)
@@
 					(size 1.27 1.27)
 				)
-				(justify right)
+				(justify left)
 			)
 		)
 		(property "Footprint" "_project:R"
-			(at 174.498 80.01 90)
+			(at 170.942 80.01 90)
 			(effects
 				(font

Commit message: finish layout
Connections:
- net GND: now also RV4.1; no longer RV4.3
- net at RV1.1: now also R6.1; no longer C3.2
- net at RV1.3: now also C3.2; no longer R6.1
- net at C13.2: now also RV4.3; no longer RV4.1
- net at C11.1, R17.2: now also RV3.1; no longer RV3.3
- net at C10.1, RV2.2: now also RV2.1, RV3.3; no longer RV2.3, RV3.1
- net at R19.1: now also RV2.3; no longer RV2.1
Other:
- note added: "TODO: silkscreen gfx"
- note added: "TODO: stompboard"
- note removed: "TODO: pot orientation"
Changed lines of the file:
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@@
 	(generator_version "9.0")
 	(paper "A4")
+	(text "TODO: silkscreen gfx"
+		(exclude_from_sim no)
+		(at 148.844 60.452 0)
+		(effects
+			(font
+				(size 1.27 1.27)
+			)
+		)
+	)
 	(text "HOOF Tone Stack"
 		(exclude_from_sim no)
@@
 		)
 	)
-	(text "https://tonestack.yuriturov.com/?s=eNpbmpj-NbFsWVKQ02_7261yOwJftyYF-TImBYX8tr_x9VB_jMa3pCDn3_YPFl_nsi1YkhQU9tv-1kP3dSJVj5KCwoFs2wKQTGJFYllSUfGCxJKWRYmZKbmlaYaJySuTgzz9Eg2SgnxSDA0MsoHmNicbmWYn-vyyZ2BgAFrRDBaH8w2TjY2BqoxSjPWAtLNhsqFBXpKzEYQyBqnNgxpulJi8CtNwVNOAphuZophuCFJmlGxmgWR4iomeOcj0ZBMQZYJsCcwHyYam2aT4wRLsByM9I5A1KWZ6FmB7IDRWXyQbGmWT4Q9TM7A_wA4Hhxm6PwB9TKNZ"
+	(text "TODO: stompboard"
 		(exclude_from_sim no)
-		(at 210.058 216.154 0)
+		(at 149.606 51.054 0)
 		(effects
 			(font
@@
 		)
 	)
-	(text "OUTPUT STAGE"
+	(text "https://tonestack.yuriturov.com/?s=eNpbmpj-NbFsWVKQ02_7261yOwJftyYF-TImBYX8tr_x9VB_jMa3pCDn3_YPFl_nsi1YkhQU9tv-1kP3dSJVj5KCwoFs2wKQTGJFYllSUfGCxJKWRYmZKbmlaYaJySuTgzz9Eg2SgnxSDA0MsoHmNicbmWYn-vyyZ2BgAFrRDBaH8w2TjY2BqoxSjPWAtLNhsqFBXpKzEYQyBqnNgxpulJi8CtNwVNOAphuZophuCFJmlGxmgWR4iomeOcj0ZBMQZYJsCcwHyYam2aT4wRLsByM9I5A1KWZ6FmB7IDRWXyQbGmWT4Q9TM7A_wA4Hhxm6PwB9TKNZ"
 		(exclude_from_sim no)
-		(at 247.142 135.382 0)
+		(at 210.058 216.154 0)
 		(effects
 			(font
@@
 		)
 	)
-	(text "TODO: pot orientation"
+	(text "OUTPUT STAGE"
 		(exclude_from_sim no)
-		(at 199.39 86.106 0)
+		(at 247.142 135.382 0)
 		(effects
 			(font
@@
 		(lib_id "Device:R_Potentiometer")
 		(at 88.9 109.22 0)
+		(mirror x)
 		(unit 1)
 		(exclude_from_sim no)
@@
 		(on_board yes)
 		(dnp no)
-		(fields_autoplaced yes)
 		(property "Reference" "RV1"
-			(at 86.36 107.9499 0)
+			(at 86.36 110.4901 0)
 			(effects
 				(font
@@
 		)
 		(property "Value" "R_SUSTAIN-A100K"
-			(at 86.36 110.4899 0)
+			(at 86.36 107.9501 0)
 			(effects
 				(font
@@
 		(lib_id "Device:R_Potentiometer")
 		(at 256.54 114.3 0)
+		(mirror x)
 		(unit 1)
 		(exclude_from_sim no)
@@
 		(on_board yes)
 		(dnp no)
-		(fields_autoplaced yes)
 		(property "Reference" "RV4"
-			(at 254 113.0299 0)
+			(at 254 115.5701 0)
 			(effects
 				(font
@@
 		)
 		(property "Value" "R_VOL-A100K"
-			(at 254 115.5699 0)
+			(at 254 113.0301 0)
 			(effects
 				(font
@@
 		(lib_id "Device:R_Potentiometer")
 		(at 200.66 110.49 0)
+		(mirror x)
 		(unit 1)
 		(exclude_from_sim no)
@@
 		(on_board yes)
 		(dnp no)
-		(fields_autoplaced yes)
 		(property "Reference" "RV3"
-			(at 198.12 109.2199 0)
+			(at 198.12 111.7601 0)
 			(effects
 				(font
@@
 		)
 		(property "Value" "R_TONE-B100K"
-			(at 198.12 111.7599 0)
+			(at 198.12 109.2201 0)
 			(effects
 				(font
@@
 		(lib_id "Device:R_Potentiometer")
 		(at 200.66 95.25 0)
+		(mirror x)
 		(unit 1)
 		(exclude_from_sim no)
@@
 		(on_board yes)
 		(dnp no)
-		(fields_autoplaced yes)
 		(property "Reference" "RV2"
-			(at 198.12 93.9799 0)
+			(at 198.12 96.5201 0)
 			(effects
 				(font
@@
 		)
 		(property "Value" "R_MID-B25K"
-			(at 198.12 96.5199 0)
+			(at 198.12 93.9801 0)
 			(effects
 				(font

Commit message: board interconnect
Parts:
- added J4: MAIN_BIC, Connector_PinSocket_2.54mm:PinSocket_1x06_P2.54mm_Vertical, symbol Connector:Conn_01x06_Socket
- added J5: SWITCH_BIC, Connector_PinSocket_2.54mm:PinSocket_1x06_P2.54mm_Vertical, symbol Connector:Conn_01x06_Socket
- SW1: footprint Connector_PinSocket_2.54mm:PinSocket_1x09_P2.54mm_Vertical -> _effects_shared_footprints:Stompbox Switch
Connections:
- net +9V: now also J4.4 (Pin_4); no longer SW1.4 (A)
- net IN: now also J4.2 (Pin_2); no longer SW1.7 (A)
- net OUT: now also J4.6 (Pin_6); no longer SW1.1 (A)
- net at SW1.5 (B): now also J5.4 (Pin_4); no longer D5.2 (A)
- net at SW1.8 (B): now also J5.1 (Pin_1); no longer J1.T
- net at SW1.2 (B): now also J5.5 (Pin_5); no longer J2.T
- new net: J5.2 (Pin_2), SW1.7 (A)
- new net: J5.6 (Pin_6), SW1.1 (A)
- new net: J2.T, J4.5 (Pin_5)
- new net: J5.3 (Pin_3), SW1.4 (A)
- new net: J1.T, J4.1 (Pin_1)
- new net LED: D5.2 (A), J4.3 (Pin_3)
Other:
- note removed: "TODO: silkscreen gfx"
- note removed: "TODO: stompboard"
- moved on the sheet: J1, J2, SW1A, SW1B, SW1C

Commit message: rev A
Connections:
- net at SW1.7 (A): now also SW1.1 (A); no longer J5.2 (Pin_2)
- net at SW1.9 (C): now also J5.2 (Pin_2); no longer SW1.3 (C)
- net at J5.6 (Pin_6): now also SW1.3 (C); no longer SW1.1 (A)
- net at J5.3 (Pin_3): now also SW1.6 (C); no longer SW1.4 (A)
Other:
- moved on the sheet: SW1A
Changed lines of the file:
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@@
 		(lib_id "_project:SW_3PDT_x3")
 		(at 107.95 167.64 0)
+		(mirror x)
 		(unit 3)
 		(exclude_from_sim no)
@@
 		(dnp no)
 		(property "Reference" "SW1"
-			(at 107.95 158.75 0)
+			(at 107.95 176.53 0)
 			(effects
 				(font
@@
 		)
 		(property "Value" "SW_3PDT_x3"
-			(at 107.95 161.29 0)
+			(at 107.95 173.99 0)
 			(effects
 				(font
@@
 	(symbol
 		(lib_id "_project:SW_3PDT_x3")
-		(at 129.54 167.64 0)
-		(mirror y)
+		(at 129.54 167.64 180)
 		(unit 1)
 		(exclude_from_sim no)
@@
 		(dnp no)
 		(property "Reference" "SW1"
-			(at 129.54 158.75 0)
+			(at 129.54 176.53 0)
 			(effects
 				(font
@@
 		)
 		(property "Value" "SW_3PDT_x3"
-			(at 129.54 161.29 0)
+			(at 129.54 173.99 0)
 			(effects
 				(font
@@
 		(lib_id "_project:SW_3PDT_x3")
 		(at 144.78 181.61 0)
+		(mirror x)
 		(unit 2)
 		(exclude_from_sim no)
@@
 		(dnp no)
 		(property "Reference" "SW1"
-			(at 144.526 187.198 0)
+			(at 144.526 176.022 0)
 			(effects
 				(font
@@
 		)
 		(property "Value" "SW_3PDT_x3"
-			(at 144.526 189.738 0)
+			(at 144.526 173.482 0)
 			(effects
 				(font
