File: dist/dynafuzz/deviever.kicad_sch (KiCad schematic)
At the start: 11 parts, among them Q1 2N5088, Q2 2N5088, Q3 MPS2907A

Commit message: schematic for dynafuzz
Parts:
- renumbered C1 to C15, C2 to C16, C3 to C17, Q1 to Q5, Q2 to Q6, Q3 to Q7, R4 to R24, R1 to R25, R2 to R26, R3 to R27, RV1 to RV5
Changed lines of the file:
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@@
 		(dnp no)
 		(fields_autoplaced yes)
-		(property "Reference" "RV1"
+		(property "Reference" "RV5"
 			(at 76.2 86.3599 0)
 			(effects
@@
 			(project "dynafuzz"
 				(path "/b401260a-0de9-4b23-a692-63e5f9163375/3a19848d-9449-4a2f-9659-066f51bd527c"
-					(reference "RV1")
+					(reference "RV5")
 					(unit 1)
 				)
@@
 		(dnp no)
 		(fields_autoplaced yes)
-		(property "Reference" "C2"
+		(property "Reference" "C16"
 			(at 123.19 78.74 90)
 			(effects
@@
 			(project "dynafuzz"
 				(path "/b401260a-0de9-4b23-a692-63e5f9163375/3a19848d-9449-4a2f-9659-066f51bd527c"
-					(reference "C2")
+					(reference "C16")
 					(unit 1)
 				)
@@
 		(dnp no)
 		(fields_autoplaced yes)
-		(property "Reference" "Q1"
+		(property "Reference" "Q5"
 			(at 110.49 86.3599 0)
 			(effects
@@
 			(project "dynafuzz"
 				(path "/b401260a-0de9-4b23-a692-63e5f9163375/3a19848d-9449-4a2f-9659-066f51bd527c"
-					(reference "Q1")
+					(reference "Q5")
 					(unit 1)
 				)
@@
 		(dnp no)
 		(fields_autoplaced yes)
-		(property "Reference" "C3"
+		(property "Reference" "C17"
 			(at 158.75 80.01 90)
 			(effects
@@
 			(project "dynafuzz"
 				(path "/b401260a-0de9-4b23-a692-63e5f9163375/3a19848d-9449-4a2f-9659-066f51bd527c"
-					(reference "C3")
+					(reference "C17")
 					(unit 1)
 				)
@@
 		(dnp no)
 		(fields_autoplaced yes)
-		(property "Reference" "R4"
+		(property "Reference" "R24"
 			(at 81.28 96.5199 0)
 			(effects
@@
 			(project "dynafuzz"
 				(path "/b401260a-0de9-4b23-a692-63e5f9163375/3a19848d-9449-4a2f-9659-066f51bd527c"
-					(reference "R4")
+					(reference "R24")
 					(unit 1)
 				)
@@
 		(dnp no)
 		(fields_autoplaced yes)
-		(property "Reference" "R2"
+		(property "Reference" "R26"
 			(at 110.49 69.8499 0)
 			(effects
@@
 			(project "dynafuzz"
 				(path "/b401260a-0de9-4b23-a692-63e5f9163375/3a19848d-9449-4a2f-9659-066f51bd527c"
-					(reference "R2")
+					(reference "R26")
 					(unit 1)
 				)
@@
 		(dnp no)
 		(fields_autoplaced yes)
-		(property "Reference" "R3"
+		(property "Reference" "R27"
 			(at 153.67 67.3099 0)
 			(effects
@@
 			(project "dynafuzz"
 				(path "/b401260a-0de9-4b23-a692-63e5f9163375/3a19848d-9449-4a2f-9659-066f51bd527c"
-					(reference "R3")
+					(reference "R27")
 					(unit 1)
 				)
@@
 		(dnp no)
 		(fields_autoplaced yes)
-		(property "Reference" "Q2"
+		(property "Reference" "Q6"
 			(at 140.97 85.0899 0)
 			(effects
@@
 			(project "dynafuzz"
 				(path "/b401260a-0de9-4b23-a692-63e5f9163375/3a19848d-9449-4a2f-9659-066f51bd527c"
-					(reference "Q2")
+					(reference "Q6")
 					(unit 1)
 				)
@@
 		(dnp no)
 		(fields_autoplaced yes)
-		(property "Reference" "C1"
+		(property "Reference" "C15"
 			(at 90.17 80.01 90)
 			(effects
@@
 			(project "dynafuzz"
 				(path "/b401260a-0de9-4b23-a692-63e5f9163375/3a19848d-9449-4a2f-9659-066f51bd527c"
-					(reference "C1")
+					(reference "C15")
 					(unit 1)
 				)
@@
 		(dnp no)
 		(fields_autoplaced yes)
-		(property "Reference" "Q3"
+		(property "Reference" "Q7"
 			(at 153.67 93.9799 0)
 			(effects
@@
 			(project "dynafuzz"
 				(path "/b401260a-0de9-4b23-a692-63e5f9163375/3a19848d-9449-4a2f-9659-066f51bd527c"
-					(reference "Q3")
+					(reference "Q7")
 					(unit 1)
 				)
@@
 		(on_board yes)
 		(dnp no)
-		(property "Reference" "R1"
+		(property "Reference" "R25"
 			(at 103.378 73.914 90)
 			(effects
@@
 			(project "dynafuzz"
 				(path "/b401260a-0de9-4b23-a692-63e5f9163375/3a19848d-9449-4a2f-9659-066f51bd527c"
-					(reference "R1")
-					(unit 1)
-				)
+					(reference "R25")
+					(unit 1)
+				)

Commit message: add vca envelope detector to dynafuzz
Parts:
- added TP5, TP6: ~, TestPoint:TestPoint_Pad_D1.5mm, symbol Connector:TestPoint
- C16: renamed from C15; footprint (none) -> Capacitor_SMD:C_0805_2012Metric
- C17: renamed from C16; footprint (none) -> Capacitor_SMD:C_0805_2012Metric
- C18: renamed from C17; footprint (none) -> Capacitor_SMD:C_0805_2012Metric
- Q3: renamed from Q5; footprint (none) -> Package_TO_SOT_THT:TO-92_Inline
- Q4: renamed from Q6; footprint (none) -> Package_TO_SOT_THT:TO-92_Inline
- Q5: renamed from Q7; footprint (none) -> Package_TO_SOT_THT:TO-92_Inline
- R17: renamed from R24; footprint (none) -> Resistor_SMD:R_0805_2012Metric
- R18: renamed from R25; footprint (none) -> Resistor_SMD:R_0805_2012Metric
- R19: renamed from R26; footprint (none) -> Resistor_SMD:R_0805_2012Metric
- R20: renamed from R27; footprint (none) -> Resistor_SMD:R_0805_2012Metric
- RV4: renamed from RV5; footprint (none) -> _effects_shared_footprints:Potentiometer_Alpha_RD901F-40-00D_Single_Vertical
Connections:
- net at C17.1, Q3.C, R18.2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: now also TP5.1
- net at C18.1, Q4.C, Q5.C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: now also TP6.1

Commit message: updates
Parts:
- renumbered C16 to C14, C17 to C15, C18 to C16
Changed lines of the file:
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@@
 		(dnp no)
 		(fields_autoplaced yes)
-		(property "Reference" "#PWR038"
+		(property "Reference" "#PWR030"
 			(at 144.78 111.76 0)
 			(effects
@@
 			(project "dynafuzz"
 				(path "/b401260a-0de9-4b23-a692-63e5f9163375/3a19848d-9449-4a2f-9659-066f51bd527c"
-					(reference "#PWR038")
+					(reference "#PWR030")
 					(unit 1)
 				)
@@
 		(dnp no)
 		(fields_autoplaced yes)
-		(property "Reference" "C17"
+		(property "Reference" "C15"
 			(at 123.19 78.74 90)
 			(effects
@@
 			(project "dynafuzz"
 				(path "/b401260a-0de9-4b23-a692-63e5f9163375/3a19848d-9449-4a2f-9659-066f51bd527c"
-					(reference "C17")
+					(reference "C15")
 					(unit 1)
 				)
@@
 		(dnp no)
 		(fields_autoplaced yes)
-		(property "Reference" "C18"
+		(property "Reference" "C16"
 			(at 158.75 80.01 90)
 			(effects
@@
 			(project "dynafuzz"
 				(path "/b401260a-0de9-4b23-a692-63e5f9163375/3a19848d-9449-4a2f-9659-066f51bd527c"
-					(reference "C18")
+					(reference "C16")
 					(unit 1)
 				)
@@
 		(dnp no)
 		(fields_autoplaced yes)
-		(property "Reference" "#PWR039"
+		(property "Reference" "#PWR031"
 			(at 151.13 66.04 0)
 			(effects
@@
 			(project "dynafuzz"
 				(path "/b401260a-0de9-4b23-a692-63e5f9163375/3a19848d-9449-4a2f-9659-066f51bd527c"
-					(reference "#PWR039")
+					(reference "#PWR031")
 					(unit 1)
 				)
@@
 		(dnp no)
 		(fields_autoplaced yes)
-		(property "Reference" "#PWR035"
+		(property "Reference" "#PWR027"
 			(at 78.74 110.49 0)
 			(effects
@@
 			(project "dynafuzz"
 				(path "/b401260a-0de9-4b23-a692-63e5f9163375/3a19848d-9449-4a2f-9659-066f51bd527c"
-					(reference "#PWR035")
+					(reference "#PWR027")
 					(unit 1)
 				)
@@
 		(dnp no)
 		(fields_autoplaced yes)
-		(property "Reference" "C16"
+		(property "Reference" "C14"
 			(at 90.17 80.01 90)
 			(effects
@@
 			(project "dynafuzz"
 				(path "/b401260a-0de9-4b23-a692-63e5f9163375/3a19848d-9449-4a2f-9659-066f51bd527c"
-					(reference "C16")
+					(reference "C14")
 					(unit 1)
 				)
@@
 		(dnp no)
 		(fields_autoplaced yes)
-		(property "Reference" "#PWR037"
+		(property "Reference" "#PWR029"
 			(at 107.95 102.87 0)
 			(effects
@@
 			(project "dynafuzz"
 				(path "/b401260a-0de9-4b23-a692-63e5f9163375/3a19848d-9449-4a2f-9659-066f51bd527c"
-					(reference "#PWR037")
+					(reference "#PWR029")
 					(unit 1)
 				)
@@
 		(dnp no)
 		(fields_autoplaced yes)
-		(property "Reference" "#PWR036"
+		(property "Reference" "#PWR028"
 			(at 107.95 68.58 0)
 			(effects
@@
 			(project "dynafuzz"
 				(path "/b401260a-0de9-4b23-a692-63e5f9163375/3a19848d-9449-4a2f-9659-066f51bd527c"
-					(reference "#PWR036")
-					(unit 1)
-				)
+					(reference "#PWR028")
+					(unit 1)
+				)
