File: dist/dynafuzz/muff.kicad_sch (KiCad schematic)
At the start: 27 parts, among them Q8 Q_NPN, Q9 Q_NPN

Commit message: updates
Parts:
- renumbered C20 to C22, C21 to C23, C22 to C24, C23 to C25, C24 to C26, C25 to C27, C26 to C28, R35 to R40, R36 to R41, R37 to R42, R38 to R43, R39 to R44, R40 to R45, R41 to R46, R42 to R47, R43 to R48, R44 to R49, R45 to R50, RV6 to RV9, TP12 to TP10, TP11 to TP9
Changed lines of the file:
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@@
 		(on_board yes)
 		(dnp no)
-		(property "Reference" "RV6"
+		(property "Reference" "RV9"
 			(at 103.378 105.41 0)
 			(effects
@@
 			(project "dynafuzz"
 				(path "/b401260a-0de9-4b23-a692-63e5f9163375/5e6de810-895a-4442-a10c-7662380a0e10"
-					(reference "RV6")
+					(reference "RV9")
 					(unit 1)
 				)
@@
 		(dnp no)
 		(fields_autoplaced yes)
-		(property "Reference" "C26"
+		(property "Reference" "C28"
 			(at 199.39 86.36 90)
 			(effects
@@
 			(project "dynafuzz"
 				(path "/b401260a-0de9-4b23-a692-63e5f9163375/5e6de810-895a-4442-a10c-7662380a0e10"
-					(reference "C26")
+					(reference "C28")
 					(unit 1)
 				)
@@
 		(on_board yes)
 		(dnp no)
-		(property "Reference" "TP12"
+		(property "Reference" "TP10"
 			(at 192.532 90.678 0)
 			(effects
@@
 			(project "dynafuzz"
 				(path "/b401260a-0de9-4b23-a692-63e5f9163375/5e6de810-895a-4442-a10c-7662380a0e10"
-					(reference "TP12")
+					(reference "TP10")
 					(unit 1)
 				)
@@
 		(dnp no)
 		(fields_autoplaced yes)
-		(property "Reference" "#PWR054"
+		(property "Reference" "#PWR063"
 			(at 146.05 128.27 0)
 			(effects
@@
 			(project "dynafuzz"
 				(path "/b401260a-0de9-4b23-a692-63e5f9163375/5e6de810-895a-4442-a10c-7662380a0e10"
-					(reference "#PWR054")
+					(reference "#PWR063")
 					(unit 1)
 				)
@@
 		(dnp no)
 		(fields_autoplaced yes)
-		(property "Reference" "R41"
+		(property "Reference" "R46"
 			(at 170.18 97.79 90)
 			(effects
@@
 			(project "dynafuzz"
 				(path "/b401260a-0de9-4b23-a692-63e5f9163375/5e6de810-895a-4442-a10c-7662380a0e10"
-					(reference "R41")
+					(reference "R46")
 					(unit 1)
 				)
@@
 		(dnp no)
 		(fields_autoplaced yes)
-		(property "Reference" "#PWR052"
+		(property "Reference" "#PWR061"
 			(at 134.62 128.27 0)
 			(effects
@@
 			(project "dynafuzz"
 				(path "/b401260a-0de9-4b23-a692-63e5f9163375/5e6de810-895a-4442-a10c-7662380a0e10"
-					(reference "#PWR052")
+					(reference "#PWR061")
 					(unit 1)
 				)
@@
 		(dnp no)
 		(fields_autoplaced yes)
-		(property "Reference" "#PWR055"
+		(property "Reference" "#PWR064"
 			(at 177.8 129.54 0)
 			(effects
@@
 			(project "dynafuzz"
 				(path "/b401260a-0de9-4b23-a692-63e5f9163375/5e6de810-895a-4442-a10c-7662380a0e10"
-					(reference "#PWR055")
+					(reference "#PWR064")
 					(unit 1)
 				)
@@
 		(dnp no)
 		(fields_autoplaced yes)
-		(property "Reference" "C21"
+		(property "Reference" "C23"
 			(at 134.62 74.93 90)
 			(effects
@@
 			(project "dynafuzz"
 				(path "/b401260a-0de9-4b23-a692-63e5f9163375/5e6de810-895a-4442-a10c-7662380a0e10"
-					(reference "C21")
+					(reference "C23")
 					(unit 1)
 				)
@@
 		(dnp no)
 		(fields_autoplaced yes)
-		(property "Reference" "#PWR057"
+		(property "Reference" "#PWR066"
 			(at 189.23 129.54 0)
 			(effects
@@
 			(project "dynafuzz"
 				(path "/b401260a-0de9-4b23-a692-63e5f9163375/5e6de810-895a-4442-a10c-7662380a0e10"
-					(reference "#PWR057")
+					(reference "#PWR066")
 					(unit 1)
 				)
@@
 		(dnp no)
 		(fields_autoplaced yes)
-		(property "Reference" "R37"
+		(property "Reference" "R42"
 			(at 137.16 107.9499 0)
 			(effects
@@
 			(project "dynafuzz"
 				(path "/b401260a-0de9-4b23-a692-63e5f9163375/5e6de810-895a-4442-a10c-7662380a0e10"
-					(reference "R37")
+					(reference "R42")
 					(unit 1)
 				)
@@
 		(dnp no)
 		(fields_autoplaced yes)
-		(property "Reference" "R40"
+		(property "Reference" "R45"
 			(at 148.59 113.0299 0)
 			(effects
@@
 			(project "dynafuzz"
 				(path "/b401260a-0de9-4b23-a692-63e5f9163375/5e6de810-895a-4442-a10c-7662380a0e10"
-					(reference "R40")
+					(reference "R45")
 					(unit 1)
 				)
@@
 		(dnp no)
 		(fields_autoplaced yes)
-		(property "Reference" "R36"
+		(property "Reference" "R41"
 			(at 127 96.52 90)
 			(effects
@@
 			(project "dynafuzz"
 				(path "/b401260a-0de9-4b23-a692-63e5f9163375/5e6de810-895a-4442-a10c-7662380a0e10"
-					(reference "R36")
+					(reference "R41")
 					(unit 1)
 				)
@@
 		(on_board yes)
 		(dnp no)
-		(property "Reference" "C22"
+		(property "Reference" "C24"
 			(at 135.89 87.884 90)
 			(effects
@@
 			(project "dynafuzz"
 				(path "/b401260a-0de9-4b23-a692-63e5f9163375/5e6de810-895a-4442-a10c-7662380a0e10"
-					(reference "C22")
+					(reference "C24")
 					(unit 1)
 				)
@@
 		(dnp no)
 		(fields_autoplaced yes)
-		(property "Reference" "R45"
+		(property "Reference" "R50"
 			(at 191.77 114.2999 0)
 			(effects
@@
 			(project "dynafuzz"
 				(path "/b401260a-0de9-4b23-a692-63e5f9163375/5e6de810-895a-4442-a10c-7662380a0e10"
-					(reference "R45")
+					(reference "R50")
 					(unit 1)
 				)
@@
 		(dnp no)
 		(fields_autoplaced yes)
-		(property "Reference" "C20"
+		(property "Reference" "C22"
 			(at 116.84 95.25 90)
 			(effects
@@
 			(project "dynafuzz"
 				(path "/b401260a-0de9-4b23-a692-63e5f9163375/5e6de810-895a-4442-a10c-7662380a0e10"
-					(reference "C20")
+					(reference "C22")
 					(unit 1)
 				)
@@
 		(dnp no)
 		(fields_autoplaced yes)
-		(property "Reference" "R35"
+		(property "Reference" "R40"
 			(at 107.95 113.0299 0)
 			(effects
@@
 			(project "dynafuzz"
 				(path "/b401260a-0de9-4b23-a692-63e5f9163375/5e6de810-895a-4442-a10c-7662380a0e10"
-					(reference "R35")
+					(reference "R40")
 					(unit 1)
 				)
@@
 		(on_board yes)
 		(dnp no)
-		(property "Reference" "R38"
+		(property "Reference" "R43"
 			(at 138.938 98.552 90)
 			(effects
@@
 			(project "dynafuzz"
 				(path "/b401260a-0de9-4b23-a692-63e5f9163375/5e6de810-895a-4442-a10c-7662380a0e10"
-					(reference "R38")
+					(reference "R43")
 					(unit 1)
 				)
@@
 		(dnp no)
 		(fields_autoplaced yes)
-		(property "Reference" "C24"
+		(property "Reference" "C26"
 			(at 177.8 76.2 90)
 			(effects
@@
 			(project "dynafuzz"
 				(path "/b401260a-0de9-4b23-a692-63e5f9163375/5e6de810-895a-4442-a10c-7662380a0e10"
-					(reference "C24")
+					(reference "C26")
 					(unit 1)
 				)
@@
 		(on_board yes)
 		(dnp no)
-		(property "Reference" "R43"
+		(property "Reference" "R48"
 			(at 182.118 99.822 90)
 			(effects
@@
 			(project "dynafuzz"
 				(path "/b401260a-0de9-4b23-a692-63e5f9163375/5e6de810-895a-4442-a10c-7662380a0e10"
-					(reference "R43")
+					(reference "R48")
 					(unit 1)
 				)
@@
 		(dnp no)
 		(fields_autoplaced yes)
-		(property "Reference" "C23"
+		(property "Reference" "C25"
 			(at 160.02 96.52 90)
 			(effects
@@
 			(project "dynafuzz"
 				(path "/b401260a-0de9-4b23-a692-63e5f9163375/5e6de810-895a-4442-a10c-7662380a0e10"
-					(reference "C23")
+					(reference "C25")
 					(unit 1)
 				)
@@
 		(dnp no)
 		(fields_autoplaced yes)
-		(property "Reference" "R39"
+		(property "Reference" "R44"
 			(at 148.59 71.1199 0)
 			(effects
@@
 			(project "dynafuzz"
 				(path "/b401260a-0de9-4b23-a692-63e5f9163375/5e6de810-895a-4442-a10c-7662380a0e10"
-					(reference "R39")
+					(reference "R44")
 					(unit 1)
 				)
@@
 		(dnp no)
 		(fields_autoplaced yes)
-		(property "Reference" "R44"
+		(property "Reference" "R49"
 			(at 191.77 72.3899 0)
 			(effects
@@
 			(project "dynafuzz"
 				(path "/b401260a-0de9-4b23-a692-63e5f9163375/5e6de810-895a-4442-a10c-7662380a0e10"
-					(reference "R44")
+					(reference "R49")
 					(unit 1)
 				)
@@
 		(dnp no)
 		(fields_autoplaced yes)
-		(property "Reference" "#PWR051"
+		(property "Reference" "#PWR060"
 			(at 105.41 127 0)
 			(effects
@@
 			(project "dynafuzz"
 				(path "/b401260a-0de9-4b23-a692-63e5f9163375/5e6de810-895a-4442-a10c-7662380a0e10"
-					(reference "#PWR051")
+					(reference "#PWR060")
 					(unit 1)
 				)
@@
 		(on_board yes)
 		(dnp no)
-		(property "Reference" "C25"
+		(property "Reference" "C27"
 			(at 179.07 89.154 90)
 			(effects
@@
 			(project "dynafuzz"
 				(path "/b401260a-0de9-4b23-a692-63e5f9163375/5e6de810-895a-4442-a10c-7662380a0e10"
-					(reference "C25")
+					(reference "C27")
 					(unit 1)
 				)
@@
 		(dnp no)
 		(fields_autoplaced yes)
-		(property "Reference" "#PWR056"
+		(property "Reference" "#PWR065"
 			(at 189.23 71.12 0)
 			(effects
@@
 			(project "dynafuzz"
 				(path "/b401260a-0de9-4b23-a692-63e5f9163375/5e6de810-895a-4442-a10c-7662380a0e10"
-					(reference "#PWR056")
+					(reference "#PWR065")
 					(unit 1)
 				)
@@
 		(dnp no)
 		(fields_autoplaced yes)
-		(property "Reference" "#PWR053"
+		(property "Reference" "#PWR062"
 			(at 146.05 69.85 0)
 			(effects
@@
 			(project "dynafuzz"
 				(path "/b401260a-0de9-4b23-a692-63e5f9163375/5e6de810-895a-4442-a10c-7662380a0e10"
-					(reference "#PWR053")
+					(reference "#PWR062")
 					(unit 1)
 				)
@@
 		(dnp no)
 		(fields_autoplaced yes)
-		(property "Reference" "R42"
+		(property "Reference" "R47"
 			(at 180.34 109.2199 0)
 			(effects
@@
 			(project "dynafuzz"
 				(path "/b401260a-0de9-4b23-a692-63e5f9163375/5e6de810-895a-4442-a10c-7662380a0e10"
-					(reference "R42")
+					(reference "R47")
 					(unit 1)
 				)
@@
 		(on_board yes)
 		(dnp no)
-		(property "Reference" "TP11"
+		(property "Reference" "TP9"
 			(at 149.352 93.218 0)
 			(effects
@@
 			(project "dynafuzz"
 				(path "/b401260a-0de9-4b23-a692-63e5f9163375/5e6de810-895a-4442-a10c-7662380a0e10"
-					(reference "TP11")
-					(unit 1)
-				)
+					(reference "TP9")
+					(unit 1)
+				)
