File: dist/dynafuzz/vca.kicad_sch (KiCad schematic)
At the start: 12 parts, among them U2 TL074

Commit message: schematic for dynafuzz
Parts:
- renumbered R35 to R28, R34 to R29, R23 to R30, R28 to R31, R29 to R32, R30 to R34, R31 to R35, R32 to R36, U2 to U1, U1 to U2
Changed lines of the file:
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@@
 		(dnp no)
 		(fields_autoplaced yes)
-		(property "Reference" "U1"
+		(property "Reference" "U2"
 			(at 111.76 97.7899 0)
 			(effects
@@
 			(project "dynafuzz"
 				(path "/b401260a-0de9-4b23-a692-63e5f9163375/f1f48dbc-08ba-440b-8310-6ec9ab55161d"
-					(reference "U1")
+					(reference "U2")
 					(unit 2)
 				)
@@
 		(dnp no)
 		(fields_autoplaced yes)
-		(property "Reference" "U1"
+		(property "Reference" "U2"
 			(at 104.14 97.7899 0)
 			(effects
@@
 			(project "dynafuzz"
 				(path "/b401260a-0de9-4b23-a692-63e5f9163375/f1f48dbc-08ba-440b-8310-6ec9ab55161d"
-					(reference "U1")
+					(reference "U2")
 					(unit 1)
 				)
@@
 		(dnp no)
 		(fields_autoplaced yes)
-		(property "Reference" "U2"
+		(property "Reference" "U1"
 			(at 173.99 69.85 0)
 			(effects
@@
 			(project "dynafuzz"
 				(path "/b401260a-0de9-4b23-a692-63e5f9163375/f1f48dbc-08ba-440b-8310-6ec9ab55161d"
-					(reference "U2")
+					(reference "U1")
 					(unit 1)
 				)
@@
 		(dnp no)
 		(fields_autoplaced yes)
-		(property "Reference" "R29"
+		(property "Reference" "R32"
 			(at 104.14 85.0899 0)
 			(effects
@@
 			(project "dynafuzz"
 				(path "/b401260a-0de9-4b23-a692-63e5f9163375/f1f48dbc-08ba-440b-8310-6ec9ab55161d"
-					(reference "R29")
+					(reference "R32")
 					(unit 1)
 				)
@@
 		(dnp no)
 		(fields_autoplaced yes)
-		(property "Reference" "R35"
+		(property "Reference" "R28"
 			(at 74.93 114.2999 0)
 			(effects
@@
 			(project "dynafuzz"
 				(path "/b401260a-0de9-4b23-a692-63e5f9163375/f1f48dbc-08ba-440b-8310-6ec9ab55161d"
-					(reference "R35")
+					(reference "R28")
 					(unit 1)
 				)
@@
 		(dnp no)
 		(fields_autoplaced yes)
-		(property "Reference" "R30"
+		(property "Reference" "R34"
 			(at 116.84 85.0899 0)
 			(effects
@@
 			(project "dynafuzz"
 				(path "/b401260a-0de9-4b23-a692-63e5f9163375/f1f48dbc-08ba-440b-8310-6ec9ab55161d"
-					(reference "R30")
+					(reference "R34")
 					(unit 1)
 				)
@@
 		(dnp no)
 		(fields_autoplaced yes)
-		(property "Reference" "R34"
+		(property "Reference" "R29"
 			(at 82.55 116.84 90)
 			(effects
@@
 			(project "dynafuzz"
 				(path "/b401260a-0de9-4b23-a692-63e5f9163375/f1f48dbc-08ba-440b-8310-6ec9ab55161d"
-					(reference "R34")
+					(reference "R29")
 					(unit 1)
 				)
@@
 		(dnp no)
 		(fields_autoplaced yes)
-		(property "Reference" "R28"
+		(property "Reference" "R31"
 			(at 92.71 106.6799 0)
 			(effects
@@
 			(project "dynafuzz"
 				(path "/b401260a-0de9-4b23-a692-63e5f9163375/f1f48dbc-08ba-440b-8310-6ec9ab55161d"
-					(reference "R28")
+					(reference "R31")
 					(unit 1)
 				)
@@
 		(on_board yes)
 		(dnp no)
-		(property "Reference" "U2"
+		(property "Reference" "U1"
 			(at 82.55 140.97 0)
 			(effects
@@
 			(project "dynafuzz"
 				(path "/b401260a-0de9-4b23-a692-63e5f9163375/f1f48dbc-08ba-440b-8310-6ec9ab55161d"
-					(reference "U2")
+					(reference "U1")
 					(unit 2)
 				)
@@
 		(dnp no)
 		(fields_autoplaced yes)
-		(property "Reference" "R23"
+		(property "Reference" "R30"
 			(at 83.82 92.71 90)
 			(effects
@@
 			(project "dynafuzz"
 				(path "/b401260a-0de9-4b23-a692-63e5f9163375/f1f48dbc-08ba-440b-8310-6ec9ab55161d"
-					(reference "R23")
+					(reference "R30")
 					(unit 1)
 				)
@@
 		(dnp no)
 		(fields_autoplaced yes)
-		(property "Reference" "R31"
+		(property "Reference" "R35"
 			(at 128.27 106.6799 0)
 			(effects
@@
 			(project "dynafuzz"
 				(path "/b401260a-0de9-4b23-a692-63e5f9163375/f1f48dbc-08ba-440b-8310-6ec9ab55161d"
-					(reference "R31")
+					(reference "R35")
 					(unit 1)
 				)
@@
 		(dnp no)
 		(fields_autoplaced yes)
-		(property "Reference" "R32"
+		(property "Reference" "R36"
 			(at 133.35 92.71 90)
 			(effects
@@
 			(project "dynafuzz"
 				(path "/b401260a-0de9-4b23-a692-63e5f9163375/f1f48dbc-08ba-440b-8310-6ec9ab55161d"
-					(reference "R32")
-					(unit 1)
-				)
+					(reference "R36")
+					(unit 1)
+				)

Commit message: add vca envelope detector to dynafuzz
Parts:
- removed R35: 100, symbol Device:R
- removed R36: 100k, symbol Device:R
- removed RV6: R_INTENSITY_B100K, symbol Device:R_Potentiometer_Trim
- removed unit 1 of U1
- removed U2: ~, symbol _project:DMMT5551
- added C19: 100n, Capacitor_SMD:C_0805_2012Metric, symbol Device:C
- added D2: D, Diode_SMD:D_0805_2012Metric, symbol Device:D
- added Q6, Q7: DMMT5401, Package_TO_SOT_SMD:SOT-23-6, symbol Transistor_BJT:DMMT5401
- added R21: 15k, Resistor_SMD:R_0805_2012Metric, symbol Device:R
- added R22, R23, R24, R25: 100k, Resistor_SMD:R_0805_2012Metric, symbol Device:R
- added R26, R27: 220k, Resistor_SMD:R_0805_2012Metric, symbol Device:R
- added RV5: 1M, _effects_shared_footprints:Potentiometer_Alpha_RD901F-40-00D_Single_Vertical, symbol Device:R_Potentiometer
- added TP10, TP7, TP8, TP9: ~, TestPoint:TestPoint_Pad_D1.5mm, symbol Connector:TestPoint
- added unit 4 of U1
- added unit 3 of U1
- added U5: LM13700, Package_SO:SOIC-16_3.9x9.9mm_P1.27mm, symbol Amplifier_Operational:LM13700
- R28: value 100 -> 1k; footprint (none) -> Resistor_SMD:R_0805_2012Metric
- R29: value 100k -> 1k; footprint (none) -> Resistor_SMD:R_0805_2012Metric
- R30: value 100k -> 10k; footprint (none) -> Resistor_SMD:R_0805_2012Metric
- R31, R33: value 100 -> 10k; footprint (none) -> Resistor_SMD:R_0805_2012Metric
- R32: footprint (none) -> Resistor_SMD:R_0805_2012Metric
- R34: value 10k -> R; footprint (none) -> Resistor_SMD:R_0805_2012Metric
- U1: footprint (none) -> Package_SO:SSOP-14_5.3x6.2mm_P0.65mm
Connections:
- net +9V: now also Q6.5 (E2), Q6.6 (E1), Q7.5 (E2), Q7.6 (E1); no longer R32.2, R34.2
- net -9V: now also R24.2
- net GND: now also R28.1, R29.1, C19.2, U1.10 (+), U1.12 (+), U5.14 (+), U5.3 (+); no longer R31.1
- net at R34.1: now also R32.2, R33.2, U1.9 (-)
- net at R32.1: now also U5.12
- net at R30.2: now also Q6.1 (C1), Q6.2 (B1), Q6.3 (B2); no longer R31.2
- net at R28.2: now also R26.1, TP9.1, U5.13 (-)
- net at R30.1: now also U1.7, R23.1, RV5.3, TP7.1
- new net: Q6.4 (C2), U5.16
- new net: Q7.1 (C1), Q7.2 (B1), Q7.3 (B2), R31.2
- new net: C19.1, D2.2 (A), R21.1
- new net: R22.2, RV5.1, RV5.2
- new net: R23.2, R24.1, R25.1, U1.13 (-)
- new net: R25.2, R31.1, TP8.1, U1.14
- new net: R33.1, U5.5
- new net: R21.2, R22.1, U1.6 (-)
- new net: Q7.4 (C2), U5.1
- new net: R27.1, R29.2, TP10.1, U5.4 (-)
- new net IN: D2.1 (K)
- new net OUT: R34.2, U1.8
- new net SIG_A: R26.2
- new net SIG_B: R27.2
- no-connect marks 0 -> 2
Other:
- note added: "$ 1 0.000005 10.20027730826997 50 5 43 5e-11 402 368 160 496 160 1 0\s0\s40\s-9\s0\s0\s0.5 0\s0\s40\s9\s0\s0\s0.5 0\s1\s-7.187713922398314\s0.6093586845133121\s100\sdefault 0\s1\s-0.6093586845133121\s0.6091038549858805\s100\sdefault 0\s1\s0\s0.6091038549858805\s100\sdefault 0\s1\s-7.812617894357531\s0.5938235381024933\s100\sdefault 0\s1\s-7.829429532678426\s0.5882196586326172\s100\sdefault 0\s-1\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"
- note added: "1Hz << RC (~10Hz) << 100Hz"
- note added: "TODO: orientation TODO: what gain range?"
- note added: "TODO: pot here?"
- note added: "TODO: what makeup gain is required?"
- note added: "TODO: what's the peak voltage?"
- note added: "current mirror"
- note added: "dual VCA"
- note added: "envelope detector"
- note added: "gain: 6.6 to 73.3 at 100mV, output -> 660mV to 7.33V"
- note added: "invert diode to counter inverting amp"
- note added: "inverting summing amp in: 0..9 out=-1*(in+-9) out: 9..0"
- note added: "output: 0V (in=silent) to 9V (in=loud)"
- note added: "protect ota by limiting to 2mA 18V/2mA=9kohm"
- note added: "summing amp with makeup gain"
- note removed: "TODO: values"

Commit message: start layout
Parts:
- RV5: value 1M -> R_THRESHOLD_B1M
- U1: footprint Package_SO:SSOP-14_5.3x6.2mm_P0.65mm -> Package_SO:SOIC-14_3.9x8.7mm_P1.27mm
Connections:
- net OUT: now also U1.14; no longer U1.8
- net at R23.2, R24.1, R25.1: now also U1.9 (-); no longer U1.13 (-)
- net at R25.2, R31.1, TP8.1: now also U1.8; no longer U1.14
- net at R32.2, R33.2, R34.1: now also U1.13 (-); no longer U1.9 (-)
- net +9V renamed +7.5V
- net -9V renamed -7.5V
Other:
- moved on the sheet: U1C, U1D

Commit message: updates
Parts:
- removed R21: 15k, Resistor_SMD:R_0805_2012Metric, symbol Device:R
- removed TP10, TP9: ~, TestPoint:TestPoint_Pad_D1.5mm, symbol Connector:TestPoint
- added C18: 1u, symbol Device:C
- added C19, C20, C21: 100n, Capacitor_SMD:C_0805_2012Metric, symbol Device:C
- added R23, R24, R27: 100k, Resistor_SMD:R_0805_2012Metric, symbol Device:R
- added RV10: R_BLEND_B100K, symbol Device:R_Potentiometer_Dual_Separate
- added RV5: RTRIM_ENVELOPE_50K, symbol Device:R_Potentiometer_Trim
- added RV7: R_RELEASE_B1M, _effects_shared_footprints:Potentiometer_Alpha_RD901F-40-00D_Single_Vertical, symbol Device:R_Potentiometer
- added RV8: R_BLEND_B10K, _effects_shared_footprints:Potentiometer_Alpha_RD901F-40-00D_Single_Vertical, symbol Device:R_Potentiometer
- added U4: TL074, Package_SO:SOIC-14_3.9x8.7mm_P1.27mm, symbol Amplifier_Operational:TL074
- added unit 1 of U5
- added unit 5 of U5
- added unit 2 of U6
- added unit 5 of U6
- added unit 4 of U6
- C17: renamed from C19; value 100n -> 1u
- R22: value 100k -> 1k
- R35: renamed from R32; value 10k -> 15k
- R36: renamed from R33; value 10k -> 15k
- R39: renamed from R34; value R -> 100k
- renumbered R23 to R25, R24 to R26, R25 to R28, R26 to R29, R27 to R30, R30 to R31, R28 to R32, R29 to R33, R31 to R34, RV5 to RV6, U1 to U5, U5 to U6
Connections:
- net IN is gone; now on an unnamed net: D2.1 (K)
- net +7.5V: now also C19.1, C20.1, C21.1, U4.4 (V+), U5.4 (V+), U6.11 (V+)
- net -7.5V: now also C19.2, C20.2, C21.2, RV8.3, U4.11 (V-), U5.11 (V-), U6.6 (V-)
- net GND: now also R35.1, R36.2, C18.2, RV8.1, U4.12 (+), U5.3 (+); no longer U5.10 (+)
- net OUT: now also U4.14; no longer U5.14
- net at C17.1: now also RV5.1, RV5.2; no longer D2.2 (A)
- net at RV6.1, RV6.2: now also U5.6 (-), RV5.3; no longer R22.2
- net at R25.1, R31.1, TP7.1: now also R27.2, U5.1; no longer RV6.3, U5.7
- net at R25.2, R26.1, R28.1: now also U5.13 (-); no longer U5.9 (-)
- net at R28.2, R34.1, TP8.1: now also U5.14; no longer U5.8
- net at R36.1, U6.5: now also U4.5 (+)
- net at R22.1: now also U5.10 (+), C18.1; no longer U5.6 (-)
- net at U6.12: now also R35.2, U4.3 (+); no longer R35.1
- new net: R22.2, RV7.1
- new net: R23.2, R24.2, R27.1, U5.2 (-)
- new net: RV10.4, U4.6 (-), U4.7
- new net: R23.1, U5.8, U5.9 (-)
- new net: D2.2 (A), U4.8, U4.9 (-)
- new net: R39.1, RV10.3, RV10.5, RV10.6, U4.13 (-)
- new net: RV6.3, RV7.2, RV7.3, U5.7
- new net: R24.1, RV8.2
- new net: RV10.1, RV10.2, U4.1, U4.2 (-)
- new net TRIGGER: U4.10 (+)
- no-connect marks 2 -> 6
Other:
- note added: "15k -> gain ~= 1"
- note added: "Could have center detent"
- note added: "Threshold controls the maximum amount of signal B on trigger Release controls how quickly the signal returns to A Blend controls how much of B there is with no trigger"
- note added: "VCA"
- note added: "buffer converts current to voltage"
- note added: "cutoff 144Hz - 144mHz (6.9ms to 6.9s)"
- note added: "lowpass filter"
- note added: "nominal Iabc ~= 0 to 0.8mA"
- note added: "out= -1*(in + -Vcc) input: 0V .. +Vcc output: +Vcc .. 0V"
- note added: "out=-1*(in+offset) in: 0 .. -Vcc out: 0 .. Vcc"
- note added: "output: 0V (in=silent) to -Vcc (in=loud)"
- note added: "protect ota by limiting to 2mA 15V/10kohm=1.5mA"
- note added: "summing amp"
- note removed: "1Hz << RC (~10Hz) << 100Hz"
- note removed: "TODO: pot here?"
- note removed: "TODO: what makeup gain is required?"
- note removed: "TODO: what's the peak voltage?"
- note removed: "dual VCA"
- note removed: "gain: 6.6 to 73.3 at 100mV, output -> 660mV to 7.33V"
- note removed: "invert diode to counter inverting amp"
- note removed: "inverting summing amp in: 0..9 out=-1*(in+-9) out: 9..0"
- note removed: "output: 0V (in=silent) to 9V (in=loud)"
- note removed: "protect ota by limiting to 2mA 18V/2mA=9kohm"
- note removed: "summing amp with makeup gain"
- moved on the sheet: C17, D2, Q6A, Q6B, Q7A, Q7B, R25, R26, R28, R29, R30, R31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
