File: dist/buzz/buzz.kicad_pcb (KiCad board)
At the start: 2 copper layers, 58.4 x 85.1 mm, 61 parts, among them J1 AudioJack_IN, J2 AudioJack_OUT, J3 Jack-DC, J4 MAIN_BIC, J5 SWITCH_BIC, Q1 Q_NPN, Q2 Q_NPN, Q3 Q_NPN, Q4 Q_NPN, SW1 SW_3PDT_x3

Commit message: update design
Parts:
- R19: value 3.3k -> 1k
- RV2: value R_MID-B25K -> R_MID-A100K
- moved RV2 12.5 mm to (182.6, 67.9), turned to -90 degrees
- moved RV3 12.5 mm to (142.5, 67.9), turned to -90 degrees
- moved D5 0.25 mm to (158.8, 108.7)
Routing:
- net Net-(C10-Pad1): track 52.3 -> 61.3 mm, vias 0 -> 1
- net Net-(C11-Pad1): track 35.1 -> 44.0 mm, vias 0 -> 1
- net Net-(R19-Pad1): track 14.3 -> 20.0 mm
- net Net-(D1-K): track 17.4 -> 20.7 mm
- net Net-(C12-Pad2): track 25.9 -> 27.8 mm
- net Net-(C3-Pad2): track 22.6 -> 23.6 mm
- net Net-(D3-A): track 64.0 -> 63.1 mm
- net Net-(D1-A): track 49.8 -> 49.1 mm
Other:
- board text added: "${REFERENCE}"
- board text added: "BUZZ FUZZ Rev C 2026-09-28"
- board text removed: "FUZZ Rev B 2026-08-25"

Commit message: design case
Routing:
- net Net-(Q1-B): track 49.2 -> 53.3 mm
- net Net-(C4-Pad1): track 10.8 -> 12.1 mm
- net Net-(C12-Pad2): track 27.8 -> 28.5 mm
Changed lines of the file:
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@@
 		)
 		(fill no)
-		(locked yes)
 		(layer "User.2")
 	)
@@
 		)
 		(fill no)
-		(locked yes)
 		(layer "User.2")
 	)
@@
 		)
 		(fill no)
-		(locked yes)
 		(layer "User.2")
 	)
@@
 		)
 		(fill no)
-		(locked yes)
 		(layer "User.2")
 	)
@@
 		)
 		(fill no)
-		(locked yes)
 		(layer "User.2")
 	)
@@
 		)
 		(fill no)
-		(locked yes)
 		(layer "User.2")
 	)
@@
 	)
 	(gr_text "${REFERENCE}"
+		(at 160.249 88.875 0)
+		(layer "B.Fab")
+		(effects
+			(font
+				(size 1 1)
+				(thickness 0.15)
+			)
+			(justify mirror)
+		)
+	)
+	(gr_text "${REFERENCE}"
 		(at 157.754 52.603 0)
 		(layer "B.Fab")
@@
 		)
 	)
-	(gr_text "${REFERENCE}"
-		(at 160.249 88.875 0)
-		(layer "B.Fab")
-		(effects
-			(font
-				(size 1 1)
-				(thickness 0.15)
-			)
-			(justify mirror)
-		)
-	)
 	(segment
 		(start 162.56 95.533)
@@
 	(segment
 		(start 162.56 104.608)
-		(end 175.728 91.44)
+		(end 162.56 103.47663)
 		(width 0.2)
 		(layer "B.Cu")
@@
 	)
 	(segment
-		(start 180.33514 91.44)
-		(end 182.372 89.40314)
+		(start 182.372 88.999)
+		(end 182.372 88.392)
 		(width 0.2)
 		(layer "B.Cu")
@@
 	)
 	(segment
+		(start 158.496 97.79)
+		(end 162.56 101.854)
+		(width 0.2)
+		(layer "B.Cu")
+		(net 2)
+	)
+	(segment
+		(start 162.56 101.854)
+		(end 162.56 104.608)
+		(width 0.2)
+		(layer "B.Cu")
+		(net 2)
+	)
+	(segment
+		(start 173.014 104.608)
+		(end 180.086 97.536)
+		(width 0.2)
+		(layer "B.Cu")
+		(net 2)
+	)
+	(segment
+		(start 180.086 91.285)
+		(end 182.372 88.999)
+		(width 0.2)
+		(layer "B.Cu")
+		(net 2)
+	)
+	(segment
+		(start 158.496 95.983)
+		(end 158.496 97.79)
+		(width 0.2)
+		(layer "B.Cu")
+		(net 2)
+	)
+	(segment
 		(start 162.56 104.608)
-		(end 162.56 103.47663)
-		(width 0.2)
-		(layer "B.Cu")
-		(net 2)
-	)
-	(segment
-		(start 182.372 89.40314)
-		(end 182.372 88.392)
-		(width 0.2)
-		(layer "B.Cu")
-		(net 2)
-	)
-	(segment
-		(start 158.496 99.41263)
-		(end 158.496 95.533)
+		(end 173.014 104.608)
 		(width 0.2)
 		(layer "B.Cu")
@@
 	)
 	(segment
-		(start 162.56 103.47663)
-		(end 158.496 99.41263)
-		(width 0.2)
-		(layer "B.Cu")
-		(net 2)
-	)
-	(segment
 		(start 182.372 83.86)
 		(end 182.92 83.312)
@@
 	)
 	(segment
-		(start 175.728 91.44)
-		(end 180.33514 91.44)
+		(start 180.086 97.536)
+		(end 180.086 91.285)
 		(width 0.2)
 		(layer "B.Cu")
@@
 	)
 	(segment
-		(start 174.324 58.246)
-		(end 171.704 58.246)
+		(start 173.736 60.452)
+		(end 178.562 60.452)
 		(width 0.2)
 		(layer "F.Cu")
@@
 	)
 	(segment
-		(start 180.086 64.008)
-		(end 174.324 58.246)
+		(start 171.704 58.42)
+		(end 173.736 60.452)
+		(width 0.2)
+		(layer "F.Cu")
+		(net 5)
+	)
+	(segment
+		(start 171.704 58.246)
+		(end 171.704 58.42)
+		(width 0.2)
+		(layer "F.Cu")
+		(net 5)
+	)
+	(segment
+		(start 178.562 60.452)
+		(end 180.086 61.976)
+		(width 0.2)
+		(layer "F.Cu")
+		(net 5)
+	)
+	(segment
+		(start 180.086 61.976)
+		(end 180.086 64.008)
 		(width 0.2)
 		(layer "F.Cu")
@@
 	)
 	(segment
-		(start 138.684 70.866)
+		(start 137.735 71.815)
 		(end 139.954 69.596)
-		(width 0.2)
-		(layer "F.Cu")
-		(net 18)
-	)
-	(segment
-		(start 136.271 70.866)
-		(end 138.684 70.866)
 		(width 0.2)
 		(layer "F.Cu")
@@
 	)
 	(segment
+		(start 132.08 78.994)
+		(end 135.703 78.994)
+		(width 0.2)
+		(layer "F.Cu")
+		(net 18)
+	)
+	(segment
+		(start 135.703 78.994)
+		(end 137.735 76.962)
+		(width 0.2)
+		(layer "F.Cu")
+		(net 18)
+	)
+	(segment
 		(start 134.62 87.924)
 		(end 134.62 81.534)
@@
 	)
 	(segment
-		(start 132.08 78.994)
-		(end 132.08 75.057)
-		(width 0.2)
-		(layer "F.Cu")
-		(net 18)
-	)
-	(segment
-		(start 132.08 75.057)
-		(end 136.271 70.866)
+		(start 137.735 76.962)
+		(end 137.735 71.815)
 		(width 0.2)
 		(layer "F.Cu")
@@
 		)
 	)
-	(group ""
-		(locked yes)
-		(members "3924f57c-b956-44bd-a275-67d66372c951" "4c3cdf65-66ea-4cbd-bdf4-72278aade1e0"
-			"907d15ea-9af6-4849-aa90-614dd7c3862d" "a20400a8-9908-4db4-8b04-9702ccc3e621"
-			"de8e3bbd-8448-4a0b-8ddf-a68f31c0dd4f" "e1dea3cd-961a-449a-9c00-2de1801d6064"
-		)
-	)
