File: dist/buzz/buzz.kicad_pcb (KiCad board)
At the start: 2 copper layers, 58.4 x 85.1 mm, 61 parts, among them J1 AudioJack_IN, J2 AudioJack_OUT, J3 Jack-DC, J4 MAIN_BIC, J5 SWITCH_BIC, Q1 Q_NPN, Q2 Q_NPN, Q3 Q_NPN, Q4 Q_NPN, SW1 SW_3PDT_x3

Commit message: rev D
Parts:
- C12: value 100n -> 1u
- R18: value 3.3k -> 10k
- moved TP2 8.89 mm to (159.8, 55.6)
- moved R6 7.25 mm to (164.6, 54.4), turned to 180 degrees
- moved C14 4.84 mm to (168.4, 53.3)
- moved R1 2.09 mm to (162.6, 95.5), turned to 90 degrees
Connections:
- R1 pad 1: IN -> Net-(C1-Pad1)
- R1 pad 2: Net-(C1-Pad1) -> IN
- RV2 pad 1: Net-(C10-Pad1) -> Net-(R19-Pad1)
- RV2 pad 3: Net-(R19-Pad1) -> Net-(C10-Pad1)
Routing:
- net Net-(D1-A): track 49.1 -> 41.3 mm
- net +9V: track 83.7 -> 90.3 mm
- net Net-(C10-Pad1): track 61.3 -> 58.8 mm
- net Net-(R19-Pad1): track 20.0 -> 22.1 mm
- net Net-(R6-Pad1): track 16.1 -> 17.0 mm
Other:
- board text added: "BUZZ FUZZ Rev D 2026-10-20"
- board text removed: "BUZZ FUZZ Rev C 2026-09-28"

Commit message: fix some drc issues
Routing:
- net Net-(D1-A): track 41.3 -> 54.5 mm
- net Net-(Q1-B): track 53.3 -> 51.6 mm
Other:
- board text removed: "${REFERENCE}"
Changed lines of the file:
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@@
 	)
 	(gr_text "+"
-		(at 161.29 110.236 0)
+		(at 161.544 110.49 0)
 		(layer "F.SilkS")
 		(effects
@@
 		)
 	)
-	(gr_text "${REFERENCE}"
-		(at 160.249 88.875 0)
-		(layer "B.Fab")
-		(effects
-			(font
-				(size 1 1)
-				(thickness 0.15)
-			)
-			(justify mirror)
-		)
-	)
-	(gr_text "${REFERENCE}"
-		(at 157.754 52.603 0)
-		(layer "B.Fab")
-		(effects
-			(font
-				(size 1 1)
-				(thickness 0.15)
-			)
-			(justify mirror)
-		)
-	)
 	(segment
 		(start 162.56 95.533)
@@
 	)
 	(segment
-		(start 162.56 104.608)
-		(end 162.56 103.47663)
-		(width 0.2)
-		(layer "B.Cu")
-		(net 2)
-	)
-	(segment
-		(start 182.372 88.999)
-		(end 182.372 88.392)
-		(width 0.2)
-		(layer "B.Cu")
-		(net 2)
-	)
-	(segment
 		(start 158.496 97.79)
 		(end 162.56 101.854)
@@
 	)
 	(segment
-		(start 171.704 58.246)
-		(end 171.704 58.42)
-		(width 0.2)
-		(layer "F.Cu")
-		(net 5)
-	)
-	(segment
 		(start 178.562 60.452)
 		(end 180.086 61.976)
@@
 	)
 	(segment
+		(start 159.004 54.864)
+		(end 159.766 55.626)
+		(width 0.2)
+		(layer "F.Cu")
+		(net 9)
+	)
+	(segment
+		(start 151.718 54.864)
+		(end 159.004 54.864)
+		(width 0.2)
+		(layer "F.Cu")
+		(net 9)
+	)
+	(segment
 		(start 163.068 78.994)
 		(end 163.068 75.779)
+		(width 0.2)
+		(layer "F.Cu")
+		(net 9)
+	)
+	(segment
+		(start 148.336 58.246)
+		(end 151.718 54.864)
 		(width 0.2)
 		(layer "F.Cu")
@@
 	)
 	(segment
-		(start 172.747 72.771)
-		(end 171.958 72.771)
-		(width 0.2)
-		(layer "B.Cu")
-		(net 14)
-	)
-	(segment
-		(start 171.958 72.771)
-		(end 140.081 72.771)
+		(start 140.081 72.771)
+		(end 172.747 72.771)
 		(width 0.2)
 		(layer "B.Cu")
@@
 	)
 	(segment
-		(start 168.344 53.34)
-		(end 168.442 53.34)
-		(width 0.4)
-		(layer "F.Cu")
-		(net 21)
-	)
-	(segment
 		(start 160.732 87.122)
 		(end 160.249 87.605)
@@
 		(start 158.75 108.712)
 		(end 158.75 104.844)
-		(width 0.4)
-		(layer "F.Cu")
-		(net 22)
-	)
-	(segment
-		(start 158.75 104.844)
-		(end 158.496 104.59)
 		(width 0.4)
 		(layer "F.Cu")
@@
 		(layers "F.Cu" "B.Cu")
 		(hatch edge 0.5)
-		(connect_pads
+		(connect_pads yes
 			(clearance 0.25)
 		)
