File: dist/buzz/buzz.kicad_sch (KiCad schematic)
At the start: 61 parts, among them J1 AudioJack_IN, J2 AudioJack_OUT, J3 Jack-DC, J4 MAIN_BIC, J5 SWITCH_BIC, Q1 Q_NPN, Q2 Q_NPN, Q3 Q_NPN, Q4 Q_NPN, SW1 SW_3PDT_x3

Commit message: update design
Parts:
- R19: value 3.3k -> 1k
- RV2: value R_MID-B25K -> R_MID-A100K
Connections:
- no-connect marks 2 -> 4
Other:
- removed sheet deviever
- removed sheet vca
- note added: "A or B taper A preferred"
- note added: "HOOF Tone Stack - modified values at tone even (45%), mids go from huge scoop at 3kHz to slight boost phase flat"
- note added: "scoop happens when MID is short 0% - R=0 - super scoop 50% - R=~15k - small scoop 80% - R=~30k - flat EQ 100% - R=100k - slight mid boost"
- note removed: "HOOF Tone Stack"
Changed lines of the file:
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@@
 	(generator_version "9.0")
 	(paper "A4")
-	(text "HOOF Tone Stack"
+	(text "scoop happens when MID is short\n0% - R=0 - super scoop\n50% - R=~15k - small scoop\n80% - R=~30k - flat EQ\n100% - R=100k - slight mid boost"
 		(exclude_from_sim no)
-		(at 198.12 143.764 0)
+		(at 199.39 78.74 0)
+		(effects
+			(font
+				(size 1.27 1.27)
+			)
+		)
+	)
+	(text "A or B taper\nA preferred"
+		(exclude_from_sim no)
+		(at 190.5 90.17 0)
+		(effects
+			(font
+				(size 1.27 1.27)
+			)
+		)
+	)
+	(text "HOOF Tone Stack - modified values\n\nat tone even (45%),\nmids go from huge scoop at 3kHz to slight boost\nphase flat"
+		(exclude_from_sim no)
+		(at 186.69 148.59 0)
 		(effects
 			(font
@@
 	)
 	(no_connect
+		(at 33.02 166.37)
+	)
+	(no_connect
+		(at 33.02 163.83)
+	)
+	(no_connect
 		(at 149.86 184.15)
 	)
@@
 			)
 		)
-		(property "Value" "3.3k"
+		(property "Value" "1k"
 			(at 208.026 93.726 90)
 			(effects
@@
 			)
 		)
-		(property "Value" "R_MID-B25K"
+		(property "Value" "R_MID-A100K"
 			(at 198.12 93.9801 0)
 			(effects
@@
 				)
 			)
-		)
-	)
-	(sheet
-		(at 5.715 -36.195)
-		(size 31.115 20.955)
-		(exclude_from_sim no)
-		(in_bom no)
-		(on_board no)
-		(dnp no)
-		(fields_autoplaced yes)
-		(stroke
-			(width 0.1524)
-			(type solid)
-		)
-		(fill
-			(color 0 0 0 0.0000)
-		)
-		(property "Sheetname" "deviever"
-			(at 5.715 -36.9066 0)
-			(effects
-				(font
-					(size 1.27 1.27)
-				)
-				(justify left bottom)
-			)
-		)
-		(property "Sheetfile" "deviever.kicad_sch"
-			(at 5.715 -14.6554 0)
-			(effects
-				(font
-					(size 1.27 1.27)
-				)
-				(justify left top)
-			)
-		)
-		(instances
-			(project "dynafuzz"
-				(path "/b401260a-0de9-4b23-a692-63e5f9163375"
-					(page "2")
-				)
-			)
-		)
-	)
-	(sheet
-		(at 48.26 -36.83)
-		(size 33.02 25.4)
-		(exclude_from_sim no)
-		(in_bom no)
-		(on_board no)
-		(dnp no)
-		(fields_autoplaced yes)
-		(stroke
-			(width 0.1524)
-			(type solid)
-		)
-		(fill
-			(color 0 0 0 0.0000)
-		)
-		(property "Sheetname" "vca"
-			(at 48.26 -37.5416 0)
-			(effects
-				(font
-					(size 1.27 1.27)
-				)
-				(justify left bottom)
-			)
-		)
-		(property "Sheetfile" "vca.kicad_sch"
-			(at 48.26 -10.8454 0)
-			(effects
-				(font
-					(size 1.27 1.27)
-				)
-				(justify left top)
-			)
-		)
-		(instances
-			(project "dynafuzz"
-				(path "/b401260a-0de9-4b23-a692-63e5f9163375"
-					(page "3")
-				)
-			)

Commit message: rev D
Parts:
- C12: value 100n -> 1u
- R18: value 3.3k -> 10k
Connections:
- net IN: now also R1.2; no longer R1.1
- net at C10.1, RV2.2, RV3.3: now also RV2.3; no longer RV2.1
- net at C1.1: now also R1.1; no longer R1.2
- net at R19.1: now also RV2.1; no longer RV2.3
Other:
- note added: "Low-resistance is heavily scooped A or B taper, A allows finer control of mids At 15K (50% on A taper pot), scoop comparable to classic Big Muff"
- note added: "NOTE: transistors are always biased when power applied, even when bypassed"
- note added: "R18 adjusts LED brightness"
- note added: "TONE STACK"
- note added: "better low end than 100n but replaceable for less parts"
- note added: "https://tonestack.yuriturov.com/?s=eNpbmpj-NbFsWVKQ02_7261yOwJftyYF-f62P2wMBklBIb_sGRgYkoKcf9s_WHydy7ZgSVJQ2G_7Ww_d14lUPUoKCgeybQtAMokViWVJRcULEkuaFyVmpuSWphkmJq9MDvL0S7HQM8pOCvJJMTQwANK-zWBGog_U6BA0vmGysTFQmVGSYXaSs2GyoUFekrMRhDJOMixdjGp4sqEpitnJRqZ4jbYEGZ1iBHKRs2GKmZ4FyHQobQxSnZdUlvkF6gODxOQVmJbgMjXZyAjJxUkmUAcDACKXfVU"
- note removed: "A or B taper A preferred"
- note removed: "HOOF Tone Stack - modified values at tone even (45%), mids go from huge scoop at 3kHz to slight boost phase flat"
- note removed: "https://tonestack.yuriturov.com/?s=eNpbmpj-NbFsWVKQ02_7261yOwJftyYF-TImBYX8tr_x9VB_jMa3pCDn3_YPFl_nsi1YkhQU9tv-1kP3dSJVj5KCwoFs2wKQTGJFYllSUfGCxJKWRYmZKbmlaYaJySuTgzz9Eg2SgnxSDA0MsoHmNicbmWYn-vyyZ2BgAFrRDBaH8w2TjY2BqoxSjPWAtLNhsqFBXpKzEYQyBqnNgxpulJi8CtNwVNOAphuZophuCFJmlGxmgWR4iomeOcj0ZBMQZYJsCcwHyYam2aT4wRLsByM9I5A1KWZ6FmB7IDRWXyQbGmWT4Q9TM7A_wA4Hhxm6PwB9TKNZ"
- note removed: "or 10k"
- note removed: "scoop happens when MID is short 0% - R=0 - super scoop 50% - R=~15k - small scoop 80% - R=~30k - flat EQ 100% - R=100k - slight mid boost"
- moved on the sheet: R1
Changed lines of the file:
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@@
 	(generator_version "9.0")
 	(paper "A4")
-	(text "scoop happens when MID is short\n0% - R=0 - super scoop\n50% - R=~15k - small scoop\n80% - R=~30k - flat EQ\n100% - R=100k - slight mid boost"
+	(text "NOTE: transistors are always biased when power applied, even when bypassed"
 		(exclude_from_sim no)
-		(at 199.39 78.74 0)
+		(at 100.33 160.02 0)
 		(effects
 			(font
@@
 		)
 	)
-	(text "A or B taper\nA preferred"
+	(text "Low-resistance is heavily scooped\nA or B taper, A allows finer control of mids\nAt 15K (50% on A taper pot), scoop comparable\nto classic Big Muff"
 		(exclude_from_sim no)
-		(at 190.5 90.17 0)
+		(at 194.31 86.36 0)
 		(effects
 			(font
-				(size 1.27 1.27)
+				(size 0.64 0.64)
 			)
 		)
 	)
-	(text "HOOF Tone Stack - modified values\n\nat tone even (45%),\nmids go from huge scoop at 3kHz to slight boost\nphase flat"
+	(text "TONE STACK"
 		(exclude_from_sim no)
-		(at 186.69 148.59 0)
+		(at 196.85 142.24 0)
 		(effects
 			(font
@@
 		)
 	)
-	(text "https://tonestack.yuriturov.com/?s=eNpbmpj-NbFsWVKQ02_7261yOwJftyYF-TImBYX8tr_x9VB_jMa3pCDn3_YPFl_nsi1YkhQU9tv-1kP3dSJVj5KCwoFs2wKQTGJFYllSUfGCxJKWRYmZKbmlaYaJySuTgzz9Eg2SgnxSDA0MsoHmNicbmWYn-vyyZ2BgAFrRDBaH8w2TjY2BqoxSjPWAtLNhsqFBXpKzEYQyBqnNgxpulJi8CtNwVNOAphuZophuCFJmlGxmgWR4iomeOcj0ZBMQZYJsCcwHyYam2aT4wRLsByM9I5A1KWZ6FmB7IDRWXyQbGmWT4Q9TM7A_wA4Hhxm6PwB9TKNZ"
+	(text "better low end than 100n\nbut replaceable for less parts"
+		(exclude_from_sim no)
+		(at 213.36 114.3 0)
+		(effects
+			(font
+				(size 0.635 0.635)
+			)
+		)
+	)
+	(text "https://tonestack.yuriturov.com/?s=eNpbmpj-NbFsWVKQ02_7261yOwJftyYF-f62P2wMBklBIb_sGRgYkoKcf9s_WHydy7ZgSVJQ2G_7Ww_d14lUPUoKCgeybQtAMokViWVJRcULEkuaFyVmpuSWphkmJq9MDvL0S7HQM8pOCvJJMTQwANK-zWBGog_U6BA0vmGysTFQmVGSYXaSs2GyoUFekrMRhDJOMixdjGp4sqEpitnJRqZ4jbYEGZ1iBHKRs2GKmZ4FyHQobQxSnZdUlvkF6gODxOQVmJbgMjXZyAjJxUkmUAcDACKXfVU"
 		(exclude_from_sim no)
 		(at 210.058 216.154 0)
@@
 		)
 	)
-	(text "DUAL GAIN"
+	(text "R18 adjusts LED brightness"
 		(exclude_from_sim no)
-		(at 144.78 124.46 0)
+		(at 195.58 43.18 90)
 		(effects
 			(font
@@
 		)
 	)
-	(text "or 10k"
+	(text "DUAL GAIN"
 		(exclude_from_sim no)
-		(at 137.16 78.486 90)
+		(at 144.78 124.46 0)
 		(effects
 			(font
@@
 	)
 	(junction
+		(at 200.66 99.06)
+		(diameter 0)
+		(color 0 0 0 0)
+	)
+	(junction
 		(at 121.92 88.9)
 		(diameter 0)
@@
 	)
 	(junction
-		(at 200.66 99.06)
-		(diameter 0)
-		(color 0 0 0 0)
-	)
-	(junction
 		(at 205.74 110.49)
 		(diameter 0)
@@
 	(wire
 		(pts
+			(xy 204.47 99.06) (xy 200.66 99.06)
+		)
+		(stroke
+			(width 0)
+			(type default)
+		)
+	)
+	(wire
+		(pts
 			(xy 172.72 100.33) (xy 172.72 104.14)
 		)
@@
 	(wire
 		(pts
-			(xy 204.47 99.06) (xy 200.66 99.06)
-		)
-		(stroke
-			(width 0)
-			(type default)
-		)
-	)
-	(wire
-		(pts
 			(xy 242.57 36.83) (xy 242.57 31.75)
 		)
@@
 	(wire
 		(pts
+			(xy 204.47 95.25) (xy 204.47 99.06)
+		)
+		(stroke
+			(width 0)
+			(type default)
+		)
+	)
+	(wire
+		(pts
 			(xy 162.56 100.33) (xy 161.29 100.33)
 		)
@@
 	(wire
 		(pts
-			(xy 204.47 95.25) (xy 204.47 99.06)
-		)
-		(stroke
-			(width 0)
-			(type default)
-		)
-	)
-	(wire
-		(pts
 			(xy 157.48 90.17) (xy 157.48 100.33)
 		)
@@
 	(symbol
 		(lib_id "Device:R")
-		(at 38.1 105.41 90)
+		(at 38.1 105.41 270)
 		(unit 1)
 		(exclude_from_sim no)
@@
 		)
 		(property "Footprint" "_project:R"
-			(at 38.1 107.188 90)
+			(at 38.1 103.632 90)
 			(effects
 				(font
@@
 			)
 		)
-		(property "Value" "100n"
+		(property "Value" "1u"
 			(at 213.614 106.68 90)
 			(effects
@@
 		(lib_id "Device:R_Potentiometer")
 		(at 200.66 95.25 0)
-		(mirror x)
 		(unit 1)
 		(exclude_from_sim no)
@@
 		(dnp no)
 		(property "Reference" "RV2"
-			(at 198.12 96.5201 0)
+			(at 198.12 93.9799 0)
 			(effects
 				(font
@@
 		)
 		(property "Value" "R_MID-A100K"
-			(at 198.12 93.9801 0)
+			(at 198.12 96.5199 0)
 			(effects
 				(font
@@
 		(dnp no)
 		(property "Reference" "C11"
-			(at 195.834 127 90)
+			(at 194.31 124.46 90)
 			(effects
 				(font
@@
 		)
 		(property "Value" "10n"
-			(at 198.374 127 90)
+			(at 196.85 124.46 90)
 			(effects
 				(font
@@
 			)
 		)
-		(property "Value" "3.3k"
+		(property "Value" "10k"
 			(at 203.2 45.7199 0)
 			(effects
@@
 		(dnp no)
 		(property "Reference" "C10"
-			(at 187.96 99.314 90)
+			(at 190.5 97.79 90)
 			(effects
 				(font
@@
 		)
 		(property "Value" "10n"
-			(at 187.96 101.854 90)
+			(at 190.5 100.33 90)
 			(effects
 				(font
