File: chorus2/basschorus/tonesplitter.kicad_sch (KiCad schematic)
At the start: 17 parts, among them U6 TL074, U7 TL074, U9 TL074

Commit message: code implementation
Parts:
- renumbered R24 to R26, R25 to R27, R27 to R28, R28 to R29, R29 to R30, R30 to R31, R31 to R32, R32 to R33, U9 to U1, U6 to U1, U7 to U1
Connections:
- net DRY_OUT: now also U1.14; no longer U1.7
- net WET_OUT: now also U1.8, U1.9 (-); no longer U1.6 (-), U1.7
- net at R31.1, R32.2: now also U1.12 (+); no longer U1.5 (+)
- net at R30.1, R33.2: now also U1.13 (-); no longer U1.6 (-)
- net at C27.2, R29.1: now also U1.10 (+); no longer U1.5 (+)
Changed lines of the file:
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@@
 		(on_board yes)
 		(dnp no)
-		(property "Reference" "R30"
+		(property "Reference" "R31"
 			(at 199.39 120.65 90)
 			(effects
@@
 			(project "basschorus"
 				(path "/7f3b4bac-3b2a-4af0-92ae-ccc3fcedc393/266c062e-3d0a-4a44-9ad1-7a160f1a9b37"
-					(reference "R30")
+					(reference "R31")
 					(unit 1)
 				)
@@
 		(on_board yes)
 		(dnp no)
-		(property "Reference" "R29"
+		(property "Reference" "R30"
 			(at 199.39 105.2322 90)
 			(effects
@@
 			(project "basschorus"
 				(path "/7f3b4bac-3b2a-4af0-92ae-ccc3fcedc393/266c062e-3d0a-4a44-9ad1-7a160f1a9b37"
-					(reference "R29")
+					(reference "R30")
 					(unit 1)
 				)
@@
 		(on_board yes)
 		(dnp no)
-		(property "Reference" "R32"
+		(property "Reference" "R33"
 			(at 217.17 98.8822 90)
 			(effects
@@
 			(project "basschorus"
 				(path "/7f3b4bac-3b2a-4af0-92ae-ccc3fcedc393/266c062e-3d0a-4a44-9ad1-7a160f1a9b37"
-					(reference "R32")
+					(reference "R33")
 					(unit 1)
 				)
@@
 		(on_board yes)
 		(dnp no)
-		(property "Reference" "R31"
+		(property "Reference" "R32"
 			(at 210.9978 120.65 90)
 			(effects
@@
 			(project "basschorus"
 				(path "/7f3b4bac-3b2a-4af0-92ae-ccc3fcedc393/266c062e-3d0a-4a44-9ad1-7a160f1a9b37"
-					(reference "R31")
+					(reference "R32")
 					(unit 1)
 				)
@@
 		(on_board yes)
 		(dnp no)
-		(property "Reference" "R27"
+		(property "Reference" "R28"
 			(at 128.27 79.8322 90)
 			(effects
@@
 			(project "basschorus"
 				(path "/7f3b4bac-3b2a-4af0-92ae-ccc3fcedc393/266c062e-3d0a-4a44-9ad1-7a160f1a9b37"
-					(reference "R27")
+					(reference "R28")
 					(unit 1)
 				)
@@
 		(on_board yes)
 		(dnp no)
-		(property "Reference" "R28"
+		(property "Reference" "R29"
 			(at 153.67 79.8322 90)
 			(effects
@@
 			(project "basschorus"
 				(path "/7f3b4bac-3b2a-4af0-92ae-ccc3fcedc393/266c062e-3d0a-4a44-9ad1-7a160f1a9b37"
-					(reference "R28")
+					(reference "R29")
 					(unit 1)
 				)
@@
 		(on_board yes)
 		(dnp no)
-		(property "Reference" "R24"
+		(property "Reference" "R26"
 			(at 101.6 96.3422 90)
 			(effects
@@
 			(project "basschorus"
 				(path "/7f3b4bac-3b2a-4af0-92ae-ccc3fcedc393/266c062e-3d0a-4a44-9ad1-7a160f1a9b37"
-					(reference "R24")
+					(reference "R26")
 					(unit 1)
 				)
@@
 		(on_board yes)
 		(dnp no)
-		(property "Reference" "R25"
+		(property "Reference" "R27"
 			(at 102.87 64.5922 90)
 			(effects
@@
 			(project "basschorus"
 				(path "/7f3b4bac-3b2a-4af0-92ae-ccc3fcedc393/266c062e-3d0a-4a44-9ad1-7a160f1a9b37"
-					(reference "R25")
+					(reference "R27")
 					(unit 1)
 				)
@@
 		(at 215.9 113.03 0)
 		(mirror x)
-		(unit 2)
-		(exclude_from_sim no)
-		(in_bom yes)
-		(on_board yes)
-		(dnp no)
-		(property "Reference" "U9"
+		(unit 4)
+		(exclude_from_sim no)
+		(in_bom yes)
+		(on_board yes)
+		(dnp no)
+		(property "Reference" "U1"
 			(at 215.9 122.3518 0)
 			(effects
@@
 			(project "basschorus"
 				(path "/7f3b4bac-3b2a-4af0-92ae-ccc3fcedc393/266c062e-3d0a-4a44-9ad1-7a160f1a9b37"
-					(reference "U9")
-					(unit 2)
+					(reference "U1")
+					(unit 4)
 				)
 			)
@@
 		(dnp no)
 		(fields_autoplaced yes)
-		(property "Reference" "#PWR048"
+		(property "Reference" "#PWR050"
 			(at 161.29 106.68 0)
 			(effects
@@
 			(project "basschorus"
 				(path "/7f3b4bac-3b2a-4af0-92ae-ccc3fcedc393/266c062e-3d0a-4a44-9ad1-7a160f1a9b37"
-					(reference "#PWR048")
+					(reference "#PWR050")
 					(unit 1)
 				)
@@
 		(on_board yes)
 		(dnp no)
-		(property "Reference" "U6"
+		(property "Reference" "U1"
 			(at 105.41 75.7682 0)
 			(effects
@@
 			(project "basschorus"
 				(path "/7f3b4bac-3b2a-4af0-92ae-ccc3fcedc393/266c062e-3d0a-4a44-9ad1-7a160f1a9b37"
-					(reference "U6")
+					(reference "U1")
 					(unit 2)
 				)
@@
 		(dnp no)
 		(fields_autoplaced yes)
-		(property "Reference" "#PWR050"
+		(property "Reference" "#PWR051"
 			(at 205.74 133.35 0)
 			(effects
@@
 			(project ""
 				(path "/7f3b4bac-3b2a-4af0-92ae-ccc3fcedc393/266c062e-3d0a-4a44-9ad1-7a160f1a9b37"
-					(reference "#PWR050")
+					(reference "#PWR051")
 					(unit 1)
 				)
@@
 		(lib_id "Amplifier_Operational:TL074")
 		(at 177.8 87.63 0)
-		(unit 2)
-		(exclude_from_sim no)
-		(in_bom yes)
-		(on_board yes)
-		(dnp no)
-		(property "Reference" "U7"
+		(unit 3)
+		(exclude_from_sim no)
+		(in_bom yes)
+		(on_board yes)
+		(dnp no)
+		(property "Reference" "U1"
 			(at 177.8 78.3082 0)
 			(effects
@@
 			(project "basschorus"
 				(path "/7f3b4bac-3b2a-4af0-92ae-ccc3fcedc393/266c062e-3d0a-4a44-9ad1-7a160f1a9b37"
-					(reference "U7")
-					(unit 2)
-				)
-			)
+					(reference "U1")
+					(unit 3)
+				)
+			)

Commit message: update filters
Parts:
- renumbered R26 to R27, R27 to R28, R28 to R29, R29 to R30, R30 to R31, R31 to R32, R32 to R33, R33 to R34
Changed lines of the file:
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@@
 		(on_board yes)
 		(dnp no)
-		(property "Reference" "R31"
+		(property "Reference" "R32"
 			(at 199.39 120.65 90)
 			(effects
@@
 			(project "basschorus"
 				(path "/7f3b4bac-3b2a-4af0-92ae-ccc3fcedc393/266c062e-3d0a-4a44-9ad1-7a160f1a9b37"
-					(reference "R31")
+					(reference "R32")
 					(unit 1)
 				)
@@
 		(on_board yes)
 		(dnp no)
-		(property "Reference" "R30"
+		(property "Reference" "R31"
 			(at 199.39 105.2322 90)
 			(effects
@@
 			(project "basschorus"
 				(path "/7f3b4bac-3b2a-4af0-92ae-ccc3fcedc393/266c062e-3d0a-4a44-9ad1-7a160f1a9b37"
-					(reference "R30")
+					(reference "R31")
 					(unit 1)
 				)
@@
 		(on_board yes)
 		(dnp no)
-		(property "Reference" "R33"
+		(property "Reference" "R34"
 			(at 217.17 98.8822 90)
 			(effects
@@
 			(project "basschorus"
 				(path "/7f3b4bac-3b2a-4af0-92ae-ccc3fcedc393/266c062e-3d0a-4a44-9ad1-7a160f1a9b37"
-					(reference "R33")
+					(reference "R34")
 					(unit 1)
 				)
@@
 		(on_board yes)
 		(dnp no)
-		(property "Reference" "R32"
+		(property "Reference" "R33"
 			(at 210.9978 120.65 90)
 			(effects
@@
 			(project "basschorus"
 				(path "/7f3b4bac-3b2a-4af0-92ae-ccc3fcedc393/266c062e-3d0a-4a44-9ad1-7a160f1a9b37"
-					(reference "R32")
+					(reference "R33")
 					(unit 1)
 				)
@@
 		(on_board yes)
 		(dnp no)
-		(property "Reference" "R28"
+		(property "Reference" "R29"
 			(at 128.27 79.8322 90)
 			(effects
@@
 			(project "basschorus"
 				(path "/7f3b4bac-3b2a-4af0-92ae-ccc3fcedc393/266c062e-3d0a-4a44-9ad1-7a160f1a9b37"
-					(reference "R28")
+					(reference "R29")
 					(unit 1)
 				)
@@
 		(on_board yes)
 		(dnp no)
-		(property "Reference" "R29"
+		(property "Reference" "R30"
 			(at 153.67 79.8322 90)
 			(effects
@@
 			(project "basschorus"
 				(path "/7f3b4bac-3b2a-4af0-92ae-ccc3fcedc393/266c062e-3d0a-4a44-9ad1-7a160f1a9b37"
-					(reference "R29")
+					(reference "R30")
 					(unit 1)
 				)
@@
 		(on_board yes)
 		(dnp no)
-		(property "Reference" "R26"
+		(property "Reference" "R27"
 			(at 101.6 96.3422 90)
 			(effects
@@
 			(project "basschorus"
 				(path "/7f3b4bac-3b2a-4af0-92ae-ccc3fcedc393/266c062e-3d0a-4a44-9ad1-7a160f1a9b37"
-					(reference "R26")
+					(reference "R27")
 					(unit 1)
 				)
@@
 		(on_board yes)
 		(dnp no)
-		(property "Reference" "R27"
+		(property "Reference" "R28"
 			(at 102.87 64.5922 90)
 			(effects
@@
 			(project "basschorus"
 				(path "/7f3b4bac-3b2a-4af0-92ae-ccc3fcedc393/266c062e-3d0a-4a44-9ad1-7a160f1a9b37"
-					(reference "R27")
+					(reference "R28")
 					(unit 1)
 				)
@@
 		(dnp no)
 		(fields_autoplaced yes)
-		(property "Reference" "#PWR049"
+		(property "Reference" "#PWR054"
 			(at 119.38 111.76 0)
 			(effects
@@
 			(project "basschorus"
 				(path "/7f3b4bac-3b2a-4af0-92ae-ccc3fcedc393/266c062e-3d0a-4a44-9ad1-7a160f1a9b37"
-					(reference "#PWR049")
+					(reference "#PWR054")
 					(unit 1)
 				)
@@
 		(dnp no)
 		(fields_autoplaced yes)
-		(property "Reference" "#PWR050"
+		(property "Reference" "#PWR055"
 			(at 161.29 106.68 0)
 			(effects
@@
 			(project "basschorus"
 				(path "/7f3b4bac-3b2a-4af0-92ae-ccc3fcedc393/266c062e-3d0a-4a44-9ad1-7a160f1a9b37"
-					(reference "#PWR050")
+					(reference "#PWR055")
 					(unit 1)
 				)
@@
 		(dnp no)
 		(fields_autoplaced yes)
-		(property "Reference" "#PWR051"
+		(property "Reference" "#PWR056"
 			(at 205.74 133.35 0)
 			(effects
@@
 			(project ""
 				(path "/7f3b4bac-3b2a-4af0-92ae-ccc3fcedc393/266c062e-3d0a-4a44-9ad1-7a160f1a9b37"
-					(reference "#PWR051")
-					(unit 1)
-				)
+					(reference "#PWR056")
+					(unit 1)
+				)

Commit message: update designs based on new calculations
Parts:
- C24, C25: value 33n -> 150n
Other:
- note added: "2nd order HPF, Q=0.5 Adjustable Cutoff: 10Hz - 10KHz"
- note removed: "2nd order HPF, Q=0.5 Adjustable Cutoff: 50Hz - 5KHz"
Changed lines of the file:
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@@
 		)
 	)
-	(text "2nd order HPF, Q=0.5\nAdjustable Cutoff: 50Hz - 5KHz"
+	(text "2nd order HPF, Q=0.5\nAdjustable Cutoff: 10Hz - 10KHz"
 		(exclude_from_sim no)
 		(at 81.28 113.03 0)
@@
 			)
 		)
-		(property "Value" "33n"
+		(property "Value" "150n"
 			(at 88.9 78.4606 90)
 			(effects
@@
 				(path "/7f3b4bac-3b2a-4af0-92ae-ccc3fcedc393/266c062e-3d0a-4a44-9ad1-7a160f1a9b37"
 					(reference "C25")
+					(unit 1)
+				)
+			)
+		)
+	)
+	(symbol
+		(lib_id "Device:C")
+		(at 153.67 74.93 270)
+		(unit 1)
+		(exclude_from_sim no)
+		(in_bom yes)
+		(on_board yes)
+		(dnp no)
+		(property "Reference" "C26"
+			(at 153.67 68.5292 90)
+			(effects
+				(font
+					(size 1.27 1.27)
+				)
+			)
+		)
+		(property "Value" "10n"
+			(at 153.67 70.8406 90)
+			(effects
+				(font
+					(size 1.27 1.27)
+				)
+			)
+		)
+		(property "Footprint" ""
+			(at 149.86 75.8952 0)
+			(effects
+				(font
+					(size 1.27 1.27)
+				)
+				(hide yes)
+			)
+		)
+		(property "Datasheet" "~"
+			(at 153.67 74.93 0)
+			(effects
+				(font
+					(size 1.27 1.27)
+				)
+				(hide yes)
+			)
+		)
+		(property "Description" ""
+			(at 153.67 74.93 0)
+			(effects
+				(font
+					(size 1.27 1.27)
+				)
+			)
+		)
+		(pin "1"
+		)
+		(pin "2"
+		)
+		(instances
+			(project "basschorus"
+				(path "/7f3b4bac-3b2a-4af0-92ae-ccc3fcedc393/266c062e-3d0a-4a44-9ad1-7a160f1a9b37"
+					(reference "C26")
+					(unit 1)
+				)
+			)
+		)
+	)
+	(symbol
+		(lib_id "Device:C")
+		(at 76.2 82.55 270)
+		(unit 1)
+		(exclude_from_sim no)
+		(in_bom yes)
+		(on_board yes)
+		(dnp no)
+		(property "Reference" "C24"
+			(at 76.2 76.1492 90)
+			(effects
+				(font
+					(size 1.27 1.27)
+				)
+			)
+		)
+		(property "Value" "150n"
+			(at 76.2 78.4606 90)
+			(effects
+				(font
+					(size 1.27 1.27)
+				)
+			)
+		)
+		(property "Footprint" ""
+			(at 72.39 83.5152 0)
+			(effects
+				(font
+					(size 1.27 1.27)
+				)
+				(hide yes)
+			)
+		)
+		(property "Datasheet" "~"
+			(at 76.2 82.55 0)
+			(effects
+				(font
+					(size 1.27 1.27)
+				)
+				(hide yes)
+			)
+		)
+		(property "Description" ""
+			(at 76.2 82.55 0)
+			(effects
+				(font
+					(size 1.27 1.27)
+				)
+			)
+		)
+		(pin "1"
+		)
+		(pin "2"
+		)
+		(instances
+			(project "basschorus"
+				(path "/7f3b4bac-3b2a-4af0-92ae-ccc3fcedc393/266c062e-3d0a-4a44-9ad1-7a160f1a9b37"
+					(reference "C24")
 					(unit 1)
 				)
@@
 				)
 			)
-		)
-	)
-	(symbol
-		(lib_id "Device:C")
-		(at 153.67 74.93 270)
-		(unit 1)
-		(exclude_from_sim no)
-		(in_bom yes)
-		(on_board yes)
-		(dnp no)
-		(property "Reference" "C26"
-			(at 153.67 68.5292 90)
-			(effects
-				(font
-					(size 1.27 1.27)
-				)
-			)
-		)
-		(property "Value" "10n"
-			(at 153.67 70.8406 90)
-			(effects
-				(font
-					(size 1.27 1.27)
-				)
-			)
-		)
-		(property "Footprint" ""
-			(at 149.86 75.8952 0)
-			(effects
-				(font
-					(size 1.27 1.27)
-				)
-				(hide yes)
-			)
-		)
-		(property "Datasheet" "~"
-			(at 153.67 74.93 0)
-			(effects
-				(font
-					(size 1.27 1.27)
-				)
-				(hide yes)
-			)
-		)
-		(property "Description" ""
-			(at 153.67 74.93 0)
-			(effects
-				(font
-					(size 1.27 1.27)
-				)
-			)
-		)
-		(pin "1"
-		)
-		(pin "2"
-		)
-		(instances
-			(project "basschorus"
-				(path "/7f3b4bac-3b2a-4af0-92ae-ccc3fcedc393/266c062e-3d0a-4a44-9ad1-7a160f1a9b37"
-					(reference "C26")
-					(unit 1)
-				)
-			)
-		)
-	)
-	(symbol
-		(lib_id "Device:C")
-		(at 76.2 82.55 270)
-		(unit 1)
-		(exclude_from_sim no)
-		(in_bom yes)
-		(on_board yes)
-		(dnp no)
-		(property "Reference" "C24"
-			(at 76.2 76.1492 90)
-			(effects
-				(font
-					(size 1.27 1.27)
-				)
-			)
-		)
-		(property "Value" "33n"
-			(at 76.2 78.4606 90)
-			(effects
-				(font
-					(size 1.27 1.27)
-				)
-			)
-		)
-		(property "Footprint" ""
-			(at 72.39 83.5152 0)
-			(effects
-				(font
-					(size 1.27 1.27)
-				)
-				(hide yes)
-			)
-		)
-		(property "Datasheet" "~"
-			(at 76.2 82.55 0)
-			(effects
-				(font
-					(size 1.27 1.27)
-				)
-				(hide yes)
-			)
-		)
-		(property "Description" ""
-			(at 76.2 82.55 0)
-			(effects
-				(font
-					(size 1.27 1.27)
-				)
-			)
-		)
-		(pin "1"
-		)
-		(pin "2"
-		)
-		(instances
-			(project "basschorus"
-				(path "/7f3b4bac-3b2a-4af0-92ae-ccc3fcedc393/266c062e-3d0a-4a44-9ad1-7a160f1a9b37"
-					(reference "C24")
-					(unit 1)
-				)
-			)

Commit message: assign parts for testing
Parts:
- added TP4: TestPoint, TestPoint:TestPoint_THTPad_2.5x2.5mm_Drill1.2mm, symbol Connector:TestPoint
- C29: renamed from C24; footprint (none) -> Capacitor_THT:C_Rect_L7.0mm_W2.5mm_P5.00mm
- C30: renamed from C25; footprint (none) -> Capacitor_THT:C_Rect_L7.0mm_W2.5mm_P5.00mm
- C31: renamed from C26; footprint (none) -> Capacitor_THT:C_Rect_L7.0mm_W2.5mm_P5.00mm
- C32: renamed from C27; footprint (none) -> Capacitor_THT:C_Rect_L7.0mm_W2.5mm_P5.00mm
- R33: renamed from R27; footprint kicad-legacy/kicad-footprints/Resistor_THT.pretty:R_Axial_DIN0204_L3.6mm_D1.6mm_P2.54mm_Vertical -> Resistor_THT:R_Axial_DIN0204_L3.6mm_D1.6mm_P5.08mm_Horizontal
- R34: renamed from R28; footprint kicad-legacy/kicad-footprints/Resistor_THT.pretty:R_Axial_DIN0204_L3.6mm_D1.6mm_P2.54mm_Vertical -> Resistor_THT:R_Axial_DIN0204_L3.6mm_D1.6mm_P5.08mm_Horizontal
- R35: renamed from R29; footprint kicad-legacy/kicad-footprints/Resistor_THT.pretty:R_Axial_DIN0204_L3.6mm_D1.6mm_P2.54mm_Vertical -> Resistor_THT:R_Axial_DIN0204_L3.6mm_D1.6mm_P5.08mm_Horizontal
- R36: renamed from R30; footprint kicad-legacy/kicad-footprints/Resistor_THT.pretty:R_Axial_DIN0204_L3.6mm_D1.6mm_P2.54mm_Vertical -> Resistor_THT:R_Axial_DIN0204_L3.6mm_D1.6mm_P5.08mm_Horizontal
- R37: renamed from R31; footprint kicad-legacy/kicad-footprints/Resistor_THT.pretty:R_Axial_DIN0204_L3.6mm_D1.6mm_P2.54mm_Vertical -> Resistor_THT:R_Axial_DIN0204_L3.6mm_D1.6mm_P5.08mm_Horizontal
- R38: renamed from R32; footprint kicad-legacy/kicad-footprints/Resistor_THT.pretty:R_Axial_DIN0204_L3.6mm_D1.6mm_P2.54mm_Vertical -> Resistor_THT:R_Axial_DIN0204_L3.6mm_D1.6mm_P5.08mm_Horizontal
- R39: renamed from R33; footprint kicad-legacy/kicad-footprints/Resistor_THT.pretty:R_Axial_DIN0204_L3.6mm_D1.6mm_P2.54mm_Vertical -> Resistor_THT:R_Axial_DIN0204_L3.6mm_D1.6mm_P5.08mm_Horizontal
- R40: renamed from R34; footprint kicad-legacy/kicad-footprints/Resistor_THT.pretty:R_Axial_DIN0204_L3.6mm_D1.6mm_P2.54mm_Vertical -> Resistor_THT:R_Axial_DIN0204_L3.6mm_D1.6mm_P5.08mm_Horizontal
- RV7: renamed from RV4; footprint kicad-legacy/Potentiometers.pretty:Potentiometer_Trimmer_Bourns_3296W -> Potentiometer_THT:Potentiometer_Vishay_T73YP_Vertical
- R_CUTOFF_1: footprint kicad-legacy/kicad-footprints/Potentiometer_THT.pretty:Potentiometer_Alps_RK09L_Double_Vertical -> Potentiometer_THT:Potentiometer_Alpha_RD902F-40-00D_Dual_Vertical_CircularHoles
- U1: footprint kicad-legacy/kicad-footprints/Package_DIP.pretty:DIP-14_W7.62mm -> Package_SO:SO-14_3.9x8.65mm_P1.27mm

Commit message: started layout
Parts:
- TP4: value TestPoint -> TONE_HP
Connections:
- net at R35.2, R_CUTOFF_1.4, U1.6 (-)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: now also TP4.1
Other:
- moved on the sheet: TP4
Changed lines of the file:
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@@
 	(symbol
 		(lib_id "Connector:TestPoint")
-		(at 121.92 85.725 180)
+		(at 121.92 85.09 180)
 		(unit 1)
 		(exclude_from_sim no)
@@
 		(fields_autoplaced yes)
 		(property "Reference" "TP4"
-			(at 124.46 87.7569 0)
+			(at 124.46 87.1219 0)
 			(effects
 				(font
@@
 			)
 		)
-		(property "Value" "TestPoint"
-			(at 124.46 90.2969 0)
+		(property "Value" "TONE_HP"
+			(at 124.46 89.6619 0)
 			(effects
 				(font
@@
 		)
 		(property "Footprint" "TestPoint:TestPoint_THTPad_2.5x2.5mm_Drill1.2mm"
-			(at 116.84 85.725 0)
+			(at 116.84 85.09 0)
 			(effects
 				(font
@@
 		)
 		(property "Datasheet" "~"
-			(at 116.84 85.725 0)
+			(at 116.84 85.09 0)
 			(effects
 				(font
@@
 		)
 		(property "Description" "test point"
-			(at 121.92 85.725 0)
+			(at 121.92 85.09 0)
 			(effects
 				(font

Commit message: update params
Parts:
- removed unit 2 of R_CUTOFF_1
- added unit 2 of RV12
- RV12: renamed from R_CUTOFF_1; value A100K -> R_CUTOFF_A100K
Connections:
- net at R35.2, TP4.1, U1.6 (-)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: now also RV12.4
- net at R34.1: now also RV12.5, RV12.6
Other:
- note added: "2nd order HPF, Q=0.5 Adjustable Cutoff: 10Hz - 1KHz"
- note added: "from .core import db tone_splitter_hp = filters.sallen_key_hp() # An adjustable sub-butterworth filter (Q=0.5) # with a cutoff from ~10Hz to ~1kHz # 1kHz # tone_splitter_hp.realize(c1="150n", c2="150n", r3="1k", r4="1k") # 100Hz tone_splitter_hp.realize(c1="150n", c2="150n", r3="11k", r4="11k") # 10Hz # tone_splitter_hp.realize(c1="150n", c2="150n", r3="101k", r4="101k") # tone_splitter_hp.plot_b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"
- note removed: "2nd order HPF, Q=0.5 Adjustable Cutoff: 10Hz - 10KHz"
Changed lines of the file:
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@@
 		)
 	)
-	(text "2nd order HPF, Q=0.5\nAdjustable Cutoff: 10Hz - 10KHz"
+	(text "2nd order HPF, Q=0.5\nAdjustable Cutoff: 10Hz - 1KHz"
 		(exclude_from_sim no)
 		(at 81.28 113.03 0)
@@
 			)
 			(justify left bottom)
+		)
+	)
+	(text "from .core import db\n\ntone_splitter_hp = filters.sallen_key_hp()\n# An adjustable sub-butterworth filter (Q=0.5)\n# with a cutoff from ~10Hz to ~1kHz\n\n# 1kHz\n# tone_splitter_hp.realize(c1=\"150n\", c2=\"150n\", r3=\"1k\", r4=\"1k\")\n# 100Hz\ntone_splitter_hp.realize(c1=\"150n\", c2=\"150n\", r3=\"11k\", r4=\"11k\")\n# 10Hz\n# tone_splitter_hp.realize(c1=\"150n\", c2=\"150n\", r3=\"101k\", r4=\"101k\")\n# tone_splitter_hp.plot_bode()\ndb(np.abs(tone_splitter_hp.evaluate(10)))\ndb(np.abs(tone_splitter_hp.evaluate(100)))\ndb(np.abs(tone_splitter_hp.evaluate(1000)))\n\n# upper bound of bandpass filter. fc=3.162kHz, Q=0.707 (butterworth)\ntone_splitter_lp = filters.sallen_key_lp()\ntone_splitter_lp.realize(r1=\"9.1k\", r2=\"5.6k\", c3=\"10n\", c4=\"4.7n\")\n# adjusted for less novel parts\ntone_splitter_lp.realize(r1=\"10k\", r2=\"5.6k\", c3=\"10n\", c4=\"4.7n\")\n# tone_splitter_lp.plot_bode()\ndb(np.abs(tone_splitter_lp.evaluate(3162))) # -3.2db\n\ntone_splitter = tone_splitter_hp.cascade(tone_splitter_lp)\ntone_stopband = db(np.abs(tone_splitter.evaluate(5_000))) # -9.3dB\n# tone_splitter.plot_bode()"
+		(exclude_from_sim no)
+		(at 16.51 133.985 0)
+		(effects
+			(font
+				(size 1.27 1.27)
+			)
+			(justify left top)
 		)
 	)
@@
 	(symbol
 		(lib_id "Device:R_Potentiometer_Dual_Separate")
-		(at 115.57 69.85 270)
-		(unit 2)
+		(at 113.03 101.6 270)
+		(unit 1)
 		(exclude_from_sim no)
 		(in_bom yes)
 		(on_board yes)
 		(dnp no)
-		(property "Reference" "R_CUTOFF_1"
-			(at 115.57 64.5922 90)
-			(effects
-				(font
-					(size 1.27 1.27)
-				)
-			)
-		)
-		(property "Value" "A100K"
-			(at 115.57 66.9036 90)
+		(property "Reference" "RV12"
+			(at 113.03 96.3422 90)
+			(effects
+				(font
+					(size 1.27 1.27)
+				)
+			)
+		)
+		(property "Value" "R_CUTOFF_A100K"
+			(at 113.03 98.6536 90)
 			(effects
 				(font
@@
 		)
 		(property "Footprint" "Potentiometer_THT:Potentiometer_Alpha_RD902F-40-00D_Dual_Vertical_CircularHoles"
-			(at 115.57 69.85 0)
+			(at 113.03 101.6 0)
 			(effects
 				(font
@@
 		)
 		(property "Datasheet" "~"
-			(at 115.57 69.85 0)
+			(at 113.03 101.6 0)
 			(effects
 				(font
@@
 		)
 		(property "Description" ""
-			(at 115.57 69.85 0)
+			(at 113.03 101.6 0)
 			(effects
 				(font
@@
 			(project "basschorus"
 				(path "/7f3b4bac-3b2a-4af0-92ae-ccc3fcedc393/266c062e-3d0a-4a44-9ad1-7a160f1a9b37"
-					(reference "R_CUTOFF_1")
-					(unit 2)
-				)
-			)
-		)
-	)
-	(symbol
-		(lib_id "Device:R_Potentiometer_Dual_Separate")
-		(at 113.03 101.6 270)
-		(unit 1)
-		(exclude_from_sim no)
-		(in_bom yes)
-		(on_board yes)
-		(dnp no)
-		(property "Reference" "R_CUTOFF_1"
-			(at 113.03 96.3422 90)
-			(effects
-				(font
-					(size 1.27 1.27)
-				)
-			)
-		)
-		(property "Value" "A100K"
-			(at 113.03 98.6536 90)
-			(effects
-				(font
-					(size 1.27 1.27)
-				)
-			)
-		)
-		(property "Footprint" "Potentiometer_THT:Potentiometer_Alpha_RD902F-40-00D_Dual_Vertical_CircularHoles"
-			(at 113.03 101.6 0)
-			(effects
-				(font
-					(size 1.27 1.27)
-				)
-				(hide yes)
-			)
-		)
-		(property "Datasheet" "~"
-			(at 113.03 101.6 0)
-			(effects
-				(font
-					(size 1.27 1.27)
-				)
-				(hide yes)
-			)
-		)
-		(property "Description" ""
-			(at 113.03 101.6 0)
-			(effects
-				(font
-					(size 1.27 1.27)
-				)
-			)
-		)
-		(pin "1"
-		)
-		(pin "2"
-		)
-		(pin "3"
-		)
-		(pin "4"
-		)
-		(pin "5"
-		)
-		(pin "6"
-		)
-		(instances
-			(project "basschorus"
-				(path "/7f3b4bac-3b2a-4af0-92ae-ccc3fcedc393/266c062e-3d0a-4a44-9ad1-7a160f1a9b37"
-					(reference "R_CUTOFF_1")
+					(reference "RV12")
 					(unit 1)
 				)
@@
 				)
 			)
+		)
+	)
+	(symbol
+		(lib_id "Device:R_Potentiometer_Dual_Separate")
+		(at 115.57 69.85 270)
+		(unit 2)
+		(exclude_from_sim no)
+		(in_bom yes)
+		(on_board yes)
+		(dnp no)
+		(property "Reference" "RV12"
+			(at 115.57 64.5922 90)
+			(effects
+				(font
+					(size 1.27 1.27)
+				)
+			)
+		)
+		(property "Value" "R_CUTOFF_A100K"
+			(at 115.57 66.9036 90)
+			(effects
+				(font
+					(size 1.27 1.27)
+				)
+			)
+		)
+		(property "Footprint" "Potentiometer_THT:Potentiometer_Alpha_RD902F-40-00D_Dual_Vertical_CircularHoles"
+			(at 115.57 69.85 0)
+			(effects
+				(font
+					(size 1.27 1.27)
+				)
+				(hide yes)
+			)
+		)
+		(property "Datasheet" "~"
+			(at 115.57 69.85 0)
+			(effects
+				(font
+					(size 1.27 1.27)
+				)
+				(hide yes)
+			)
+		)
+		(property "Description" ""
+			(at 115.57 69.85 0)
+			(effects
+				(font
+					(size 1.27 1.27)
+				)
+			)
+		)
+		(pin "1"
+		)
+		(pin "2"
+		)
+		(pin "3"
+		)
+		(pin "4"
+		)
+		(pin "5"
+		)
+		(pin "6"
+		)
+		(instances
+			(project "basschorus"
+				(path "/7f3b4bac-3b2a-4af0-92ae-ccc3fcedc393/266c062e-3d0a-4a44-9ad1-7a160f1a9b37"
+					(reference "RV12")
+					(unit 2)
+				)
+			)
