File: chorus2/basschorus/basschorus.kicad_sch (KiCad schematic)
At the start: 56 parts, among them J1 IN, J2 Jack-DC, J3 OUT, SW1 SW_3PDT_x3, U1 TL074, U2 TL074, U3 TL074, U4 LM317_TO-220, U5 MAX1044, U6 LM317_TO-220, U7 LM337_TO220

Commit message: resize to get under engineering fee size
Parts:
- J1, J3: footprint _effects_shared_footprints:Jack_6.35mm_Neutrik_NMJ6HCD3_Horizontal -> _project:JackHeaders
- SW1: footprint _effects_shared_footprints:Stompbox Switch -> Connector_PinHeader_2.54mm:PinHeader_1x09_P2.54mm_Vertical
Changed lines of the file:
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@@
 			)
 		)
-		(property "Footprint" "_effects_shared_footprints:Jack_6.35mm_Neutrik_NMJ6HCD3_Horizontal"
+		(property "Footprint" "_project:JackHeaders"
 			(at 277.495 147.32 0)
 			(effects
@@
 			)
 		)
-		(property "Footprint" "_effects_shared_footprints:Stompbox Switch"
+		(property "Footprint" "Connector_PinHeader_2.54mm:PinHeader_1x09_P2.54mm_Vertical"
 			(at 35.56 119.38 0)
 			(effects
@@
 			)
 		)
-		(property "Footprint" "_effects_shared_footprints:Stompbox Switch"
+		(property "Footprint" "Connector_PinHeader_2.54mm:PinHeader_1x09_P2.54mm_Vertical"
 			(at 260.985 142.24 0)
 			(effects
@@
 			)
 		)
-		(property "Footprint" "_effects_shared_footprints:Jack_6.35mm_Neutrik_NMJ6HCD3_Horizontal"
+		(property "Footprint" "_project:JackHeaders"
 			(at 20.32 124.46 0)
 			(effects
@@
 			)
 		)
-		(property "Footprint" "_effects_shared_footprints:Stompbox Switch"
+		(property "Footprint" "Connector_PinHeader_2.54mm:PinHeader_1x09_P2.54mm_Vertical"
 			(at 78.74 28.575 0)
 			(effects
