File: chorus2/basschorus/basschorus.kicad_pcb (KiCad board)
At the start: 4 copper layers, 89.4 x 97.5 mm, 136 parts, among them J1 IN, J2 Jack-DC, J3 OUT, J4 AVR-ISP-6, SW1 SW_3PDT_x3, U1 TL074, U2 TL074, U3 TL074, U4 LM317_TO-220, U5 MAX1044, U6 LM317_TO-220, U7 LM337_TO220, U8 ATtiny25-20S

Commit message: basic layout
Parts:
- removed R_CUTOFF_1: A100K, Potentiometer_THT:Potentiometer_Alpha_RD902F-40-00D_Dual_Vertical_CircularHoles
- added REF**: TestPoint_Keystone_5005-5009_Compact, TestPoint:TestPoint_Keystone_5005-5009_Compact, F.Cu at (106.7, 101.6)
- added REF**: TestPoint_Keystone_5005-5009_Compact, TestPoint:TestPoint_Keystone_5005-5009_Compact, F.Cu at (111.8, 101.6)
- added REF**: TestPoint_Keystone_5005-5009_Compact, TestPoint:TestPoint_Keystone_5005-5009_Compact, F.Cu at (106.7, 106.7)
- added REF**: TestPoint_Keystone_5005-5009_Compact, TestPoint:TestPoint_Keystone_5005-5009_Compact, F.Cu at (111.8, 111.8)
- added REF**: TestPoint_Keystone_5005-5009_Compact, TestPoint:TestPoint_Keystone_5005-5009_Compact, F.Cu at (149.9, 63.5)
- added REF**: TestPoint_Keystone_5005-5009_Compact, TestPoint:TestPoint_Keystone_5005-5009_Compact, F.Cu at (149.9, 73.7)
- added REF**: TestPoint_Keystone_5005-5009_Compact, TestPoint:TestPoint_Keystone_5005-5009_Compact, F.Cu at (111.8, 106.7)
- added REF**: TestPoint_Keystone_5005-5009_Compact, TestPoint:TestPoint_Keystone_5005-5009_Compact, F.Cu at (106.7, 111.8)
- added REF**: TestPoint_Keystone_5005-5009_Compact, TestPoint:TestPoint_Keystone_5005-5009_Compact, F.Cu at (149.9, 68.6)
- added REF**: TestPoint_Keystone_5005-5009_Compact, TestPoint:TestPoint_Keystone_5005-5009_Compact, F.Cu at (154.9, 68.6)
- added REF**: TestPoint_Keystone_5005-5009_Compact, TestPoint:TestPoint_Keystone_5005-5009_Compact, F.Cu at (154.9, 83.8)
- added REF**: TestPoint_Keystone_5005-5009_Compact, TestPoint:TestPoint_Keystone_5005-5009_Compact, F.Cu at (149.9, 88.9)
- added REF**: TestPoint_Keystone_5005-5009_Compact, TestPoint:TestPoint_Keystone_5005-5009_Compact, F.Cu at (154.9, 73.7)
- added REF**: TestPoint_Keystone_5005-5009_Compact, TestPoint:TestPoint_Keystone_5005-5009_Compact, F.Cu at (144.8, 78.7)
- added REF**: TestPoint_Keystone_5005-5009_Compact, TestPoint:TestPoint_Keystone_5005-5009_Compact, F.Cu at (149.9, 78.7)
- added REF**: TestPoint_Keystone_5005-5009_Compact, TestPoint:TestPoint_Keystone_5005-5009_Compact, F.Cu at (144.8, 83.8)
- added REF**: TestPoint_Keystone_5005-5009_Compact, TestPoint:TestPoint_Keystone_5005-5009_Compact, F.Cu at (144.8, 88.9)
- added REF**: TestPoint_Keystone_5005-5009_Compact, TestPoint:TestPoint_Keystone_5005-5009_Compact, F.Cu at (149.9, 83.8)
- added REF**: TestPoint_Keystone_5005-5009_Compact, TestPoint:TestPoint_Keystone_5005-5009_Compact, F.Cu at (154.9, 88.9)
- added REF**: TestPoint_Keystone_5005-5009_Compact, TestPoint:TestPoint_Keystone_5005-5009_Compact, F.Cu at (154.9, 63.5)
- added REF**: TestPoint_Keystone_5005-5009_Compact, TestPoint:TestPoint_Keystone_5005-5009_Compact, F.Cu at (154.9, 78.7)
- added RV12: R_CUTOFF_A100K, Potentiometer_THT:Potentiometer_Alpha_RD902F-40-00D_Dual_Vertical_CircularHoles, F.Cu at (114.3, 94.0)
- R1, R10, R11, R12, R13, R14, R15, R16, R17, R18, R19, R2, R20, R21, R22, R23, R24, R25, R26, R27, R28, R29, R3, R30, R31, R32, R33, R34, R35, R36, R37, R38, R39, R4, R40, R41, R42, R43, R44, R45, R46, R47, R5, R6, R7, R8, R9: footprint Resistor_THT:R_Axial_DIN0204_L3.6mm_D1.6mm_P5.08mm_Horizontal -> Resistor_THT:R_Axial_DIN0204_L3.6mm_D1.6mm_P2.54mm_Vertical
- TP7: value COMP_GAIN -> C_GAIN
- TP8: value COMP_IN -> C_IN
- TP9: value COMP_OUT -> C_OUT
- moved R39 158.5 mm to (133.3, 149.9), turned to -90 degrees
- moved R38 157.7 mm to (141.0, 152.4), turned to 180 degrees
- moved R37 152.9 mm to (146.1, 147.3)
- moved R40 149.6 mm to (146.1, 152.4)
- moved RV7 137.8 mm to (152.4, 148.6), turned to -90 degrees
- moved C1 136.6 mm to (137.1, 135.9)
- moved U1 136.4 mm to (139.6, 143.5)
- moved R33 128.8 mm to (119.4, 133.3)
- moved R36 127.6 mm to (146.1, 138.4)
- moved R35 124.4 mm to (148.6, 133.3), turned to 180 degrees
- moved C31 123.2 mm to (151.1, 141.0)
- moved C29 120.2 mm to (127.1, 139.7)
- moved R34 118.4 mm to (119.4, 138.4)
- moved C32 113.8 mm to (156.1, 135.9), turned to 180 degrees
- moved TP4 105.3 mm to (156.2, 130.8)
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Connections:
- C23 pad 2: Net-(U2A-+) -> Net-(U2D--)
- C28 pad 1: Net-(U2B--) -> Net-(U2A-+)
- C30 pad 1: Net-(U1B-+) -> Net-(U1A-+)
- C32 pad 2: Net-(U1C-+) -> Net-(U1D--)
- R10 pad 1: Net-(U2D--) -> Net-(U2B--)
- R11 pad 2: Net-(U2D--) -> Net-(U2B--)
- R2 pad 1: Net-(U1A-+) -> Net-(U1B-+)
- R25 pad 1: Net-(U2A-+) -> Net-(U2D--)
- R3 pad 1: Net-(U1A-+) -> Net-(U1B-+)
- R31 pad 1: Net-(U2B--) -> Net-(U2A-+)
- R33 pad 2: Net-(U1B-+) -> Net-(U1A-+)
- R35 pad 2: Net-(U1B--) -> Net-(U1A--)
- R36 pad 1: Net-(U1C-+) -> Net-(U1D--)
- R37 pad 1: Net-(U1D--) -> Net-(U1C-+)
- R38 pad 1: Net-(U1D-+) -> Net-(U1C--)
- R39 pad 2: Net-(U1D-+) -> Net-(U1C--)
- R40 pad 2: Net-(U1D--) -> Net-(U1C-+)
- R5 pad 2: Net-(U1A-+) -> Net-(U1B-+)
- R9 pad 1: Net-(U2D--) -> Net-(U2B--)
- RV2 pad 3: Net-(U2D--) -> Net-(U2B--)
- RV6 pad 2: Net-(U2A--) -> Net-(U2D-+)
- TP1 pad 1: Net-(U2A--) -> Net-(U2D-+)
- TP4 pad 1: Net-(U1B--) -> Net-(U1A--)
- U1 pad 1: /tone splitter/IN -> Net-(U1A--)
- U1 pad 12: Net-(U1D-+) -> /Compressor/IN
- U1 pad 14: /tone splitter/DRY_OUT -> /Compressor/IN
- U1 pad 2: GND -> Net-(U1A--)
- U1 pad 6: Net-(U1B--) -> GND
- U1 pad 7: Net-(U1B--) -> /tone splitter/IN
- U1 pad 8: /Compressor/IN -> /tone splitter/DRY_OUT
- U1 pad 9: /Compressor/IN -> Net-(U1C--)
- U2 pad 1: /BBD/SIG_IN -> /reconstruction filter/OUT
- U2 pad 12: GND -> Net-(U2D-+)
- U2 pad 14: Net-(SW1C-A) -> /BBD/SIG_IN
- U2 pad 2: Net-(U2A--) -> GND
- U2 pad 7: /reconstruction filter/OUT -> Net-(SW1C-A)
Routing:
- net -7.5V: track 29.5 -> 152.7 mm
- net +9V: track 60.4 -> 180.9 mm
- net +7.5V: track 33.7 -> 145.1 mm
- net Net-(U1A--): track 0.00 -> 93.8 mm, vias 0 -> 1
- net /Compressor/IN: track 0.00 -> 80.3 mm, vias 0 -> 1
- net Net-(SW1C-A): track 5.31 -> 76.1 mm
- net /Compressor/OUT: track 0.00 -> 57.8 mm, vias 0 -> 2
- net +5V: track 153.4 -> 209.1 mm, vias 0 -> 2
- net Net-(R2-Pad2): track 25.2 -> 77.2 mm
- net /tone splitter/DRY_OUT: track 0.00 -> 47.6 mm
- net Net-(R34-Pad1): track 0.00 -> 45.5 mm
- net /BBD/SIG_IN: track 32.8 -> 78.1 mm, vias 0 -> 1
- net Net-(R33-Pad1): track 0.00 -> 45.1 mm
- net /tone splitter/IN: track 0.00 -> 39.6 mm
- net Net-(D4-A): track 0.00 -> 38.1 mm
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Other:
- board size 89.4 x 97.5 mm -> 95.2 x 118.1 mm
- board text added: "BassChorus PREREV 0 2026-10-26"

Commit message: cleanup
Parts:
- added TP23: GND, TestPoint:TestPoint_THTPad_2.5x2.5mm_Drill1.2mm, F.Cu at (121.9, 175.3)
- added TP24: GND, TestPoint:TestPoint_THTPad_2.5x2.5mm_Drill1.2mm, F.Cu at (127.0, 175.3)
- R4: value 10k -> 1k
- TP7: value C_GAIN -> CGAIN
- TP8: value C_IN -> CIN
- TP9: value C_OUT -> COUT
- moved R43 9.16 mm to (129.5, 119.4)
- moved TP1 8.13 mm to (119.4, 111.8)
- moved R26 5.08 mm to (124.5, 116.8)
- moved R41 2.54 mm to (134.6, 99.1)
- moved R42 2.54 mm to (129.5, 99.1)
- moved RV8 2.54 mm to (129.5, 106.7)
- moved RV9 2.54 mm to (129.6, 94.0)
Connections:
- J1 pad TN: GND -> unconnected-(J1-PadTN)
- J3 pad TN: GND -> unconnected-(J3-PadTN)
Routing:
- net Net-(U3A--): track 20.6 -> 12.2 mm
- net +5V: track 209.1 -> 216.6 mm, vias 2 -> 3
- net GND: track 15.0 -> 21.9 mm, vias 4 -> 7
- net Net-(U2D-+): track 29.5 -> 35.9 mm, vias 0 -> 1
- net Net-(RV8-Pad3): track 23.3 -> 28.9 mm
- net Net-(D3-A): track 15.7 -> 20.1 mm
- net /Compressor/IN: track 80.3 -> 77.8 mm
- net Net-(R26-Pad2): track 9.72 -> 7.62 mm
- net Net-(U3B-+): track 22.0 -> 20.7 mm
Other:
- board size 95.2 x 118.1 mm -> 95.2 x 117.9 mm

Commit message: resize to get under engineering fee size
Parts:
- J1, J3: footprint _effects_shared_footprints:Jack_6.35mm_Neutrik_NMJ6HCD3_Horizontal -> _project:JackHeaders
- SW1: footprint _effects_shared_footprints:Stompbox Switch -> Connector_PinHeader_2.54mm:PinHeader_1x09_P2.54mm_Vertical
- moved TP23 18.3 mm to (132.1, 160.0)
- moved TP24 18.3 mm to (137.2, 160.0)
- moved J3 18.1 mm to (73.7, 160.0), turned to 90 degrees
- moved SW1 15.7 mm to (121.9, 160.0)
- moved D1 14.8 mm to (86.4, 160.0), turned to 0 degrees
- moved J1 10.2 mm to (149.9, 160.0), turned to -90 degrees
- moved R4 3.59 mm to (96.5, 160.0), turned to 180 degrees
Routing:
- net Net-(SW1C-B): track 24.2 -> 32.4 mm
- net Net-(SW1A-C): track 12.0 -> 16.2 mm
- net Net-(SW1B-B): track 18.0 -> 22.2 mm, vias 0 -> 1
- net Net-(SW1A-A): track 22.7 -> 19.7 mm
- net Net-(SW1C-A): track 76.1 -> 73.3 mm
- net Net-(SW1A-B): track 29.2 -> 30.3 mm
Other:
- board size 95.2 x 117.9 mm -> 95.5 x 101.6 mm
